File: TI980A-Arithmetic-Unit/AU1-INT-LOGIC.kicad_sch (KiCad schematic)
At the start: 29 parts, among them U121 74H11N, U13 74H00N, U154 74H30N, U166 7402N, U166 74H30N, U167 74H11N, U168 74H21N, U169 7400N, U170 7404N, U180 7400N, U181 7474N, U212 7420N, U212 7474N, U22 74H04N, U27 74H103N, U35 74H103N, U47 7404N, U56 74H00N, U64 7400N, U76 74H00N, U8 74H04N, U80 7410N, U80 7474N, U81 7404N, U90 7474N

Commit message: Finished Up to Column 3 on AU2
Parts:
- R22: value ~ -> (none)
- renumbered U166 to U171, U166 to U188, U181 to U189, U154 to U203, U212 to U216, U80 to U230
