File: TI980A-Arithmetic-Unit/AU1.kicad_sch (KiCad schematic)
At the start: 71 parts, among them U1 7413N, U10 74H04N, U11 74H04N, U12 74LS74, U13 74H00N, U14 74H10, U2 7474N, U21 7437N, U22 74H04N, U23 74H04N, U24 74H04N, U25 74H40N, U26 7402N, U27 74H103N, U28 74H04N, U29 74H04N, U3 7437N, U30 74H04N, U31 74H10N, U32 74H103N, U33 74H21N, U34 7432N, U35 74H103N, U36 7402N, U37 7408N, U4 7404N, U43 74H52N, U44 7400, U45 7404N, U46 74H52N, U47 7404N, U48 7408N, U49 7474N, U5 7408N, U50 7410N, U51 74H11N, U52 74H61N, U53 74H61N, U54 7402N, U55 7402N, U56 74H00N, U57 7410N, U58 7402N, U59 7432N, U6 7404N, U60 7402N, U61 7430N, U62 7410N, U63 7486N, U64 7400N, U64A 7400N, U65 7430N, U66 7404N, U7 74H05N, U8 74H04N, U9 74H54W

Commit message: Updated Schematics and Library
Parts:
- removed U4: 7404N, symbol 74xx:74LS04
- added J1: Circuit Type Test, symbol Connector_Generic:Conn_02x08_Counter_Clockwise
- added R10, R11, R12, R13, R14, R15, R16, R9: R, symbol Device:R
- added U100, U111, U115, U127, U134, U67, U68, U69, U74, U76, U84, U86, U97: 7410N, symbol 74xx:74LS10
- added U101, U128, U80, U90: 7474N, symbol 74xx:74LS74
- added U102, U106, U108, U119, U131, U82, U94, U95, U96, U98: 74H52N, symbol TI980A:74H52N
- added U103, U92: 74163, symbol 74xx:74LS163
- added U104: 7408N, symbol 74xx:74LS08
- added U105, U110, U116, U121, U124: 74H11N, symbol 74xx:74LS11
- added U107, U135, U78, U79: 7451N, symbol TI980A:7451N
- added U109, U123, U93: 7404N, symbol 74xx:74LS04
- added U112, U136, U70, U87, U91: 7420N, symbol 74xx:74LS20
- added U113, U129, U73, U77, U85, U99: 7400N, symbol 74xx:7400
- added U114, U81: 74H54W, symbol TI980A:74H54N
- added U117: 74H04N, symbol 74xx:74LS04
- added U118: 74H21N, symbol 74xx:74LS21
- added U120: 74188N, Package_DIP:DIP-16_W7.62mm, symbol TI980A:74188
- added U122: 74157N, symbol 74xx:74LS157
- added U126, U130: 74H01N, Package_DIP:DIP-14_W7.62mm, symbol TI980A:74H01N
- added U132: 74H05N, symbol 74xx:74LS05
- added U133, U89: 74H22N, symbol 74xx:74LS22
- added U137: 7427N, symbol 74xx:74LS27
- added U138: 74S22N, symbol 74xx:74LS22
- added U139: 74S65N, symbol TI980A:74S65N
- added U4: 74H20N, symbol 74xx:74LS20
- added U71: 74S11N, symbol 74xx:74LS11
- added U72: 74H10N, symbol 74xx:74LS10
- added U75: 7437N, symbol 74xx:74LS37
- added U83: 7486N, symbol 74xx:74LS86
- added U88: 7442, symbol 74xx:74LS42
- U9: Location AU1 Column 14 Row 012 -> AU1 Column 14 Row 02
- renumbered U64A to U64
Connections:
- net ALUEQZ: now also U68.5
- net AR14: now also U82.10, U83.9
- net AR15: now also U83.1
- net AR2: now also U83.12
- net BYTEINC: now also U75.11
- net CPUCR: now also U81.10
- net CYCOMP: now also U124.11, U124.5
- net DMAREC: now also U80.9 (Q)
- net ENATI2: now also U124.8
- net ENIRLOAD: now also U72.12
- net ENPCINC: now also U65.8
- net ENSR16LD: now also U55.1
- net EXTSTCK: now also U81.3
- net FSWON: now also U133.4
- net GND: now also J1.10 (Pin_10), J1.11 (Pin_11), J1.12 (Pin_12), J1.13 (Pin_13), U81.1, U81.13
- net IR8: now also U82.4
- net IR9T: now also U83.10, U83.2
- net L1: now also U14.2, U133.2
- net L8: now also U67.4, U68.13, U82.13, U84.11
- net L9: now also U77.10, U78.9
- net LBC: now also U37.13
- net M0LF: now also U55.10
- net M1LE: now also U55.13
- net M5: now also U68.2, U77.9
- net M8: now also U14.1, U37.12, U64.1
- net MADOIT: now also U4.8
- net ME: now also U124.3, U133.1, U78.10
- net PNLENQ: now also U81.6; no longer U14.1
- net SELBFR: now also J1.8 (Pin_8)
- net ST10: now also U84.10
- net ST7: now also U84.3
- net ST8: now also U84.1
- net VCC1: now also J1.14 (Pin_14), J1.15 (Pin_15), J1.16 (Pin_16), R10.1, R11.1, R12.1, R13.1, R14.1, R15.1, R16.1, R9.1, U128.1 (~{R}), U128.10 (~{S}), U128.13 (~{R}), U128.4 (~{S}), U133.5, U70.9, U71.11, U79.13, U80.1 (~{R}), U80.10 (~{S}), U80.13 (~{R}), U80.4 (~{S}), U81.2
- net XRMAX: now also U82.1
- net ~{ADRV}: now also U68.1, U82.3
- net ~{ALUEQ8K}: now also U14.13
- net ~{APOPCOMP}: now also U124.1
- net ~{BRLD}: now also U78.8
- net ~{CLKONQ}: now also U81.4; no longer U14.2
- net ~{CYC}: now also U81.9
- net ~{EXTSTCK}: now also R14.2
- net ~{FCLKT}: now also U80.11 (C)
- net ~{GCLKF:1}: now also U128.11 (C)
- net ~{GCLKF:2}: now also U80.3 (C)
- net ~{IFLAGQ}: now also U70.13
- net ~{INTABORT}: now also R9.2, U124.2
- net ~{L5}: now also U67.1
- net ~{L6}: now also U67.2
- net ~{LC}: now also U55.3, U73.13
- net ~{LE}: now also U55.12
- net ~{LF}: now also U55.9
- net ~{LSB11}: now also U80.6 (~{Q})
- net ~{MA}: now also U73.12
- net ~{MC}: now also U55.2
- net ~{MDIDSW}: now also U44.10
- net ~{MDIESW}: now also U44.9
- net ~{R36}: now also U65.11
- net ~{SELPA1}: now also R15.2
- net ~{SETRUN}: no longer U31.13
- net ~{SKIP}: now also U65.6
- net ~{STEPULS}: now also U31.13, U81.5; no longer U14.13
- net ~{STPCK}: now also U81.8
- net ~{STPIOCLK}: no longer U14.12
- net ~{M8L1ALU}: now reaches U48.1
- net ~{M8L1ALU}: now also U14.12
- net ~{M8L0}: now reaches U48.2
- net ~{M8L0}: now also U64.3
- net ~{ENARCLR}: now reaches U48.3
- net ~{MO}: now reaches U55.8
- net ~{PCIS08}: now reaches U65.1
- net ~{PCIS08}: now also U67.6
- net ~{PCISA3}: now reaches U65.12
- net ~{PCISA3}: now also U70.8
- net ~{PCIS0B}: now reaches U65.2
- net ~{PCIS0B}: now also U67.8
- net ~{PCIS7D}: now reaches U65.3
- net ~{PCIS7D}: now also U68.6
- net ~{PCISAD}: now reaches U65.4
- net ~{PCISAD}: now also U4.13, U69.6
- net ~{ENPCOUT}: now reaches U65.5
- net ~{ENPCOUT}: now also U4.9
- net LA: now reaches U62.10
- net ST2T: now reaches U62.11
- net ~{MBLAST2}: now reaches U62.8
- net MB: now reaches U62.9
- net ~{M1}: now reaches U55.11
- net MDI: now reaches U44.8
- net MDI: now also U74.13
- net L0: now reaches U64.2
- net L0: now also U124.10, U127.5
- net M8LBC: now reaches U37.11
- new net ADRB: U82.12
- new net AR0XAR2: U83.11
- new net AR14XIR9: U83.8
- new net AR15XIR9: U83.3
- new net BFR3: U126.3
- new net BFR4: U126.11
- new net BFR6: U126.8
- new net BFR7: R11.2, U126.6
- new net BSDQ: U128.5 (Q)
- new net BSDQD: R13.2, U128.2 (D)
- new net C8OP: R12.2
- new net DBL: R16.2
- new net DMARECD: U80.12 (D)
- new net ENLRAINC: U124.6
- new net ESPQ: U84.13
- new net EXTFORM: U67.11, U71.9
- new net FORCE00: J1.9 (Pin_9), U79.1
- new net INSRTOP: U126.1, U126.12, U126.4, U126.9
- new net IOQ: U84.5
- new net IR6EXTF: U67.5, U71.8
- new net IR8T: U127.3
- new net L3: U124.4, U70.12
- new net L4: U124.13, U82.2
- new net L567: U67.12
- new net L6: U82.11
- new net L7: U82.5
- new net LB: U67.10
- new net LD: U68.4, U69.4, U78.13
- new net LE: U74.2
- new net LSB11: U80.5 (Q)
- new net M0: U67.3, U67.9
- new net M1: U78.1
- new net M5J1: U82.8
- new net M5T: U127.4
- new net M7: U68.3
- new net M8J1: U68.8
- new net MA: U69.3, U70.10
- new net MAL2CYC: U80.2 (D)
- new net MC: U124.9
- new net MCL4P4: U124.12
- new net MD: U74.1
- new net RDYIO: U128.12 (D)
- new net RDYQ: U128.9 (Q), U69.5
- new net RR: R10.2
- new net SC0: U127.11
- new net SC1: U127.10
- new net SCNT06: U127.9
- new net SELJ0: J1.1 (Pin_1)
- new net SELJ1: J1.2 (Pin_2)
- new net SELJ2: J1.3 (Pin_3)
- new net SELJ3: J1.4 (Pin_4)
- new net SELOP: J1.7 (Pin_7), U79.8
- new net SELPA: J1.5 (Pin_5)
- new net SELPA1: J1.6 (Pin_6)
- new net ~{AR0T}: U83.13
- new net ~{BSDQ}: U128.6 (~{Q})
- new net ~{BYTEINCA}: U68.12, U75.12, U75.13, U77.8
- new net ~{DMAREC}: U80.8 (~{Q})
- new net ~{EXPM}: U84.12
- new net ~{EXTFORM}: U84.9
- new net ~{FNPCOUT}: U72.13
- new net ~{FORCE00}: U79.10
- new net ~{IOM}: U84.6
- new net ~{IR6T}: U71.10
- new net ~{L7}: U67.13
- new net ~{M0L4BFR}: U4.12, U72.2
- new net ~{M0L8J1}: U84.8
- new net ~{M5L0IR8}: U127.6
- new net ~{M8L0J1}: U68.9
- new net ~{M8L456J1}: U68.10
- new net ~{M8LEJ1}: U68.11
- new net ~{MAISDE}: U4.10, U74.12
- new net ~{MALC}: U72.1, U73.11
- new net ~{MEM0}: U126.2
- new net ~{MEM13}: U127.1
- new net ~{MEM14}: U127.2
- new net ~{MEM15}: U127.13
- new net ~{MEM1}: U126.13
- new net ~{MEM3}: U126.10
- new net ~{MEM4}: U126.5
- new net ~{PRINTINH}: U84.2, U84.4
- new net ~{RDYQ}: U128.8 (~{Q})
- new net ~{RRDESZ}: U127.12
- new net ~{SCNT1E}: U127.8
- new net ~{SELBFRCK}: U128.3 (C)
- new net ~{SELOP}: U79.9
- new net ~{SELPA}: U133.6
- no-connect marks 95 -> 114
Other:
- note added: "A Register [AR]"
- note added: "B Register and Control"
- note added: "BYTEINC CT To AU1 AU Interconnect P2 Pin 9 To AU2 AU Interconnect P2 Pin 9"
- note added: "E Register and Controls AU1 Part"
- note added: "ENAR16LD CT To AU1 AU Interconnect P2 Pin 49 To AU2 AU Interconnect P2 Pin 49"
- note added: "ENIRLOAD CT To AU1 AU Interconnect P1 Pin 26 To AU2 AU Interconnect P1 Pin 26"
- note added: "ENPCINC CT To AU1 AU Interconnect P2 Pin 41 To AU2 AU Interconnect P2 Pin 41"
- note added: "Intruction Register Clock Enable"
- note added: "M1LE CT To AU1 AU Interconnect P2 Pin 35 To AU2 AU Interconnect P2 Pin 35"
- note added: "MOLF CT To AU2 AU Interconnect P2 Pin 31"
- note added: "Memory Address Register and Control AU1 Part"
- note added: "S Register ALU 1 Part"
- note added: "S Register Bit 16 Load Control"
- note added: "Status Register"
- note added: "~{ENARCLR} CT To AU1 AU Interconnect P2 Pin 36 To AU2 AU Interconnect P2 Pin 36"
- note added: "~{MADOIT} CT To AU1 AU Interconnect P2 Pin 24 To AU2 AU Interconnect P2 Pin 24"
- note added: "~{MBLAST2} CT To AU1 AU Interconnect P2 Pin 13 To AU2 AU Interconnect P2 Pin 13"
- note added: "~{MBLAST2} CT To AU1 AU Interconnect P2 Pin 30 To AU2 AU Interconnect P2 Pin 30"
- note removed: "Buffered Synchronized Reset Signal"

Commit message: Finished Columns 1, 2, 3, 10, 11, 12, 13, and 14
Parts:
- added J2: Circuit Type Test, symbol Connector_Generic:Conn_02x08_Counter_Clockwise
- added R17, R18, R19, R20, R23, R24, R25, R26, R27, R29, R30, R31, R58, R59, R60, R61, R66, R68, R70, R71, R72: R, symbol Device:R
- added R57, R65: ~, symbol Device:R
- added U125: 74H51N, symbol TI980A:7451N
- added U140, U141, U144, U147: 74H52N, symbol TI980A:74H52N
- added U142, U143: 74175N, symbol 74xx:74LS175
- added U145, U146, U155, U157: 74187, Package_DIP:DIP-16_W7.62mm, symbol TI980A:74187
- added U148, U149, U150, U152, U158, U159, U161, U162, U163, U164: 74H61N, Package_DIP:DIP-14_W7.62mm, symbol TI980A:74H61N
- added U151, U160: 7451N, symbol TI980A:7451N
- added U153: 74S22N, symbol 74xx:74LS22
- added U154: 74H30N, symbol 74xx:74LS30
- added U156: 74H04N, symbol 74xx:74LS04
- added U165: 74LS83, symbol 74xx:74LS83
- U109: Location AU1 Column 13 Row 16 -> AU1 Column 11 Row 16
- U123: Location AU1 Column 13 Row 20 -> AU1 Column 10 Row 20
- U139: Location (none) -> AU1 Column 10 Row 19
- U79: value 7451N -> 74H51N
Connections:
- net ~{SC0} is gone; now on an unnamed net: U62.13
- net A0: now also U63.13
- net A1: now also U63.12
- net ADRV: now also U104.12
- net ALU0T: now also U138.4, U138.9
- net ALUEQZ: now also U139.10, U139.6
- net AR0: now also U22.13, U63.10, U88.13 (A2)
- net AR1: now also U63.9
- net AR14XIR9: now also U107.1, U109.5
- net AR15: now also U123.1
- net AR15XIR9: now also U113.4
- net BFR3: now also R23.2, U164.3
- net BFR4: now also U132.4, R18.2, U152.6
- net BFR6: now also U132.8
- net BFR7: now also U132.2, U164.6
- net BSDQ: now also U129.10, U134.4
- net BSDQD: now also U120.4 (D3)
- net C8OP: now also U105.1
- net CYCOMP: now also U121.5
- net DBL: now also U101.2 (D), U120.2 (D1)
- net ENATI1: now also U121.6
- net ER0: now also U88.14 (A1)
- net ER14: now also U110.10, U110.2, U123.5, U63.4
- net ER15: now also U63.5
- net EXTFORM: now also U135.10, U93.12, U99.13
- net FCLKT: now also U23.10, U24.5
- net FORCE00: now also U125.1, U125.5, U151.1, U151.5, U160.1, U160.5
- net GND: now also U103.8 (GND), U120.15 (~{CE}), U120.8 (GND), U122.15 (E), U122.8 (GND), U131.12, U131.13, U88.12 (A3), U88.8 (GND), U92.8 (GND), U142.8 (GND), U143.8 (GND), U145.13 (~{CE1}), U145.14 (~{CE2}), U145.8 (GND), U146.13 (~{CE1}), U146.14 (~{CE2}), U146.8 (GND), U155.13 (~{CE1}), U155.14 (~{CE2}), U155.8 (GND), U157.13 (~{CE1}), U157.14 (~{CE2}), U157.8 (GND), U165.11 (B1), U165.12 (GND), U165.16 (B4), U165.4 (B3), U165.7 (B2)
- net INAQ: now also U13.3
- net INSRTOP: now also U130.4
- net IR0: now also U158.13
- net IR1: now also U122.5 (I0b)
- net IR10T: now also U131.10, U131.4
- net IR11: now also U121.11
- net IR12T: now also U123.13, U89.2, U97.4
- net IR2: now also U122.2 (I0a)
- net IR3: now also U122.14 (I0d), U122.3 (I1a)
- net IR4: now also U122.11 (I0c)
- net IR5: now also U110.4, U137.10, U66.13
- net IR6: now also U109.13, U122.6 (I1b), U135.13, U137.9
- net IR7: now also U122.13 (I1d), U93.3
- net IR8: now also U122.10 (I1c)
- net IR8T: now also U117.3
- net J1SELA: now also U108.8
- net J1SELB: now also U102.8
- net L0: now also U121.13, U131.2
- net L1: now also U113.5, U22.4
- net L3: now also U110.11, U14.4, U5.13, U91.12
- net L5: now also U131.11, U137.1
- net L6: now also U107.9, U137.2
- net L7: now also U104.13, U134.5
- net L8: now also U110.5, U111.5, U136.13, U22.6
- net LA: now also U135.4, U137.13
- net LB: now also U105.9, U135.9, U73.5
- net LBC: now also U139.1, U86.2
- net LD: now also U100.13, U100.5, U112.13, U72.10, U97.13, U97.5, U99.10
- net LE: now also U107.4, U72.5, U73.2, U86.5
- net M0: now also U108.4, U113.13, U114.13
- net M3: now also U108.11
- net M4: now also U89.1
- net M5: now also U108.13, U114.3
- net M5J1: now also U108.12
- net M5T: now also U117.6
- net M8: now also U108.2, U130.9, U139.13, U86.1
- net M8J1: now also U108.1
- net M8LA: now also U138.13, U153.5
- net M8LE: now also U139.4
- net MA: now also U102.2, U105.10, U114.10, U119.3, U121.9, U72.9, U73.1, U91.10, U98.1
- net MAL2CYC: now also U121.8
- net MB: now also U102.11, U105.4, U114.6, U119.12, U121.3, U98.12
- net MC: now also U102.13, U119.10, U14.3
- net MD: now also U102.4, U98.10
- net MDR10: now also U112.12, U131.1, U87.12
- net ME: now also U119.1
- net MEM0: now also U23.1
- net MEM1: now also U24.1
- net MEM10: now also U10.11
- net MEM11: now also U10.1
- net MEM12: now also U100.10, U104.2, U109.9, U24.3
- net MEM13: now also U23.13
- net MEM14: now also U23.3
- net MEM15: now also U8.9
- net MEM2: now also U10.13
- net MEM3: now also U8.3
- net MEM4: now also U8.5
- net MEM5: now also U8.11
- net MEM7: now also U23.9
- net MEM8: now also U10.5
- net MEM9: now also U10.3
- net NRA0: now also J2.1 (Pin_1), U141.8, U142.4 (D0)
- net NRA1: now also U106.8, J2.2 (Pin_2), U142.5 (D1)
- net NRA2: now also J2.3 (Pin_3), U140.8, U142.12 (D2)
- net NRA3: now also J2.4 (Pin_4), U142.13 (D3), U144.8
- net NRA4: now also J2.5 (Pin_5), U143.4 (D0), U147.8
- net NRA5: now also U95.8, J2.6 (Pin_6), U143.5 (D1)
- net NRA6: now also U96.8, J2.7 (Pin_7), U143.12 (D2)
- net NRA7: now also U94.8, J2.8 (Pin_8), U143.13 (D3)
- net R22: now also U22.11, U89.10
- net R39: now also U103.7 (CEP), U85.10, U92.7 (CEP)
- net RDYQ: now also U112.9, U72.11, U97.3
- net RM: now also U148.11, U156.9, U158.11
- net RR: now also U104.1, U120.3 (D2)
- net SC0: now also U116.5, U139.12, U86.13, U92.14 (Q0)
- net SC1: now also U103.11 (Q3), U115.13, U116.13, U116.4
- net SC2: now also U103.12 (Q2)
- net SC3: now also U100.2, U103.13 (Q1), U107.10, U73.4, U93.1
- net SC4: now also U103.14 (Q0), U115.2, U116.2
- net SCNT06: now also U115.1, U116.1, U116.3, U66.1
- net SCNTZ: now also U105.11, U105.3
- net SELBFR: now also U150.2, U150.5, U151.8, U152.5, U161.2, U163.5, U164.2, U164.4
- net SELJ0: now also U106.1, U94.1, U95.1, U96.1, U140.1, U141.1, U144.1, U147.1, U160.8
- net SELJ1: now also U106.10, U94.10, U95.10, U96.10, U125.6, U140.10, U141.10, U144.10, U147.10
- net SELJ2: now also U106.12, U94.12, U95.12, U96.12, U125.8, U140.12, U141.12, U144.12, U147.12
- net SELJ3: now also U106.4, U94.4, U95.4, U96.4, U140.4, U141.4, U144.4, U147.4
- net SELOP: now also U148.12
- net SELPA: now also U149.12, U149.2, U149.5, U151.6, U152.12, U161.12, U162.2, U163.2, U164.12
- net SELPA1: now also U148.2, U148.5, U150.12, U152.2, U160.6, U161.5, U162.12, U162.5, U163.12
- net SELPA1A: now also U98.8
- net ST0: now also U123.9
- net ST1: now also U85.2
- net ST11: now also U13.10
- net ST12: now also U86.9
- net ST14: now also U13.9
- net ST2: now also U123.11, U135.5
- net TERM: now also U12.9 (Q)
- net UR0: now also U88.15 (A0), U153.2
- net VCC1: now also U101.1 (~{R}), U101.10 (~{S}), U101.13 (~{R}), U101.4 (~{S}), U102.5, U103.10 (CET), U103.16 (VCC), U105.13, U106.3, U108.5, U114.4, U119.5, U12.10 (~{S}), U12.13 (~{R}), U120.16 (VCC), U122.16 (VCC), U88.16 (VCC), U89.13, U89.5, U90.1 (~{R}), U90.10 (~{S}), U90.13 (~{R}), U90.4 (~{S}), U91.9, U92.16 (VCC), U92.4 (D1), U92.5 (D2), U92.6 (D3), U94.3, U95.3, U96.3, U98.3, U98.5, R17.1, R18.1, R19.1, R20.1, R23.1, R24.1, R25.1, R26.1, R27.1, R29.1, R30.1, R31.1, R57.1, R58.1, R59.1, R60.1, R61.1, R65.1, R66.1, R68.1, R70.1, R71.1, R72.1, U125.13, U125.4, U140.3, U141.3, U142.1 (~{Mr}), U142.16 (VCC), U143.1 (~{Mr}), U143.16 (VCC), U144.3, U145.16 (VCC), U146.16 (VCC), U147.3, U148.1, U148.13, U148.4, U149.1, U149.11, U149.4, U150.1, U150.11, U150.4, U151.13, U151.4, U152.1, U152.11, U152.4, U153.13, U154.11, U154.12, U154.6, U155.16 (VCC), U157.16 (VCC), U158.1, U158.4, U159.1, U159.11, U159.3, U159.4, U160.13, U160.4, U161.1, U161.11, U161.4, U162.1, U162.11, U162.4, U163.1, U163.11, U163.4, U164.1, U164.11, U164.5, U165.13 (C0), U165.5 (VCC)
- net ~{AEQZ}: now also U86.3
- net ~{ALUEQ8K}: now also U139.3, U153.9
- net ~{AR0T}: now also U22.12
- net ~{BSDQ}: now also U136.12, U137.11
- net ~{ENAPI2}: now also U14.6
- net ~{ENDRLOAD}: now also U5.8
- net ~{ENPCOUT}: now also U5.9
- net ~{EXPREC}: now also U8.12
- net ~{EXTFORM}: now also U87.6, U93.13
- net ~{FCLKT}: now also U12.11 (C), U24.6
- net ~{FORCE00}: now also U125.10, U125.3, U151.10, U151.3, U160.10, U160.3
- net ~{GCLKF:1}: now also U103.2 (CP), U92.2 (CP), U142.9 (Cp), U143.9 (Cp)
- net ~{GCLKF:2}: now also U90.11 (C), U90.3 (C)
- net ~{GOIO}: now also U93.8
- net ~{IFLAGQ}: now also U91.13
- net ~{IR10T}: now also U116.10
- net ~{IR6T}: now also U109.12, U110.3, U136.9
- net ~{IR8}: now also U117.4
- net ~{L1}: now also U22.3
- net ~{L8}: now also U22.5
- net ~{LDBTSW}: now also R26.2
- net ~{LF}: now also U89.4
- net ~{LRAMAX}: now also U5.12
- net ~{M0L8J1}: now also U136.4, U136.8
- net ~{M5L0IR8}: now also U104.4
- net ~{M5}: now also U117.5
- net ~{M8LEJ1}: now also U72.6
- net ~{MADSW}: now also R31.2
- net ~{MAESW}: now also R30.2
- net ~{MA}: now also U89.9
- net ~{MEM0}: now also U23.2
- net ~{MEM13}: now also U103.5 (D2), U23.12
- net ~{MEM14}: now also U103.4 (D1), U23.4
- net ~{MEM15}: now also U103.3 (D0), U8.8
- net ~{MEM1}: now also U24.2, U28.11
- net ~{MEM3}: now also U118.4, U28.13, U8.4
- net ~{MEM4}: now also U28.3, U8.6
- net ~{MRESETQ}: now also U121.1
- net ~{PCISA3}: now also U91.8
- net ~{PRINTINH}: now also U86.10; no longer U84.2
- net ~{R44}: now also U5.10
- net ~{RDYQ}: now also U100.1, U100.3
- net ~{RUNFFQ}: now also U107.5, U89.12
- net ~{SCER}: now also U86.12
- net ~{SCNT0F}: now also U110.13, U110.9, U115.12, U134.9
- net ~{SCNT1E}: now also U111.10, U115.10, U134.1, U97.2
- net ~{SELBFRCK}: now also U101.11 (C), U101.3 (C)
- net ~{SELJ1}: now also U139.8, R27.2, U125.2
- net ~{SELJ3}: now also U130.11, U130.8, U89.6, U89.8, R29.2
- net ~{SELPA1}: now also U138.8, U153.6, U153.8, U160.2
- net ~{SELPA}: now also U132.12, U132.6, U138.6, U151.2
- net ~{ST15}: now also U154.2
- net ~{ST2CLR}: now also U104.6
- net ~{ST5}: now also U109.1, U85.12, U154.3
- net ~{ST6}: now also U85.13, U154.4
- net ~{SYSCLK}: now also U23.11
- net ~{MEM11}: now reaches U10.2
- net ~{MEM11}: now also U118.12, U92.3 (D0)
- net SCNT0F: now reaches U116.12
- net SCNT0F: now also U135.3
- net ~{OVRST}: now reaches U104.5
- net MEM0A: now reaches U118.1
- net MEM0A: now also U120.14 (A4), U24.12, U33.1
- net MEM1A: now reaches U118.2
- net MEM1A: now also U120.13 (A3), U28.10, U33.2
- net ~{MEM2}: now reaches U118.5
- net ~{MEM2}: now also U10.12, U117.9, U130.5, U33.5
- net OPA: now reaches U118.6
- net MEM7A: now reaches U24.8
- net ~{MEM7}: now reaches U24.9
- net ~{MEM7}: now also U23.8, U91.2
- net LF: now reaches U115.11
- net LF: now also U107.3, U121.4
- net ~{MALFPA}: now reaches U115.8
- net ~{MALFPA}: now also U115.5
- net ~{AR1XIR9}: now reaches U115.9
- net ~{AR1XIR9}: now also U109.4
- net SPAREBFR: now reaches U120.1 (D0)
- net MEM4A: now reaches U120.10 (A0)
- net MEM4A: now also U28.4, U33.4
- net MEM3A: now reaches U120.11 (A1)
- net MEM3A: now also U28.12
- net MEM2A: now reaches U120.12 (A2)
- net MEM2A: now also U117.8
- net C80P: now reaches U120.5 (D4)
- net ~{INSRTOPA}: now reaches U120.6 (D5)
- net ~{SPLIMM}: now reaches U120.7 (D6)
- net ~{SPLIMM}: now also U117.1
- net ILLOP: now reaches U120.9 (D7)
- net ILLOP: now also R19.2
- net ~{M0L8PA1}: now reaches U113.11
- net ~{M0L8PA1}: now also U113.9
- net M0L8PA1: now reaches U113.12
- net M0L8PA1: now also U110.6
- net ~{CLCNT}: now reaches U92.1 (~{MR})
- net ~{CLCNT}: now also U103.1 (~{MR})
- net SCCRY: now reaches U92.10 (CET)
- net SCCRY: now also U103.15 (TC)
- net ~{LDSC}: now reaches U92.9 (~{PE})
- net ~{LDSC}: now also U103.9 (~{PE})
- net ~{SC4}: now reaches U100.4
- net ~{MALDPA}: now reaches U100.6
- net ~{MALDPA}: now also U115.4
- net ~{MEM0A}: now reaches U24.13
- net ~{STOT}: now reaches U85.1
- net STO1: now reaches U85.3
- net RR12: now reaches U101.12 (D)
- net RR12: now also U104.3
- net ~{RRINTINH}: now reaches U101.8 (~{Q})
- net ~{RRINTINH}: now also U84.2
- net RRINTINH: now reaches U101.9 (Q)
- net M8L23AJ3: now reaches U66.10
- net M8L23AJ3: now also U130.10
- net ~{M8L23AJ3}: now reaches U66.11
- net ~{M8L23AJ3}: now also U135.6
- net BFR5: now reaches U132.10
- net BFR5: now also U130.6, R20.2, U163.6
- net FORCZ: now reaches U132.11
- net FORCZ: now also U104.9, U118.8, U132.1, U132.3, U132.9
- net SELPAB: now reaches U132.5
- net SELPAB: now also U119.8
- net SHIFT: now reaches U105.12
- net SHIFT: now also U118.9
- net ~{MEM5}: now reaches U105.2
- net ~{MEM5}: now also U117.11, U8.10
- net ~{M0L9DOP}: now reaches U129.8
- net ~{M0L9DOP}: now also U112.2
- net L9D: now reaches U129.9
- net M0L8BEJ2: now reaches U66.8
- net M0L8BEJ2: now also U114.1
- net ~{M0L8BEJ2}: now reaches U66.9
- net ~{M0L8BEJ2}: now also U135.8
- net AL0E1U0: now reaches U139.11
- net M7L3: now reaches U139.2
- net AEUZ6: now reaches U139.5
- net AEUZ6: now also U109.10
- net M8LD: now reaches U139.9
- net M5L7J2: now reaches U114.2
- net M5L7J2: now also U104.11
- net MBL2J2: now reaches U114.5
- net ~{SELJ2A}: now reaches U114.8
- net MALCDJ2: now reaches U114.9
- net MALCDJ2: now also U99.6
- net MEM9A: now reaches U28.8
- net ~{MEM9}: now reaches U28.9
- net ~{MEM9}: now also U10.4, U91.4
- net ~{MFLCPA1}: now reaches U129.11
- net ~{MFLCPA1}: now also U113.10
- net MFLC: now reaches U129.12
- net MFLC: now also U130.12
- net IR911: now reaches U129.13
- net MPEM: now reaches U22.8
- net ~{MPEM}: now reaches U22.9
- net ~{MPEM}: now also U13.8, U154.1
- net ~{AEUZ6}: now reaches U109.11
- net ~{AEUZ6}: now also U88.7 (6)
- net AR0XAR1: now reaches U63.8
- net DBLQ: now reaches U101.5 (Q)
- net DBLQ: now also U99.12
- net ~{DBLQ}: now reaches U101.6 (~{Q})
- net M3L567J1: now reaches U108.10
- net M0J1: now reaches U108.3
- net M0J1: now also U136.6
- net ~{ST5T}: now reaches U109.2
- net M0L0J3: now reaches U121.12
- net ST56: now reaches U121.2
- net ST56: now also U85.11
- net ~{AR0XAR2}: now reaches U97.1
- net ~{MBLDPA}: now reaches U97.12
- net ~{MBLDPA}: now also U111.13
- net ~{M5L2PA}: now reaches U134.12
- net L2: now reaches U134.13
- net L2: now also U116.11, U121.10, U131.5, U134.11
- net ~{A0XA1}: now reaches U134.2
- net ~{IR12T}: now reaches U112.10
- net ~{IR12T}: now also U123.12
- net ~{MALDJ1}: now reaches U112.8
- net ~{MALDJ1}: now also U97.11
- net ENTERMFF: now reaches U12.12 (D)
- net ENTERMFF: now also U105.6
- net ~{TERM}: now reaches U12.8 (~{Q})
- net L8F: now reaches U135.1
- net ~{AEUZ0}: now reaches U88.1 (0)
- net ~{AEUZ8}: now reaches U88.10 (8)
- net ~{AEUZ9}: now reaches U88.11 (9)
- net ~{AEUZ1}: now reaches U88.2 (1)
- net ~{AEUZ1}: now also U73.9
- net ~{AEUZ2}: now reaches U88.3 (2)
- net ~{AEUZ2}: now also U85.4
- net ~{AEUZ3}: now reaches U88.4 (3)
- net ~{AEUZ4}: now reaches U88.5 (4)
- net ~{AEUZ4}: now also U73.10
- net ~{AEUZ5}: now reaches U88.6 (5)
- net ~{AEUZ7}: now reaches U88.9 (7)
- net ~{AEUZ7}: now also U85.5
- net ~{MALBJ1}: now reaches U73.6
- net ~{MALBJ1}: now also U97.9
- net DMAQ: now reaches U86.11
- net ~{DMAM}: now reaches U86.8
- net ~{MEM12}: now reaches U103.6 (D3)
- net ~{MEM12}: now also U24.4
- net LC: now reaches U100.11
- net LC: now also U107.13, U111.11, U113.1, U87.13
- net ~{MALCJ2}: now reaches U100.8
- net ~{MALCJ2}: now also U99.4
- net ~{MEM8}: now reaches U100.9
- net ~{MEM8}: now also U10.6, U87.9
- net AEUZ14: now reaches U73.8
- net AEUZ14: now also U72.3
- net ~{MALDJ2}: now reaches U97.6
- net ~{MALDJ2}: now also U99.5
- net AR1XIR9: now reaches U107.2
- net AR1XIR9: now also U109.3
- net ~{MALEFJ3}: now reaches U107.6
- net ~{MALEFJ3}: now also U66.3
- net ~{IR7T}: now reaches U93.4
- net SELPAA: now reaches U132.13
- net M8L3PA1: now reaches U110.8
- net ~{DBLEXTF}: now reaches U99.11
- net ~{DBLEXTF}: now also U111.4
- net E14XE15: now reaches U63.6
- net E14XE15: now also U123.3
- net ~{IR5T}: now reaches U134.3
- net ~{IR5T}: now also U136.10, U66.12
- net ~{M0L7OP}: now reaches U134.6
- net ~{M0L7OP}: now also U112.4
- net ~{MALDRDYQ}: now reaches U72.8
- net ~{MCLDJ1}: now reaches U99.8
- net ST01: now reaches U99.9
- net ~{ST0T}: now reaches U123.8
- net L8A: now reaches U129.1
- net ~{SCNT06}: now reaches U129.2
- net ~{SCNT06}: now also U66.2
- net ~{MAL8AA}: now reaches U129.3
- net ENGOFF: now reaches U90.2 (D)
- net ENGOFF: now also U105.8
- net GO: now reaches U90.5 (Q)
- net GO: now also U93.9
- net ~{GO}: now reaches U90.6 (~{Q})
- net ~{MAL8APA}: now reaches U115.3
- net MAL8DFPA: now reaches U115.6
- net MAL8DFPA: now also U119.4
- net ~{MEM12A}: now reaches U109.8
- net ~{MEM12A}: now also U87.10
- net ~{SC3}: now reaches U93.2
- net ~{AR14XIR9}: now reaches U109.6
- net ~{M0L7J1}: now reaches U136.1
- net ~{M0LEJ1}: now reaches U136.2
- net ~{M0LBJ1}: now reaches U136.5
- net L23: now reaches U135.2
- net SPLIMM: now reaches U130.1
- net SPLIMM: now also U117.2
- net IMM: now reaches U130.2
- net BFR1: now reaches U130.3
- net BFR1: now also R17.2, U161.3
- net ~{IR9T}: now reaches U130.13
- net ~{MBL6CJ3}: now reaches U107.8
- net ~{MALCPA1}: now reaches U99.1
- net ~{MALDPA1}: now reaches U99.2
- net ~{MALDPA1}: now also U100.12
- net MAPA1: now reaches U99.3
- net MAPA1: now also U98.2
- net M8LB: now reaches U138.1
- net at U138.2: no longer names the net of U138.2
- net ~{UR0T}: now reaches U138.5
- net ~{UR0T}: now also U138.10
- net ~{ST2T}: now reaches U138.12
- net ~{ST2T}: now also U123.10, U153.4
- net ~{AEQ7}: now reaches U72.4
- net ~{IAQ}: now reaches U22.10
- net ~{IAQ}: now also U13.1
- net ~{BFR0}: now reaches U118.10
- net CFZ: now reaches U118.13
- net L2467: now reaches U105.5
- net MFM0PA1: now reaches U113.8
- net SCNT1E: now reaches U116.6
- net ~{MEM6}: now reaches U28.5
- net ~{MEM6}: now also U91.1
- net MEM6A: now reaches U28.6
- net ~{MEM10}: now reaches U10.10
- net ~{MEM10}: now also U91.5
- net R66: now reaches U95.11
- net R66: now also U106.5, R66.2, U145.10 (D2)
- net R70: now reaches U95.13
- net R70: now also U95.5, R70.2, U155.10 (D2)
- net R62: now reaches U95.2
- net R62: now also U157.10 (D2)
- net $00001227: now reaches U95.9
- net $00001227: now also U159.8, U163.10, U163.8, U163.9
- net ~{M0L56AOP}: now reaches U112.1
- net ~{M0L56AOP}: now also U137.12
- net ~{M0L8OP}: now reaches U112.5
- net ~{M0L8OP}: now also U111.6
- net M0OP: now reaches U112.6
- net ~{MALE}: now reaches U13.2
- net ~{MALE}: now also U73.3
- net ~{MALCJ1}: now reaches U87.8
- net ~{MALCJ1}: now also U97.10
- net ~{RM}: now reaches U122.1 (S)
- net ~{RM}: now also U156.8
- net SELOPRM6: now reaches U122.12 (Zd)
- net SELOPRM6: now also U158.3
- net SELOPRM4: now reaches U122.4 (Za)
- net SELOPRM4: now also U159.13
- net SELOPRM5: now reaches U122.7 (Zb)
- net SELOPRM5: now also U159.6
- net SELOPRM7: now reaches U122.9 (Zc)
- net SELOPRM7: now also U158.6
- net ~{M8LCPA}: now reaches U111.8
- net ~{AP14XIR9}: now reaches U111.9
- net ~{M3LCJ3}: now reaches U129.4
- net ~{M3LCJ3}: now also U113.3
- net ~{M3L1J3}: now reaches U129.5
- net ~{M3L1J3}: now also U113.6
- net M3L1CJ3: now reaches U129.6
- net ~{AR15T}: now reaches U123.2
- net ~{AR15T}: now also U153.10
- net MBl2J2: now reaches U116.8
- net SC3B: now reaches U116.9
- net SC3B: now also U131.3
- net MBL025J1: now reaches U131.8
- net MBL025J1: now also U102.10
- net OPB: now reaches U33.6
- net R68: now reaches U94.11
- net R68: now also R68.2, U144.5, U145.12 (D0)
- net R72: now reaches U94.13
- net R72: now also U94.5, R72.2, U155.12 (D0)
- net R64: now reaches U94.2
- net R64: now also U157.12 (D0)
- net $00001217: now reaches U94.9
- net $00001217: now also U158.8, U161.8, U164.10, U164.8
- net ~{ER14T}: now reaches U134.10
- net ~{ER14T}: now also U123.6
- net ~{M8L2PA}: now reaches U134.8
- net IR56BSD: now reaches U111.3
- net ~{IR56BSD}: now reaches U137.8
- net MDPA1: now reaches U98.11
- net MBL3PA1: now reaches U98.13
- net MEM0PA1: now reaches U98.4
- net MALEFJ3: now reaches U66.4
- net L56: now reaches U110.1
- net M8L5J1: now reaches U110.12
- net MCL4PA: now reaches U119.11
- net MBPA: now reaches U119.13
- net MBPA: now also U111.12
- net MEL3PA: now reaches U119.2
- net MEL3PA: now also U5.11
- net A0XA1: now reaches U63.11
- net AEUZ27: now reaches U86.4
- net AEUZ27: now also U85.6
- net ~{M8LEJ2}: now reaches U86.6
- net ST5T: now reaches U113.2
- net MAJ1: now reaches U97.8
- net MAJ1: now also U102.1
- net IOINT: now reaches U90.12 (D)
- net MEM5A: now reaches U117.10
- net MCJ1: now reaches U102.12
- net MDJ1: now reaches U102.3
- net M67910: now reaches U91.6
- net ~{E14XE15}: now reaches U123.4
- net EXRCEQ: now reaches U8.13
- net SELBFR8: now reaches U104.10
- net FORALA: now reaches U104.8
- net CYCOMPA: now reaches U14.5
- net ~{CNT}: now reaches U85.8
- net ~{MAL0RDYQ}: now reaches U85.9
- net ~{MBLA8PA}: now reaches U111.1
- net ~{MBLCPA}: now reaches U111.2
- net R67: now reaches U96.11
- net R67: now also U140.5, U145.11 (D1)
- net R71: now reaches U96.13
- net R71: now also U96.5, R71.2, U155.11 (D1)
- net R63: now reaches U96.2
- net R63: now also U157.11 (D1)
- net $00001222: now reaches U96.9
- net $00001222: now also U158.9, U162.8, U162.9
- net R58: now reaches U106.11
- net R58: now also U106.13, U106.2, R58.2, U146.10 (D2)
- net $00001247: now reaches U106.9
- net $00001247: now also U152.10, U152.9, U159.9, U161.9
- net EXTFORMA: now reaches U87.1
- net EXTFORMA: now also U87.2, U87.4, U87.5
- net ESPQ renamed EXPQ
- new net $00001232: U147.9, U152.8, U159.10, U161.10, U162.10
- new net $00001237: U144.9, U148.8, U149.8, U158.10, U164.9
- new net $00001242: U140.9, U148.10, U148.9, U149.10, U150.9
- new net $00001251: U141.9, U149.9, U150.10, U150.8
- new net BFR0: R25.2, U150.6
- new net BFR2: R24.2, U150.3
- new net INTINT: U154.8
- new net M8L1: U153.12
- new net R57: R57.2, U141.11, U141.13, U141.2, U146.9 (D3)
- new net R59: R59.2, U140.11, U140.13, U140.2, U146.11 (D1)
- new net R60: R60.2, U144.11, U144.13, U144.2, U146.12 (D0)
- new net R61: R61.2, U147.2, U157.9 (D3)
- new net R65: R65.2, U141.5, U145.9 (D3), U147.11
- new net R69: U147.13, U147.5, U155.9 (D3)
- new net RAC0: U142.2 (Q0), U145.15 (A7), U146.15 (A7), U149.3, U150.13, U155.15 (A7), U157.15 (A7)
- new net RAC1: U142.7 (Q1), U145.1 (A6), U146.1 (A6), U152.13, U152.3, U155.1 (A6), U157.1 (A6)
- new net RAC2: U142.10 (Q2), U145.2 (A5), U146.2 (A5), U148.3, U149.13, U155.2 (A5), U157.2 (A5)
- new net RAC3: U142.15 (Q3), U145.3 (A4), U146.3 (A4), U148.6, U149.6, U155.3 (A4), U157.3 (A4)
- new net RAC4: U143.2 (Q0), U145.4 (A3), U146.4 (A3), U155.4 (A3), U157.4 (A3), U161.13, U165.1 (A4)
- new net RAC5: U143.7 (Q1), U163.3, U165.3 (A3)
- new net RAC5B: U145.7 (A2), U146.7 (A2), U155.7 (A2), U156.10, U157.7 (A2)
- new net RAC6: U143.10 (Q2), U145.6 (A1), U146.6 (A1), U155.6 (A1), U157.6 (A1), U162.3, U165.8 (A2)
- new net RAC7: U143.15 (Q3), U164.13, U165.10 (A1)
- new net RAC7B: U145.5 (A0), U146.5 (A0), U155.5 (A0), U156.2, U157.5 (A0)
- new net RAINC4: U162.13, U165.15 (S4)
- new net RAINC5: U163.13, U165.2 (S3)
- new net RAINC6: U162.6, U165.6 (S2)
- new net RAINC7: U161.6, U165.9 (S1)
- new net SELBFRC: U156.4
- new net SELPOP: U158.12, U158.2, U158.5, U159.12, U159.2, U159.5
- new net ~{ALU0T}: U153.1
- new net ~{ILOPQ}: U154.5
- new net ~{RAC0}: J2.9 (Pin_9), U142.3 (~{Q0})
- new net ~{RAC1}: J2.10 (Pin_10), U142.6 (~{Q1})
- new net ~{RAC2}: J2.11 (Pin_11), U142.11 (~{Q2})
- new net ~{RAC3}: J2.12 (Pin_12), U142.14 (~{Q3})
- new net ~{RAC4}: J2.13 (Pin_13), U143.3 (~{Q0})
- new net ~{RAC5}: J2.14 (Pin_14), U143.6 (~{Q1}), U156.11
- new net ~{RAC6}: J2.15 (Pin_15), U143.11 (~{Q2})
- new net ~{RAC7}: J2.16 (Pin_16), U143.14 (~{Q3}), U156.1
- new net ~{SELBFR}: U151.9, U156.3
- new net ~{SELJ0}: U160.9
- new net ~{SELJ2}: U125.9
- no-connect marks 114 -> 151
Other:
- note added: "1 16"
- note added: "1 9"
- note added: "13"
- note added: "16"
- note added: "2 10"
- note added: "2 15"
- note added: "3 11"
- note added: "3 14"
- note added: "4 12"
- note added: "4 13"
- note added: "5 12"
- note added: "5 13"
- note added: "6 11"
- note added: "6 14"
- note added: "7 10"
- note added: "7 15"
- note added: "8"
- note added: "8 16"
- note added: "8 9"
- note added: "DMAREC CB To XA11 P1 Pin 73 To XA07(AU1) P1 Pin 69"
- note added: "LSB11 Resets the Highest Priority EXP. Interrupt"
- note added: "Masked Memory Parity Error Interrupt"
- note added: "Masked Optional Expanded Interrupt"
- note added: "Passives Located at AU1 Column 2 Row 02"
- note added: "Synchronized DMA Interrupt Reconized Signal"
- title: (none) -> Arithmetic Unit #1
- moved on the sheet: CTP1, CTP2, J1, R22, XA7-P1, XA7-P2

Commit message: Added IO Interface Card
P2 needs to be finished for its proper pinout
Parts:
- removed U91: 7420N, symbol 74xx:74LS20
- added R21, R28, R32, R35, R36, R38, R39, R40, R41, R42, R43, R44, R46, R47, R48, R62, R63, R64, R67, R69: R, symbol Device:R
- added R33, R34, R37, R45: ~, symbol Device:R
- added U166, U172: 74H30N, symbol 74xx:74LS30
- added U167: 74H11N, symbol 74xx:74LS11
- added U168, U171, U178: 7402N, symbol 74xx:7402
- added U169: 74H103N, symbol TI980A:74H103N
- added U170: 7400N, symbol 74xx:7400
- added U173, U174: 74187, Package_DIP:DIP-16_W7.62mm, symbol TI980A:74187
- added U175: 74S03N, symbol 74xx:74LS03
- added U176: 7404N, symbol 74xx:74LS04
- added U177, U184: 7420N, symbol 74xx:74LS20
- added U179: 74154, symbol 74xx_IEEE:74154
- added U180: 7430N, symbol 74xx:74LS30
- added U181: 7474N, symbol 74xx:74LS74
- added U182: 74S04N, symbol 74xx:74LS04
- added U183: 74H51N, symbol TI980A:7451N
- added U91: 74S10N, symbol 74xx:74LS10
Connections:
- net ADRV: now also U170.1
- net BFR0: now also U173.9 (D3)
- net BFR1: now also U173.10 (D2)
- net BFR2: now also U173.11 (D1)
- net BFR3: now also U173.12 (D0)
- net BFR4: now also U174.9 (D3)
- net BFR5: now also U174.10 (D2)
- net BFR6: now also R36.2, U174.11 (D1)
- net BFR7: now also U174.12 (D0)
- net BKFFK: now also U169.3 (K)
- net BKPTJ: now also U169.14 (J)
- net BKPTQ: now also U169.12 (Q)
- net ENAR16LD: now also U168.13
- net ENPCOUT: now also U170.8
- net GCLKE:1: now also U169.1 (CLK), U169.5 (CLK)
- net GND: now also U173.8 (GND), U174.8 (GND)
- net ILLOP: now also U173.14 (~{CE2}), U174.14 (~{CE2})
- net INT: now also U166.8, U170.4
- net IOQ: now also U90.9 (Q)
- net L1: now also U177.5
- net L8: now also U177.13
- net M5L8: now also U170.12
- net M67910: now also U70.6
- net M8L1: now also U171.13, U175.10
- net M8LA: now also U168.1
- net M8LE: now also U168.4
- net MAL4: now also U168.10
- net MCL6: now also U171.1
- net MEM5A: now also U173.2 (A5), U174.2 (A5)
- net MEM6A: now also U173.3 (A4), U174.3 (A4)
- net MEM7A: now also U173.4 (A3), U174.4 (A3)
- net MEM9A: now also U173.6 (A1), U174.6 (A1)
- net OPA: now also U173.15 (A7), U174.15 (A7)
- net OPB: now also U173.1 (A6), U174.1 (A6)
- net R22: now also R22.2, U27.3 (K)
- net R62: now also R62.2
- net R63: now also R63.2
- net R64: now also R64.2
- net R67: now also R67.2
- net R69: now also R69.2
- net RSTRUN: now also U169.10 (K)
- net RUNFFQ: now also U169.9 (Q)
- net SETRUN: now also U169.7 (J)
- net SR16: now also U170.13
- net VCC1: now also R21.1, R28.1, R32.1, R33.1, R34.1, R35.1, R36.1, R37.1, R38.1, R39.1, R40.1, R41.1, R42.1, R43.1, R44.1, R45.1, R46.1, R47.1, R48.1, R62.1, R63.1, R64.1, R67.1, R69.1, U166.12, U169.6 (~{R}), U172.12, U173.16 (VCC), U174.16 (VCC)
- net ~{ARDSW}: now also R41.2
- net ~{ARESW}: now also R43.2
- net ~{BKPTQ}: now also U169.13 (~{Q})
- net ~{BRESW}: now also R46.2
- net ~{BYTFLAG}: now also U170.2
- net ~{DEVTHERE}: now also R28.2, U175.5
- net ~{DMAM}: now also U166.2
- net ~{EN00}: now also U167.10, U170.3
- net ~{EXPINT}: now also R44.2
- net ~{EXPM}: now also U166.1
- net ~{FORCE00}: now also U167.8
- net ~{IAQBFR}: now also U167.13, U170.9
- net ~{IFLAGQ}: now also U170.5
- net ~{INHMUA1}: now also U170.11
- net ~{INSTV}: now also U167.11
- net ~{INTM}: now also U170.6
- net ~{IOM}: now also U166.3
- net ~{IOQ}: now also U90.8 (~{Q})
- net ~{L1}: now also U171.12
- net ~{L3}: now also U171.6
- net ~{L4}: now also U168.9
- net ~{L6}: now also U168.12, U171.3
- net ~{LA}: now also U168.3
- net ~{LDBTSW}: now also U177.4
- net ~{LE}: now also U168.6
- net ~{LF}: now also U171.9
- net ~{M0L4BFR}: now also U167.1
- net ~{M8}: now also U168.2, U168.5, U171.11
- net ~{MADSW}: now also U177.10
- net ~{MAESW}: now also U177.12
- net ~{MALEBFR}: now also U167.2, U170.10
- net ~{MA}: now also U168.8
- net ~{MC}: now also U168.11, U171.2, U171.5
- net ~{MDESW}: now also R48.2
- net ~{MDIDSW}: now also R38.2
- net ~{MDIESW}: now also R39.2
- net ~{MEM10}: now also U70.5
- net ~{MEM6}: now also U70.1
- net ~{MEM7}: now also U70.2
- net ~{MEM9}: now also U70.4
- net ~{MPEM}: now also U166.4
- net ~{MRDSW}: now also R37.2
- net ~{MRESETQA}: now also U169.2 (~{R})
- net ~{MRESETQ}: now also U167.9
- net ~{PCESW}: now also R42.2
- net ~{RSTSW}: now also U177.2
- net ~{RUNFFQ}: now also U169.8 (~{Q}), U177.1
- net ~{RUNSW}: now also R47.2
- net ~{SELBFR}: now also U167.12, U172.11
- net ~{SELJ0}: now also U172.8
- net ~{SELJ1}: now also U172.1
- net ~{SELJ2A}: now also U71.1
- net ~{SELJ2}: now also U71.12, U172.2
- net ~{SELJ3}: now also U172.3, U175.6, U175.8
- net ~{SELOP}: now also U172.6
- net ~{SELPA1}: now also U172.5
- net ~{SELPA}: now also R33.2, U172.4
- net ~{SIESW}: now also R40.2
- net ~{SPLIMM}: now also R34.2
- net ~{ST5}: now also U166.6
- net ~{ST6}: now also U166.11
- net ~{STDSW}: now also R45.2
- net ~{STESW}: now also R21.2
- net ~{SELJ2C}: now reaches U71.13
- net ~{SELJ2B}: now reaches U71.2
- new net ALUEQ8K: U175.9
- new net EXRECD: U167.6
- new net ILLOPA: U173.13 (~{CE1}), U174.13 (~{CE1})
- new net MCL3: U171.4, U175.4
- new net MEM10A: U173.5 (A0), U174.5 (A0)
- new net MEM8A: U173.7 (A2), U174.7 (A2)
- new net MFLF: U167.3, U171.10
- new net ~{INTRTOPA}: R35.2
- new net ~{MDL1PA1}: U177.6
- new net ~{MDL8PA1}: U177.8
- new net ~{MF}: U171.8
- new net ~{ST16}: U166.5
- new net ~{T2OR6}: U167.5
- new net ~{T4OR6}: U167.4
- new net ~{XRDSW}: R32.2, U177.9
- no-connect marks 151 -> 161
Other:
- moved on the sheet: R22
