File: TI980A-Arithmetic-Unit/AU1.kicad_sch (KiCad schematic)
At the start: 292 parts, among them J1 Circuit Type Test, J2 Circuit Type Test, U1 7413N, U10 74H04N, U100 7410N, U101 7474N, U102 74H52N, U103 74163, U104 7408N, U105 74H11N, U106 74H52N, U107 7451N, U108 74H52N, U109 7404N, U11 74H04N, U110 74H11N, U111 7410N, U112 7420N, U113 7400N, U114 74H54W, U115 7410N, U116 74H11N, U117 74H04N, U118 74H21N, U119 74H52N, U12 74LS74, U120 74188N, U121 74H11N, U122 74157N, U123 7404N, U124 74H11N, U125 74H51N, U126 74H01N, U127 7410N, U128 7474N, U129 7400N, U13 74H00N, U130 74H01N, U131 74H52N, U132 74H05N, U133 74H22N, U134 7410N, U135 7451N, U136 7420N, U137 7427N, U138 74S22N, U139 74S65N, U14 74H10, U140 74H52N, U141 74H52N, U142 74175N, U143 74175N, U144 74H52N, U145 74187, U146 74187, U147 74H52N, U148 74H61N, U149 74H61N, U150 74H61N, U151 7451N, U152 74H61N, U153 74S22N, U155 74187, U156 74H04N, U157 74187, U158 74H61N, U159 74H61N, U160 7451N, U161 74H61N, U162 74H61N, U163 74H61N, U164 74H61N, U165 74LS83, U167 74H11N, U171 7402N, U172 74H30N, U173 74187, U174 74187, U175 74S03N, U176 7404N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

Commit message: All Register Except Status Register Done
Other:
- note added: "A Register Control [AR]"
- note added: "ALU Function Selects on AU1"
- note added: "AU1 Clocks"
- note added: "B Register Control"
- note added: "Console Control Enable Signals Derived From the Lock Switch"
- note added: "Data Bus A Select Logic on AU1"
- note added: "E Register Control AU1 Part"
- note added: "Instruction Register Controlon AU1"
- note added: "Memory Address Register Control AU1 Part"
- note added: "PFAIL"
- note added: "Part of ALU S2 Select Input"
- note added: "Program Counter Control Logic on AU1"
- note removed: "A Register [AR]"
- note removed: "ALU Function Selects on AU1 Part of ALU S2 Select Input"
- note removed: "B Register and Control"
- note removed: "Console Control Enable Signals Derrived From the Lock Switch"
- note removed: "E Register and Controls AU1 Part"
- note removed: "Memory Address Register and Control AU1 Part"
- note removed: "Part of Data Bus A Select Logic on AU1"
- note removed: "Part of Instruction Register Circuit on AU1"
- note removed: "Program Counter (PC) and Control Logic on AU1"

Commit message: Added IO Card Images and Fixed Error on AU1
Connections:
- net $00001222: now also U52.9
- net TRP1413: no longer U52.12
Changed lines of the file:
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@@
 	)
 	(junction
+		(at 746.76 168.91)
+		(diameter 0)
+		(color 0 0 0 0)
+	)
+	(junction
 		(at 877.57 274.32)
 		(diameter 0)
@@
 	)
 	(junction
-		(at 52.07 723.9)
-		(diameter 0)
-		(color 0 0 0 0)
-	)
-	(junction
 		(at 59.69 33.02)
 		(diameter 0)
@@
 	(wire
 		(pts
-			(xy 41.91 723.9) (xy 52.07 723.9)
-		)
-		(stroke
-			(width 0)
-			(type default)
-		)
-	)
-	(wire
-		(pts
 			(xy 642.62 556.26) (xy 670.56 556.26)
 		)
@@
 	(wire
 		(pts
-			(xy 19.05 726.44) (xy 26.67 726.44)
+			(xy 712.47 185.42) (xy 720.09 185.42)
 		)
 		(stroke
@@
 	(wire
 		(pts
+			(xy 746.76 168.91) (xy 746.76 182.88)
+		)
+		(stroke
+			(width 0)
+			(type default)
+		)
+	)
+	(wire
+		(pts
 			(xy 233.68 99.06) (xy 233.68 102.87)
 		)
@@
 	(wire
 		(pts
-			(xy 19.05 723.9) (xy 26.67 723.9)
+			(xy 712.47 182.88) (xy 720.09 182.88)
 		)
 		(stroke
@@
 	(wire
 		(pts
+			(xy 735.33 182.88) (xy 746.76 182.88)
+		)
+		(stroke
+			(width 0)
+			(type default)
+		)
+	)
+	(wire
+		(pts
 			(xy 633.73 415.29) (xy 641.35 415.29)
 		)
@@
 	)
 	(label "BFR6"
-		(at 19.05 726.44 0)
+		(at 712.47 185.42 0)
 		(effects
 			(font
@@
 		)
 	)
-	(label "TRP1413"
-		(at 52.07 723.9 180)
+	(label "$00001222"
+		(at 746.76 182.88 180)
 		(effects
 			(font
@@
 	)
 	(label "SELBFR"
-		(at 19.05 723.9 0)
+		(at 712.47 182.88 0)
 		(effects
 			(font
@@
 	)
 	(symbol
+		(lib_name "74H61N_4")
 		(lib_id "TI980A:74H61N")
 		(at 67.31 708.66 0)
@@
 		(pin "8"
 		)
-		(pin "12"
+		(pin "9"
 		)
 		(pin "5"
@@
 	(symbol
 		(lib_id "power:VCC")
-		(at 26.67 721.36 90)
+		(at 720.09 180.34 90)
 		(unit 1)
 		(body_style 1)
@@
 		(fields_autoplaced yes)
 		(property "Reference" "#PWR0345"
-			(at 30.48 721.36 0)
+			(at 723.9 180.34 0)
 			(hide yes)
 			(show_name no)
@@
 		)
 		(property "Value" "VCC1"
-			(at 22.86 721.3599 90)
+			(at 716.28 180.3399 90)
 			(show_name no)
 			(do_not_autoplace no)
@@
 		)
 		(property "Footprint" ""
-			(at 26.67 721.36 0)
+			(at 720.09 180.34 0)
 			(hide yes)
 			(show_name no)
@@
 		)
 		(property "Datasheet" ""
-			(at 26.67 721.36 0)
+			(at 720.09 180.34 0)
 			(hide yes)
 			(show_name no)
@@
 		)
 		(property "Description" "Power symbol creates a global label with name \"VCC\""
-			(at 26.67 721.36 0)
+			(at 720.09 180.34 0)
 			(hide yes)
 			(show_name no)
@@
 	)
 	(symbol
+		(lib_name "74H61N_5")
 		(lib_id "TI980A:74H61N")
-		(at 34.29 723.9 0)
+		(at 727.71 182.88 0)
 		(unit 1)
 		(body_style 1)
@@
 		(dnp no)
 		(property "Reference" "U52"
-			(at 34.7345 715.01 0)
+			(at 728.1545 173.99 0)
 			(hide yes)
 			(show_name no)
@@
 		)
 		(property "Value" "74H61N"
-			(at 34.7345 717.55 0)
+			(at 728.1545 176.53 0)
 			(show_name no)
 			(do_not_autoplace no)
@@
 		)
 		(property "Footprint" "Package_DIP:DIP-14_W7.62mm"
-			(at 34.29 723.646 0)
+			(at 727.71 182.626 0)
 			(hide yes)
 			(show_name no)
@@
 		)
 		(property "Datasheet" ""
-			(at 34.29 723.9 0)
+			(at 727.71 182.88 0)
 			(hide yes)
 			(show_name no)
@@
 		)
 		(property "Description" "Tripple 3-Input Expanders"
-			(at 34.29 723.646 0)
+			(at 727.71 182.626 0)
 			(hide yes)
 			(show_name no)
@@
 		)
 		(property "Location" "AU1 Column 7 Row 09"
-			(at 34.29 715.01 0)
+			(at 727.71 173.99 0)
 			(show_name no)
 			(do_not_autoplace no)
@@
 		(pin "8"
 		)
-		(pin "12"
+		(pin "9"
 		)
 		(pin "5"
@@
 	)
 	(symbol
+		(lib_name "74H61N_3")
 		(lib_id "TI980A:74H61N")
 		(at 66.04 745.49 0)
@@
 		(pin "8"
 		)
-		(pin "12"
+		(pin "9"
 		)
 		(pin "5"
