File: TI980A-Arithmetic-Unit/TI980A-Arithmetic-Unit.kicad_sch (KiCad schematic)
At the start: 0 parts

Commit message: Finished Columns 1, 2, 3, 10, 11, 12, 13, and 14
Other:
- company: (none) -> Texas Instruments
- title: (none) -> 960713-9901
Changed lines of the file:
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@@
 	(generator_version "9.0")
 	(paper "A4")
+	(title_block
+		(title "960713-9901")
+		(company "Texas Instruments")
+		(comment 1 "TI980A Arithmetic Unit")
+		(comment 2 "Derived from Maintenance Manual VIII & IX")
+	)
 	(sheet
 		(at 153.035 63.5)
