File: TI980A-Arithmetic-Unit/AU2.kicad_sch (KiCad schematic)
At the start: 15 parts, among them U15 74H40N, U16 74H40N, U17 74H40N, U18 74H11N, U19 74H04N, U20 74H40N, U38 74H21N, U39 7485, U40 7485, U41 7485, U42 7485

Commit message: Finished Up to Column 3 on AU2
Parts:
- added R100, R101, R102, R103, R104, R105, R106, R107, R108, R109, R110, R111, R112, R113, R114, R115, R116, R117, R118, R119, R120, R121, R122, R123, R124, R125, R126, R127, R128, R129, R130, R131, R14, R40, R81, R82, R83, R84, R85, R86, R87, R88, R89, R90, R91, R92, R93, R94, R95, R96, R97, R98, R99: R, symbol Device:R
- added U231, U253: 7451N, symbol TI980A:7451N
- added U232: 74H101, Package_DIP:DIP-14_W7.62mm, symbol TI980A:74H101
- added U233, U234, U235, U236, U238, U239, U240, U241, U242, U248, U249, U250, U251, U252: 74187, Package_DIP:DIP-16_W7.62mm, symbol TI980A:74187
- added U237, U265: 74H04N, symbol 74xx:74LS04
- added U243, U244: 7430N, symbol 74xx:74LS30
- added U245, U263, U272: 74H11N, symbol 74xx:74LS11
- added U246, U256: 74H00N, symbol 74xx:7400
- added U247, U257, U258, U259, U264: 74H74N, symbol 74xx:74LS74
- added U254: 74LS37, symbol 74xx:74LS37
- added U255: 74S65N, symbol TI980A:74S65N
- added U260: 7410N, symbol 74xx:74LS10
- added U261: 7420N, symbol 74xx:74LS20
- added U262: 74H21N, symbol 74xx:74LS21
- added U266, U270, U271: 74LS153, symbol 74xx:74LS153
- added U267: 74H20N, symbol 74xx:74LS20
- added U268: 7474N, symbol 74xx:74LS74
- added U269: 74LS181, symbol 74xx:74LS181
- added U273: 74174N, symbol 74xx:74LS174
- added U274: 74S10N, symbol 74xx:74LS10
- U19: Location AU2 Column 4 Row 04 -> AU2 Column 5 Row 04
Connections:
- net A0: now also U269.19 (A3)
- net AR16: now also U232.6 (Q)
- net BYTEINC: now also U232.11 (K2A), U232.12 (K2B), U232.3 (J2A), U232.4 (J2B)
- net ENAR16LD: now also U232.1 (J1A), U232.9 (K1A)
- net ER0: now also U264.9 (Q), U266.12 (I2b)
- net ER1: now also U266.11 (I1b)
- net GCLKB:1: now also U232.13 (CLK)
- net GND: now also U232.7 (GND), U233.13 (~{CE1}), U233.14 (~{CE2}), U233.8 (GND), U234.13 (~{CE1}), U234.14 (~{CE2}), U234.8 (GND), U235.13 (~{CE1}), U235.14 (~{CE2}), U235.8 (GND), U236.13 (~{CE1}), U236.14 (~{CE2}), U236.8 (GND), U238.13 (~{CE1}), U238.14 (~{CE2}), U238.8 (GND), U239.13 (~{CE1}), U239.14 (~{CE2}), U239.8 (GND), U240.13 (~{CE1}), U240.14 (~{CE2}), U240.8 (GND), U241.13 (~{CE1}), U241.14 (~{CE2}), U241.8 (GND), U242.13 (~{CE1}), U242.14 (~{CE2}), U242.8 (GND), U248.13 (~{CE1}), U248.14 (~{CE2}), U248.8 (GND), U249.13 (~{CE1}), U249.14 (~{CE2}), U249.8 (GND), U250.13 (~{CE1}), U250.14 (~{CE2}), U250.8 (GND), U251.13 (~{CE1}), U251.14 (~{CE2}), U251.8 (GND), U252.13 (~{CE1}), U252.14 (~{CE2}), U252.8 (GND), U266.1 (Ea), U266.10 (I0b), U266.13 (I3b), U266.15 (Eb), U266.5 (I1a), U266.8 (GND), U269.12 (GND), U270.8 (GND), U271.8 (GND), U273.8 (GND)
- net IFLAGQ: now also U19.9
- net INAQ: now also U256.10
- net M3: now also U231.9
- net MAR0: now also U271.6 (I0a)
- net MAR1: now also U271.10 (I0b)
- net MAR2: now also U270.6 (I0a)
- net MAR3: now also U270.10 (I0b)
- net NRA0: now also U257.12 (D)
- net NRA1: now also U259.12 (D)
- net NRA2: now also U258.12 (D)
- net NRA3: now also U257.2 (D)
- net NRA4: now also U258.2 (D)
- net NRA5: now also U259.2 (D)
- net NRA6: now also U247.12 (D)
- net NRA7: now also U247.2 (D)
- net PNL0: now also XA8-P2.11 (Pin_11), R123.2
- net PNL1: now also XA8-P2.14 (Pin_14), R130.2
- net PNL10: now also XA8-P2.72 (Pin_72)
- net PNL12: now also XA8-P1.36 (Pin_36)
- net PNL13: now also XA8-P2.70 (Pin_70)
- net PNL14: now also XA8-P1.47 (Pin_47)
- net PNL15: now also XA8-P2.66 (Pin_66)
- net PNL2: now also XA8-P2.13 (Pin_13), R128.2
- net PNL3: now also XA8-P2.19 (Pin_19), R121.2
- net PNL4: now also XA8-P2.42 (Pin_42)
- net PNL5: now also XA8-P2.44 (Pin_44)
- net PNL6: now also XA8-P2.45 (Pin_45)
- net PNL7: now also XA8-P2.48 (Pin_48)
- net PNL8: now also XA8-P2.65 (Pin_65)
- net PNL9: now also XA8-P2.68 (Pin_68)
- net R22: now also U251.10 (D2)
- net R39: now also U241.11 (D1)
- net UR0: now also U271.5 (I1a)
- net VCC1: now also R100.1, R101.1, R102.1, R103.1, R104.1, R105.1, R106.1, R107.1, R108.1, R109.1, R110.1, R111.1, R112.1, R113.1, R114.1, R115.1, R116.1, R117.1, R118.1, R119.1, R120.1, R121.1, R122.1, R123.1, R124.1, R125.1, R126.1, R127.1, R128.1, R129.1, R130.1, R131.1, R14.1, R40.1, R81.1, R82.1, R83.1, R84.1, R85.1, R86.1, R87.1, R88.1, R89.1, R90.1, R91.1, R92.1, R93.1, R94.1, R95.1, R96.1, R97.1, R98.1, R99.1, U232.14 (VCC), U232.5 (Pre), U233.16 (VCC), U234.16 (VCC), U235.16 (VCC), U236.16 (VCC), U238.16 (VCC), U239.16 (VCC), U240.16 (VCC), U241.16 (VCC), U242.16 (VCC), U244.12, U247.1 (~{R}), U247.10 (~{S}), U247.13 (~{R}), U247.4 (~{S}), U248.16 (VCC), U249.16 (VCC), U250.16 (VCC), U251.16 (VCC), U252.16 (VCC), U253.13, U254.13, U254.2, U255.10, U255.11, U255.12, U255.13, U255.3, U255.5, U255.6, U257.1 (~{R}), U257.10 (~{S}), U257.13 (~{R}), U257.4 (~{S}), U258.1 (~{R}), U258.10 (~{S}), U258.13 (~{R}), U258.4 (~{S}), U259.1 (~{R}), U259.10 (~{S}), U259.13 (~{R}), U259.4 (~{S}), U264.1 (~{R}), U264.10 (~{S}), U264.13 (~{R}), U264.4 (~{S}), U266.16 (VCC), U268.1 (~{R}), U268.10 (~{S}), U268.13 (~{R}), U268.4 (~{S}), U269.24 (VCC), U270.16 (VCC), U271.16 (VCC), U273.1 (~{Mr}), U273.16 (VCC)
- net ~{GCLKC:1}: now also U268.3 (C)
- net ~{GCLKC:2}: now also U247.11 (C), U247.3 (C), U257.11 (C), U257.3 (C), U258.11 (C), U258.3 (C), U259.11 (C), U259.3 (C), U264.3 (C)
- net ~{GCLK}: now also XA8-P1.63 (Pin_63)
- net ~{R19}: now also U233.11 (D1)
- net ~{R36}: now also U248.12 (D0)
- net ~{R44}: now also U238.12 (D0)
- net ~{RUNFFQ}: now also U256.9
- net EXPADR9: now reaches XA8-P1.10 (Pin_10)
- net ~{DP11}: now reaches XA8-P1.11 (Pin_11)
- net ~{APIMALD}: now reaches XA8-P1.12 (Pin_12)
- net EXPADR10: now reaches XA8-P1.13 (Pin_13)
- net IOUT5: now reaches XA8-P1.14 (Pin_14)
- net EXPADR11: now reaches XA8-P1.15 (Pin_15)
- net IOUT7: now reaches XA8-P1.16 (Pin_16)
- net EXPADR12: now reaches XA8-P1.17 (Pin_17)
- net ~{DP6}: now reaches XA8-P1.18 (Pin_18)
- net ~{APIST0}: now reaches XA8-P1.19 (Pin_19)
- net ~{SNS1}: now reaches XA8-P1.20 (Pin_20)
- net EXPADR13: now reaches XA8-P1.21 (Pin_21)
- net IOUT6: now reaches XA8-P1.22 (Pin_22)
- net ~{DP15}: now reaches XA8-P1.23 (Pin_23)
- net IOUT3: now reaches XA8-P1.24 (Pin_24)
- net ~{DP12}: now reaches XA8-P1.25 (Pin_25)
- net MEM8: now reaches XA8-P1.26 (Pin_26)
- net ~{DP5}: now reaches XA8-P1.27 (Pin_27)
- net ~{SNS2}: now reaches XA8-P1.28 (Pin_28)
- net ~{DP14}: now reaches XA8-P1.29 (Pin_29)
- net MEM11: now reaches XA8-P1.30 (Pin_30)
- net ~{DP13}: now reaches XA8-P1.31 (Pin_31)
- net PML11: now reaches XA8-P1.32 (Pin_32)
- net MEM9: now reaches XA8-P1.33 (Pin_33)
- net MEM10: now reaches XA8-P1.34 (Pin_34)
- net ~{SNS3}: now reaches XA8-P1.35 (Pin_35)
- net MEM12: now reaches XA8-P1.37 (Pin_37)
- net MEM7: now reaches XA8-P1.38 (Pin_38)
- net MEM13: now reaches XA8-P1.39 (Pin_39)
- net ~{INSTV}: now reaches XA8-P1.40 (Pin_40)
- net MEM15: now reaches XA8-P1.41 (Pin_41)
- net ~{SNS4}: now reaches XA8-P1.42 (Pin_42)
- net MEM14: now reaches XA8-P1.43 (Pin_43)
- net EXPADR8: now reaches XA8-P1.44 (Pin_44)
- net MPERR: now reaches XA8-P1.45 (Pin_45)
- net ~{ADRV}: now reaches XA8-P1.46 (Pin_46)
- net MEM6: now reaches XA8-P1.48 (Pin_48)
- net ~{APIS2CK}: now reaches XA8-P1.49 (Pin_49)
- net ~{DP8}: now reaches XA8-P1.5 (Pin_5)
- net MEM2: now reaches XA8-P1.50 (Pin_50)
- net MEM2: now also U273.6 (D2)
- net ~{APIST2}: now reaches XA8-P1.51 (Pin_51)
- net ~{CPUCR}: now reaches XA8-P1.52 (Pin_52)
- net ~{APIST1}: now reaches XA8-P1.53 (Pin_53)
- net EXPADR14: now reaches XA8-P1.55 (Pin_55)
- net ~{APIS01CK}: now reaches XA8-P1.57 (Pin_57)
- net ~{DP7}: now reaches XA8-P1.6 (Pin_6)
- net IOUT15: now reaches XA8-P1.65 (Pin_65)
- net IOUT11: now reaches XA8-P1.66 (Pin_66)
- net IOUT12: now reaches XA8-P1.67 (Pin_67)
- net IOUT8: now reaches XA8-P1.68 (Pin_68)
- net IOUT14: now reaches XA8-P1.69 (Pin_69)
- net ~{DP9}: now reaches XA8-P1.7 (Pin_7)
- net IOUT10: now reaches XA8-P1.70 (Pin_70)
- net IOUT13: now reaches XA8-P1.71 (Pin_71)
- net IOUT9: now reaches XA8-P1.72 (Pin_72)
- net IOUT4: now reaches XA8-P1.8 (Pin_8)
- net ~{DP10}: now reaches XA8-P1.9 (Pin_9)
- net ~{IFLAG}: now reaches U19.8
- net ~{IFLAG}: now also U18.10
- net ~{R41}: now reaches U38.1
- net ~{R41}: now also R96.2, U238.9 (D3)
- net ~{ENSXR}: now reaches U38.2
- net ~{ENDXR}: now reaches U38.4
- net ~{LREENXR}: now reaches U38.5
- net ~{ENXRLOAD}: now reaches U38.6
- net ST4: now reaches U18.11
- net ST4: now also U268.9 (Q)
- net ST4G: now reaches U18.8
- net ST4G: now also XA8-P2.32 (Pin_32)
- net HLTINAQ: now reaches U18.9
- net HLTINAQ: now also U256.8
- net ~{ALU15}: now reaches U19.12
- net ALU15: now reaches U19.13
- net ALU15: now also U266.4 (I2a), U272.3
- net ~{ALU0}: now reaches U19.10
- net ~{ALU0}: now also U260.5
- net ALU0: now reaches U19.11
- net ALU0: now also U18.3, U266.6 (I0a), U269.13 (F3)
- net ~{API4}: now reaches XA8-P2.10 (Pin_10)
- net ~{API4}: now also U256.13
- net ~{API3}: now reaches XA8-P2.12 (Pin_12)
- net ~{API3}: now also U246.5
- net ~{API11}: now reaches XA8-P2.15 (Pin_15)
- net ~{API11}: now also U256.5
- net ~{API1}: now reaches XA8-P2.16 (Pin_16)
- net ~{API1}: now also U246.2
- net ~{DP4}: now reaches XA8-P2.17 (Pin_17)
- net ~{DP4}: now also R125.2
- net ~{API2}: now reaches XA8-P2.18 (Pin_18)
- net ~{API2}: now also U246.13
- net ALUB3: now reaches XA8-P2.20 (Pin_20)
- net ALUB3: now also U245.6
- net ~{API15}: now reaches XA8-P2.21 (Pin_21)
- net ~{API15}: now also U246.10
- net ALUB1: now reaches XA8-P2.22 (Pin_22)
- net ALUB1: now also U245.12
- net MEM5: now reaches XA8-P2.23 (Pin_23)
- net MEM5: now also U273.14 (D5)
- net MEM0: now reaches XA8-P2.24 (Pin_24)
- net MEM0: now also U273.3 (D0)
- net ALUB4: now reaches XA8-P2.25 (Pin_25)
- net ALUB4: now also U272.12
- net MEM1: now reaches XA8-P2.26 (Pin_26)
- net MEM1: now also U273.4 (D1)
- net MEM4: now reaches XA8-P2.27 (Pin_27)
- net MEM4: now also U273.13 (D4)
- net MEM3: now reaches XA8-P2.28 (Pin_28)
- net MEM3: now also U273.11 (D3)
- net ALUB11: now reaches XA8-P2.29 (Pin_29)
- net ALUB11: now also U272.8
- net ALUB0: now reaches XA8-P2.30 (Pin_30)
- net ALUB0: now also U18.6
- net ALUB15: now reaches XA8-P2.31 (Pin_31)
- net ALUB15: now also U272.6
- net ALUB2: now reaches XA8-P2.33 (Pin_33)
- net ALUB2: now also U245.8
- net ~{API14}: now reaches XA8-P2.34 (Pin_34)
- net ~{DP0}: now reaches XA8-P2.35 (Pin_35)
- net IOUT2: now reaches XA8-P2.36 (Pin_36)
- net ~{DP1}: now reaches XA8-P2.37 (Pin_37)
- net IOUT0: now reaches XA8-P2.38 (Pin_38)
- net ~{DP2}: now reaches XA8-P2.39 (Pin_39)
- net ~{DP3}: now reaches XA8-P2.40 (Pin_40)
- net ~{APISTORE}: now reaches XA8-P2.41 (Pin_41)
- net CPUSTR: now reaches XA8-P2.43 (Pin_43)
- net IOUT1: now reaches XA8-P2.46 (Pin_46)
- net ~{MALOAD}: now reaches XA8-P2.47 (Pin_47)
- net ENAPI: now reaches XA8-P2.49 (Pin_49)
- net ENAPI: now also U246.1, U246.12, U246.4, U246.9, U256.1, U256.12, U256.4
- net ~{API9}: now reaches XA8-P2.50 (Pin_50)
- net ~{API8}: now reaches XA8-P2.51 (Pin_51)
- net ~{API6}: now reaches XA8-P2.52 (Pin_52)
- net ~{API13}: now reaches XA8-P2.53 (Pin_53)
- net ALUB8: now reaches XA8-P2.54 (Pin_54)
- net ~{API12}: now reaches XA8-P2.55 (Pin_55)
- net ~{API5}: now reaches XA8-P2.56 (Pin_56)
- net ~{API10}: now reaches XA8-P2.57 (Pin_57)
- net ~{API7}: now reaches XA8-P2.58 (Pin_58)
- net ALUB6: now reaches XA8-P2.59 (Pin_59)
- net ST9G: now reaches XA8-P2.60 (Pin_60)
- net ALUB9: now reaches XA8-P2.61 (Pin_61)
- net ~{APICYCRQ}: now reaches XA8-P2.62 (Pin_62)
- net ALUB14: now reaches XA8-P2.63 (Pin_63)
- net ~{APIMAINC}: now reaches XA8-P2.64 (Pin_64)
- net ALUB5: now reaches XA8-P2.67 (Pin_67)
- net ALUB13: now reaches XA8-P2.69 (Pin_69)
- net ALUB10: now reaches XA8-P2.71 (Pin_71)
- net ALUB12: now reaches XA8-P2.73 (Pin_73)
- net ALUB7: now reaches XA8-P2.74 (Pin_74)
- net ~{ENMAINC}: now reaches XA8-P2.75 (Pin_75)
- net ~{API0}: now reaches XA8-P2.9 (Pin_9)
- net ~{API0}: now also U256.2
- net ENALUB: now reaches U18.4
- net ENALUB: now also U245.10, U245.2, U245.4, U272.10, U272.2, U272.4
- net API0: now reaches U18.5
- net API0: now also U256.3
- net ENARCLR renamed ~{ENARCLR}
- net MBLBC renamed M8LBC
- new net A1: U269.21 (A2)
- new net A2: U269.23 (A1)
- new net A3: U269.2 (A0)
- new net AEQB: R127.2, U269.14 (A=B)
- new net ALU1: U245.1, U255.2, U269.11 (F2)
- new net ALU11: U272.9
- new net ALU2: U245.9, U255.9, U269.10 (F1)
- new net ALU3: U245.3, U255.1, U269.9 (F0)
- new net ALU4: U255.4, U272.1
- new net ALUM: U269.8 (M)
- new net ALUS0: U269.6 (S0)
- new net ALUS1: U254.11, U269.5 (S1)
- new net ALUS2: U269.4 (S2)
- new net ALUS3: U254.3, U269.3 (S3)
- new net ALUZ115: R119.2, U255.8
- new net AOI15: U272.5
- new net API1: U245.13, U246.3
- new net API11: U256.6, U272.11
- new net API15: U246.8
- new net API2: U245.11, U246.11
- new net API3: U245.5, U246.6
- new net API4: U256.11, U272.13
- new net AXB0: U260.4
- new net B0: U269.18 (B3), U271.7 (Za)
- new net B1: U269.20 (B2), U271.9 (Zb)
- new net B2: U269.22 (B1), U270.7 (Za)
- new net B3: U269.1 (B0), U270.9 (Zb)
- new net BMAD1: U270.14 (S0), U271.14 (S0)
- new net ENERS0: U267.8
- new net ENLRLOAD: U261.8
- new net ENMPYOV: U265.8
- new net ENMRLOAD: U261.6
- new net ENRMLOV: U264.5 (Q)
- new net ER15: U232.2 (J1B), U266.3 (I3a)
- new net ERIN0: U264.12 (D)
- new net INHMSB: U270.1 (Ea), U270.15 (Eb), U271.1 (Ea), U271.15 (Eb)
- new net IR8A: U270.13 (I3b), U270.3 (I3a), U271.13 (I3b), U271.3 (I3a)
- new net LSC0: U265.6
- new net LSC15: U266.9 (Zb)
- new net MDR0: U271.4 (I2a), U273.2 (Q0)
- new net MDR1: U271.12 (I2b), U273.5 (Q1)
- new net MDR2: U270.4 (I2a), U273.7 (Q2)
- new net MDR3: U270.12 (I2b), U273.10 (Q3)
- new net MDR4: U273.12 (Q4)
- new net MDR5: U273.15 (Q5)
- new net NSC0: U265.4
- new net R1: R87.2, U249.9 (D3)
- new net R14: R104.2, U239.10 (D2), U266.2 (S1)
- new net R15: R110.2, U239.11 (D1), U266.14 (S0)
- new net R20: R131.2, U233.12 (D0)
- new net R23: R105.2, U251.11 (D1)
- new net R24: R101.2, U251.12 (D0)
- new net R25: R102.2, U236.9 (D3)
- new net R30: R90.2, U250.10 (D2)
- new net R31: R99.2, U250.11 (D1)
- new net R35: R40.2, U248.11 (D1)
- new net R37: U241.9 (D3)
- new net R43: R100.2, U238.11 (D1)
- new net R46: R85.2, U235.10 (D2)
- new net R47: R116.2, U235.11 (D1)
- new net R49: R97.2, U234.9 (D3)
- new net R5: R103.2, U252.9 (D3), U270.2 (S1), U271.2 (S1)
- new net R50: R92.2, U234.10 (D2)
- new net R51: U234.11 (D1)
- new net R53: R108.2, U240.9 (D3), U265.11
- new net R54: R106.2, U240.10 (D2)
- new net R56: R118.2, U240.12 (D0)
- new net R7: R117.2, U252.11 (D1), U253.10
- new net R8: R112.2, U252.12 (D0), U253.1
- new net RAA0: U233.15 (A7), U234.15 (A7), U235.15 (A7), U236.15 (A7), U248.15 (A7), U249.15 (A7), U250.15 (A7), U251.15 (A7), U252.15 (A7), U257.9 (Q)
- new net RAA1: U233.1 (A6), U234.1 (A6), U235.1 (A6), U236.1 (A6), U248.1 (A6), U249.1 (A6), U250.1 (A6), U251.1 (A6), U252.1 (A6), U259.9 (Q)
- new net RAA2: U233.2 (A5), U234.2 (A5), U235.2 (A5), U236.2 (A5), U248.2 (A5), U249.2 (A5), U250.2 (A5), U251.2 (A5), U252.2 (A5), U258.9 (Q)
- new net RAA3: U233.3 (A4), U234.3 (A4), U235.3 (A4), U236.3 (A4), U248.3 (A4), U249.3 (A4), U250.3 (A4), U251.3 (A4), U252.3 (A4), U257.5 (Q)
- new net RAA4: U233.4 (A3), U234.4 (A3), U235.4 (A3), U236.4 (A3), U248.4 (A3), U249.4 (A3), U250.4 (A3), U251.4 (A3), U252.4 (A3), U258.5 (Q)
- new net RAA5: U233.7 (A2), U234.7 (A2), U235.7 (A2), U236.7 (A2), U248.7 (A2), U249.7 (A2), U250.7 (A2), U251.7 (A2), U252.7 (A2), U259.5 (Q)
- new net RAA6: U233.6 (A1), U234.6 (A1), U235.6 (A1), U236.6 (A1), U247.9 (Q), U248.6 (A1), U249.6 (A1), U250.6 (A1), U251.6 (A1), U252.6 (A1)
- new net RAA7: U233.5 (A0), U234.5 (A0), U235.5 (A0), U236.5 (A0), U247.5 (Q), U248.5 (A0), U249.5 (A0), U250.5 (A0), U251.5 (A0), U252.5 (A0)
- new net RAB0: U237.2, U238.15 (A7), U239.15 (A7), U240.15 (A7), U241.15 (A7), U242.15 (A7)
- new net RAB1: U237.4, U238.1 (A6), U239.1 (A6), U240.1 (A6), U241.1 (A6), U242.1 (A6)
- new net RAB2: U237.12, U238.2 (A5), U239.2 (A5), U240.2 (A5), U241.2 (A5), U242.2 (A5), U243.3, U244.3
- new net RAB3: U238.3 (A4), U239.3 (A4), U240.3 (A4), U241.3 (A4), U242.3 (A4), U243.4, U244.4, U265.12
- new net RAB4: U237.6, U238.4 (A3), U239.4 (A3), U240.4 (A3), U241.4 (A3), U242.4 (A3)
- new net RAB5: U238.7 (A2), U239.7 (A2), U240.7 (A2), U241.7 (A2), U242.7 (A2), U243.6, U244.6, U265.2
- new net RAB6: U237.8, U238.6 (A1), U239.6 (A1), U240.6 (A1), U241.6 (A1), U242.6 (A1), U243.11
- new net RAB7: U237.10, U238.5 (A0), U239.5 (A0), U240.5 (A0), U241.5 (A0), U242.5 (A0), U243.12, U244.11
- new net RSC0: U266.7 (Za)
- new net SRAR16: U231.8
- new net ST3: U253.9
- new net ST40: U268.12 (D)
- new net SUBIMM: U268.5 (Q)
- new net UR1: U271.11 (I1b)
- new net UR2: U270.5 (I1a)
- new net UR3: U270.11 (I1b)
- new net ~{ADDIMM}: U243.8, U268.2 (D)
- new net ~{AL0TOCO}: U265.10
- new net ~{AR16}: U231.10, U232.8 (~{Q})
- new net ~{ARDOIT}: U262.12
- new net ~{ASIMM}: U244.8, U264.2 (D)
- new net ~{CY2}: U260.6
- new net ~{CYIN}: U253.8
- new net ~{CYZ}: U269.7 (Cn)
- new net ~{ENARLOAD}: U262.8
- new net ~{ENDAR}: U262.10
- new net ~{ENDER}: U267.12
- new net ~{ENDLR}: U261.12
- new net ~{ENDMR}: U261.4
- new net ~{ENDPC}: U263.10, U263.2
- new net ~{ENDSR}: U262.4
- new net ~{ENMALOAD}: U263.8
- new net ~{ENMPYOV}: U265.9
- new net ~{ENMRLOV}: U264.6 (~{Q})
- new net ~{ENPCLOAD}: U263.12
- new net ~{ENSER}: U267.10
- new net ~{ENSLR}: U261.9
- new net ~{ENSMR}: U261.2
- new net ~{ENSPC}: U263.11, U263.13
- new net ~{ENSRLOAD}: U262.6
- new net ~{ENSSR}: U262.2
- new net ~{ER0CLK}: U264.11 (C)
- new net ~{ER0}: U264.8 (~{Q})
- new net ~{ER15}: U232.10 (K1B)
- new net ~{LRFENAR}: U262.9
- new net ~{LRFENER}: U267.13
- new net ~{LRFENLR}: U261.13
- new net ~{LRFENMR}: U261.5
- new net ~{LRFENSR}: U262.5
- new net ~{LSC0}: U265.5
- new net ~{M3A}: U231.13
- new net ~{MDCLK}: U273.9 (Cp)
- new net ~{NSC0}: U265.3
- new net ~{R10}: R122.2, U242.10 (D2)
- new net ~{R11}: R124.2, U242.11 (D1), U254.12
- new net ~{R12}: R120.2, U242.12 (D0)
- new net ~{R13}: R109.2, U239.9 (D3)
- new net ~{R16}: R107.2, U239.12 (D0)
- new net ~{R17}: U233.9 (D3)
- new net ~{R18}: R81.2, U233.10 (D2)
- new net ~{R21}: R129.2, U251.9 (D3)
- new net ~{R26}: R84.2, U236.10 (D2)
- new net ~{R27}: R115.2, U236.11 (D1)
- new net ~{R28}: R83.2, U236.12 (D0)
- new net ~{R29}: R111.2, U250.9 (D3), U267.9
- new net ~{R2}: R89.2, U249.10 (D2)
- new net ~{R32}: R88.2, U250.12 (D0)
- new net ~{R33}: U248.9 (D3)
- new net ~{R34}: U248.10 (D2)
- new net ~{R38}: R94.2, U241.10 (D2), U261.1
- new net ~{R3}: R91.2, U249.11 (D1)
- new net ~{R40}: R114.2, U241.12 (D0), U262.13
- new net ~{R42}: R98.2, U238.10 (D2), U263.1
- new net ~{R45}: R14.2, U235.9 (D3), U263.9
- new net ~{R48}: R86.2, U235.12 (D0), U262.1
- new net ~{R4}: R93.2, U249.12 (D0)
- new net ~{R52}: R82.2, U234.12 (D0)
- new net ~{R55}: R113.2, U240.11 (D1), U261.10
- new net ~{R6}: R95.2, U252.10 (D2)
- new net ~{R9}: R126.2, U242.9 (D3), U254.1
- new net ~{RAA0}: U237.1, U243.1, U244.1, U257.8 (~{Q})
- new net ~{RAA1}: U237.3, U243.2, U244.2, U259.8 (~{Q})
- new net ~{RAA2}: U237.13, U258.8 (~{Q})
- new net ~{RAA3}: U257.6 (~{Q}), U265.13
- new net ~{RAA4}: U237.5, U243.5, U244.5, U258.6 (~{Q})
- new net ~{RAA5}: U259.6 (~{Q}), U265.1
- new net ~{RAA6}: U237.9, U247.8 (~{Q})
- new net ~{RAA7}: U237.11, U247.6 (~{Q})
- new net ~{SR16}: U231.1
- new net ~{ST479CK}: U268.11 (C)
- new net ~{ST4}: U268.8 (~{Q})
- new net ~{STLD}: U260.3
- new net ~{SUBIMM}: U268.6 (~{Q})
- no-connect marks 57 -> 98
Other:
- note removed: "CLKONQ CT To AU1 AU Interconnect Pin 25 to AU2 AU Interconnect Pin 25"
- note removed: "CT To AU1 AU Interconnect P3 Pin 20 To AU2 AU Interconnect P3 Pin 20"
- moved on the sheet: AX08-CTP1, AX08-CTP2, XA8-P1, XA8-P2

Commit message: Finished Columns 4 and 5 on AU2
Parts:
- added R132, R133, R134, R135, R136, R137, R138, R139: R, symbol Device:R
- added U275, U296, U304: 7442N, symbol 74xx:74LS42
- added U276, U278, U288, U289, U303: 74H51N, symbol TI980A:7451N
- added U277, U292: 74H11N, symbol 74xx:74LS11
- added U279, U285, U287, U293, U295, U299: 74153N, symbol 74xx:74LS153
- added U280, U281, U282, U283, U284: 74151N, symbol 74xx:74LS151
- added U286, U294: 74163N, symbol 74xx:74LS163
- added U290, U291, U297: 74H00N, symbol 74xx:7400
- added U298: 74H21N, symbol 74xx:74LS21
- added U300: 74H04N, symbol 74xx:74LS04
- added U301: 74H103N, symbol TI980A:74H103N
- added U302: 7410N, symbol 74xx:74LS10
- added U305: 74S65N, symbol TI980A:74S65N
- added U306: 7404N, symbol 74xx:74LS04
- added U307: 74H101, Package_DIP:DIP-14_W7.62mm, symbol TI980A:74H101
- added U308: 74S20N, symbol 74xx:74LS20
- U254: value 74LS37 -> 7437N
- U264: value 74H74N -> 7474N
- U266: value 74LS153 -> 74153N
- U269: value 74LS181 -> 74181
- U270, U271: value 74LS153 -> 74153
- U274: Location (none) -> AU2 Column 4 Row 21
Connections:
- net A0: now also U297.8, U298.1, U300.9
- net A1: now also U297.11, U298.2
- net A2: now also U297.6, U298.4
- net A3: now also U297.3, U298.5
- net ALU0: now also U274.2, U279.12 (I2b)
- net ALU0T: now also U276.1, U278.5
- net ALU1: now also U278.3, U279.13 (I3b), U287.4 (I2a)
- net ALU11: now also U287.10 (I0b)
- net ALU15: now also U293.10 (I0b), U299.5 (I1a)
- net ALU2: now also U279.11 (I1b), U287.12 (I2b), U287.3 (I3a)
- net ALU3: now also U287.13 (I3b), U287.5 (I1a), U295.4 (I2a)
- net ALU4: now also U287.11 (I1b), U295.12 (I2b), U295.3 (I3a)
- net ALUB6: now also U292.6
- net ALUB8: now also U292.12
- net ALUB9: now also U292.8
- net ALUS2: now also U278.13
- net API3: now also U290.11
- net BMAD1: now also U285.14 (S0)
- net BYTEINC: now also U307.11 (K2A), U307.12 (K2B), U307.3 (J2A), U307.4 (J2B)
- net CPUSTR: now also U289.6
- net ENALUB: now also U292.10, U292.2, U292.4
- net ENAPI: now also U288.1, U288.5, U289.1, U289.5, U290.1, U290.12, U290.4, U290.9, U291.1, U291.12, U291.4, U291.9
- net ENMPYOV: now also U274.1
- net ENNSC0: now also U276.9
- net ENNSC15: now also U303.2
- net ENRMLOV: now also U278.1
- net ER15: now also U306.1, U307.2 (J1B)
- net GCLKA:1: now also U276.3, U276.5
- net GCLKB:1: now also U301.1 (CLK), U301.5 (CLK), U307.13 (CLK)
- net GND: now also U275.8 (GND), U279.1 (Ea), U279.15 (Eb), U279.8 (GND), U280.1 (I3), U280.8 (GND), U281.1 (I3), U281.8 (GND), U282.1 (I3), U282.8 (GND), U283.1 (I3), U283.8 (GND), U284.1 (I3), U284.8 (GND), U285.8 (GND), U286.8 (GND), U287.1 (Ea), U287.15 (Eb), U287.8 (GND), U293.1 (Ea), U293.15 (Eb), U293.8 (GND), U294.8 (GND), U295.1 (Ea), U295.15 (Eb), U295.8 (GND), U296.8 (GND), U299.1 (Ea), U299.15 (Eb), U299.8 (GND), U304.8 (GND), U305.2, U305.3, U307.7 (GND)
- net IFLAGQ: now also U277.4
- net INAQ: now also U277.3
- net INHMSB: now also U285.1 (Ea), U285.15 (Eb), U302.12
- net IR0: now also U280.13 (I6)
- net IR1: now also U281.13 (I6)
- net IR13: now also U296.13 (A2)
- net IR2: now also U283.13 (I6)
- net IR3: now also U282.13 (I6)
- net IR4: now also U284.13 (I6)
- net IR8A: now also U285.13 (I3b), U285.3 (I3a), U300.2
- net LSC0: now also U279.5 (I1a)
- net LSC15: now also U299.11 (I1b)
- net M3: now also U306.11
- net M4: now also U305.5
- net MAL4: now also U305.11
- net MAR0: now also U286.11 (Q3)
- net MAR1: now also U286.12 (Q2)
- net MAR2: now also U286.13 (Q1)
- net MAR3: now also U286.14 (Q0)
- net MAR4: now also U285.6 (I0a), U294.11 (Q3)
- net MAR5: now also U285.10 (I0b), U294.12 (Q2)
- net MAR6: now also U294.13 (Q1)
- net MAR7: now also U294.14 (Q0)
- net MDR4: now also U285.4 (I2a)
- net MDR5: now also U285.12 (I2b)
- net MEM0: now also U280.14 (I5)
- net MEM1: now also U281.14 (I5)
- net MEM2: now also U283.14 (I5)
- net MEM3: now also U282.14 (I5)
- net MEM4: now also U284.14 (I5)
- net NSC0: now also U279.3 (I3a)
- net PNL0: now also U280.15 (I4)
- net PNL1: now also U281.15 (I4)
- net PNL2: now also U283.15 (I4)
- net PNL3: now also U282.15 (I4)
- net PNL4: now also R138.2, U284.15 (I4)
- net PNL5: now also R136.2
- net PNL6: now also R134.2
- net PNL7: now also R132.2
- net R1: now also U305.10
- net R20: now also U288.2
- net R30: now also U276.4
- net R47: now also U305.4
- net R5: now also U285.2 (S1)
- net R53: now also U278.4
- net RSC0: now also U279.4 (I2a)
- net SC2: now also U275.13 (A2)
- net SC3: now also U275.14 (A1)
- net SC4: now also U275.15 (A0)
- net SR16: now also U307.6 (Q)
- net ST0: now also U280.4 (I0)
- net ST1: now also U281.4 (I0)
- net ST2: now also U283.4 (I0)
- net ST3: now also U282.4 (I0)
- net ST4: now also U284.4 (I0)
- net SUBIMM: now also U278.9
- net UR0: now also U306.3
- net VCC1: now also R132.1, R133.1, R134.1, R135.1, R136.1, R137.1, R138.1, R139.1, U275.16 (VCC), U277.5, U279.16 (VCC), U280.16 (VCC), U281.16 (VCC), U282.16 (VCC), U283.16 (VCC), U284.16 (VCC), U285.16 (VCC), U286.1 (~{MR}), U286.16 (VCC), U287.16 (VCC), U288.13, U288.3, U288.9, U289.10, U289.3, U293.16 (VCC), U294.1 (~{MR}), U294.16 (VCC), U295.16 (VCC), U296.16 (VCC), U299.16 (VCC), U301.2 (~{R}), U301.6 (~{R}), U304.16 (VCC), U305.1, U305.9, U307.14 (VCC), U307.5 (Pre)
- net ~{AL0TOCO}: now also U278.2
- net ~{ALU0}: now also U276.10
- net ~{ALU15}: now also U303.3
- net ~{ALUEQ8K}: now also U274.12
- net ~{API10}: now also U290.5
- net ~{API12}: now also U290.10
- net ~{API3}: now also U290.13
- net ~{API5}: now also U291.5
- net ~{API6}: now also U291.2
- net ~{API7}: now also U291.10
- net ~{API8}: now also U290.2
- net ~{API9}: now also U291.13
- net ~{APISTORE}: now also U289.4
- net ~{BYTESHFT}: now also U277.2
- net ~{CPUCR}: now also U288.6
- net ~{DIVIT}: now also U277.13
- net ~{DP0}: now also R139.2, U280.3 (I1)
- net ~{DP1}: now also R137.2, U281.3 (I1)
- net ~{DP2}: now also R135.2, U283.3 (I1)
- net ~{DP3}: now also R133.2, U282.3 (I1)
- net ~{DP4}: now also U284.3 (I1)
- net ~{ENDAR}: now also U304.1 (0)
- net ~{ENDER}: now also U304.2 (1)
- net ~{ENDLR}: now also U304.6 (5)
- net ~{ENDMR}: now also U304.4 (3)
- net ~{ENDPC}: now also U302.10, U304.9 (7)
- net ~{ENDSR}: now also U304.5 (4)
- net ~{ENDXR}: now also U304.3 (2)
- net ~{ENMAINC}: now also U288.10
- net ~{ENMALOAD}: now also U286.9 (~{PE}), U294.9 (~{PE})
- net ~{ENSPC}: now also U277.11, U302.9
- net ~{ER0CLK}: now also U276.6
- net ~{ER15}: now also U306.2, U307.10 (K1B)
- net ~{GCLKC:1}: now also U286.2 (CP), U294.2 (CP)
- net ~{INHMUA1}: now also U274.10, U302.1
- net ~{INHMUA2}: now also U308.10
- net ~{INHMUB1}: now also U302.2, U308.12
- net ~{INHMUB2}: now also U274.11
- net ~{IR8}: now also U300.1
- net ~{LRFENAR}: now also U275.1 (0)
- net ~{LRFENER}: now also U275.2 (1)
- net ~{LRFENLR}: now also U275.6 (5)
- net ~{LRFENMR}: now also U275.4 (3)
- net ~{LRFENSR}: now also U275.5 (4)
- net ~{LSC0}: now also U278.6
- net ~{M2LC}: now also U308.13
- net ~{M3A}: now also U306.10
- net ~{MALOAD}: now also U289.8
- net ~{MCL4}: now also U277.9
- net ~{MRESETQ}: now also U302.4, U306.9
- net ~{NSC0}: now also U276.8
- net ~{R16}: now also U277.1
- net ~{R18}: now also U277.10
- net ~{R21}: now also U289.2
- net ~{R45}: now also U302.11
- net ~{R52}: now also U302.13
- net ~{SR16}: now also U307.8 (~{Q})
- net ~{ST15}: now also U305.12
- net ~{ST5}: now also U301.8 (~{Q})
- net ~{ST6}: now also U301.13 (~{Q})
- net ~{STLD}: now also U300.6, U302.3
- net INHLSA: now reaches U274.8
- net ~{AMADQA}: now reaches U274.9
- net ALUZI15: now reaches U274.13
- new net ALU10: U287.6 (I0a)
- new net ALU12: U295.6 (I0a)
- new net ALU13: U295.10 (I0b), U299.4 (I2a)
- new net ALU14: U293.6 (I0a), U299.12 (I2b), U299.3 (I3a)
- new net ALU15A: U303.5
- new net ALU5: U293.4 (I2a), U295.13 (I3b), U295.5 (I1a)
- new net ALU6: U292.3, U293.12 (I2b), U293.3 (I3a), U295.11 (I1b), U299.6 (I0a)
- new net ALU7: U293.13 (I3b), U293.5 (I1a), U299.10 (I0b)
- new net ALU8: U279.6 (I0a), U292.1, U293.11 (I1b)
- new net ALU9: U279.10 (I0b), U292.9
- new net AMAD1: U280.9 (S2), U281.9 (S2), U282.9 (S2), U283.9 (S2), U284.9 (S2)
- new net AMAD2: U280.10 (S1), U281.10 (S1), U282.10 (S1), U283.10 (S1), U284.10 (S1)
- new net AMAD3: U280.11 (S0), U281.11 (S0), U282.11 (S0), U283.11 (S0), U284.11 (S0)
- new net API10: U290.6
- new net API12: U290.8
- new net API5: U291.6
- new net API6: U291.3, U292.5
- new net API7: U291.8
- new net API8: U290.3, U292.13
- new net API9: U291.11, U292.11
- new net APICYCRQ: U288.4
- new net APIMALD: U289.13
- new net B4: U285.7 (Za)
- new net B5: U285.9 (Zb)
- new net C0: U279.7 (Za), U286.6 (D3)
- new net C1: U279.9 (Zb), U286.5 (D2)
- new net C14: U299.7 (Za)
- new net C15: U299.9 (Zb)
- new net C2: U286.4 (D1), U287.7 (Za)
- new net C3: U286.3 (D0), U287.9 (Zb)
- new net C4: U294.6 (D3), U295.7 (Za)
- new net C5: U294.5 (D2), U295.9 (Zb)
- new net C6: U293.7 (Za), U294.4 (D1)
- new net C7: U293.9 (Zb), U294.3 (D0)
- new net CADRA: U279.14 (S0), U287.14 (S0), U293.14 (S0), U295.14 (S0), U299.14 (S0)
- new net CADRB: U277.12, U279.2 (S1), U287.2 (S1), U293.2 (S1), U295.2 (S1), U299.2 (S1)
- new net ENDMSC: U304.13 (A2)
- new net ENMAINC: U286.7 (CEP), U288.8, U294.7 (CEP)
- new net ENMALOAD: U289.9, U302.8
- new net ENMASK: U277.6, U300.11
- new net ER15SELA: U306.13
- new net ER15SELB: U306.5
- new net ERLD: U276.2
- new net ERSR16LD: U307.1 (J1A), U307.9 (K1A)
- new net INHMSA: U308.8
- new net INVB0: U300.12
- new net IR12: U296.12 (A3), U305.6
- new net IR14: U296.14 (A1), U304.14 (A1)
- new net IR15: U296.15 (A0), U304.15 (A0)
- new net LDST: U300.5
- new net MACR2: U294.10 (CET)
- new net MACR3: U286.10 (CET), U294.15 (TC)
- new net MRESETQA: U306.8
- new net NSC15: U299.13 (I3b), U300.4
- new net PCS0: U280.12 (I7)
- new net PCS1: U281.12 (I7)
- new net PCS2: U283.12 (I7)
- new net PCS3: U282.12 (I7)
- new net PCS4: U284.12 (I7)
- new net SOOA: U298.6
- new net ST5: U301.9 (Q)
- new net ST56A: U305.13
- new net ST5J: U301.7 (J)
- new net ST6: U301.12 (Q)
- new net ST6J: U301.14 (J)
- new net STLDCLR: U301.10 (K), U301.3 (K), U302.6
- new net SZEA: U298.8
- new net UR4: U285.5 (I1a)
- new net UR5: U285.11 (I1b)
- new net ~{A0}: U300.8
- new net ~{ALS0}: U297.9, U298.9
- new net ~{ALS1}: U297.12, U298.10
- new net ~{ALS2}: U297.4, U298.12
- new net ~{ALS3}: U297.1, U298.13
- new net ~{AMAD0A}: U280.7 (~{E}), U281.7 (~{E}), U282.7 (~{E}), U283.7 (~{E}), U284.7 (~{E}), U305.8, U308.9
- new net ~{AMS0}: U280.6 (~{Z}), U297.10
- new net ~{AMS1}: U281.6 (~{Z}), U297.13
- new net ~{AMS2}: U283.6 (~{Z}), U297.5
- new net ~{AMS3}: U282.6 (~{Z}), U297.2
- new net ~{AMS4}: U284.6 (~{Z})
- new net ~{ENALUB1}: U277.8
- new net ~{ENDBR}: U304.7 (6)
- new net ~{ENDMSD}: U304.12 (A3)
- new net ~{ENDST}: U304.10 (8)
- new net ~{ENDZ1}: U304.11 (9)
- new net ~{ENNSC0}: U276.13
- new net ~{ENNSC15}: U303.4
- new net ~{ENRMLOV}: U278.10
- new net ~{ER15SELA}: U306.12
- new net ~{ER15SELB}: U306.6
- new net ~{INTCLR}: U300.10, U302.5
- new net ~{INVB0}: U278.8, U300.13
- new net ~{LRFENBR}: U275.7 (6)
- new net ~{LRFENXR}: U275.3 (2)
- new net ~{MALB}: U275.12 (A3)
- new net ~{NSC15}: U300.3, U303.6
- new net ~{SETBIT0}: U280.2 (I2), U296.1 (0)
- new net ~{SETBIT1}: U281.2 (I2), U296.2 (1)
- new net ~{SETBIT2}: U283.2 (I2), U296.3 (2)
- new net ~{SETBIT3}: U282.2 (I2), U296.4 (3)
- new net ~{SETBIT4}: U284.2 (I2), U296.5 (4)
- new net ~{SETBIT5}: U296.6 (5)
- new net ~{SETBIT6}: U296.7 (6)
- new net ~{SETBIT7}: U296.9 (7)
- new net ~{UR0}: U306.4
- no-connect marks 98 -> 123

Commit message: Finished Column 6 on AU2
Parts:
- added R140, R141, R142, R143, R144, R145, R146, R147: R, symbol Device:R
- added U309, U310: 74H11N, symbol 74xx:74LS11
- added U311, U312, U314, U317: 74153N, symbol 74xx:74LS153
- added U313, U315, U316: 74151N, symbol 74xx:74LS151
- added U318: 74H30N, symbol 74xx:74LS30
- added U319, U323: 7442N, symbol 74xx:74LS42
- added U320: 74H04N, symbol 74xx:74LS04
- added U321: 7410N, symbol 74xx:74LS10
- added U322: 7437N, symbol 74xx:74LS37
- added U324: 7420N, symbol 74xx:74LS20
- added U325: 7486N, symbol 74xx:74LS86
- added U326: 74H52N, symbol TI980A:74H52N
- added U327: 74H00N, symbol 74xx:7400
Connections:
- net ALU0: now also U311.6 (I0a)
- net ALU0T: now also U325.1, U326.2
- net ALU1: now also U311.10 (I0b)
- net ALU10: now also U310.3, U311.11 (I1b), U317.12 (I2b), U317.3 (I3a)
- net ALU11: now also U314.4 (I2a), U317.13 (I3b), U317.5 (I1a)
- net ALU12: now also U309.3, U314.12 (I2b), U314.3 (I3a), U317.11 (I1b)
- net ALU13: now also U310.1, U314.13 (I3b), U314.5 (I1a)
- net ALU14: now also U314.11 (I1b)
- net ALU2: now also U317.6 (I0a)
- net ALU3: now also U317.10 (I0b)
- net ALU4: now also U314.6 (I0a)
- net ALU5: now also U309.1, U314.10 (I0b)
- net ALU7: now also U309.9, U311.4 (I2a)
- net ALU8: now also U311.12 (I2b), U311.3 (I3a)
- net ALU9: now also U311.13 (I3b), U311.5 (I1a), U317.4 (I2a)
- net ALUB10: now also U310.6
- net ALUB12: now also U309.6
- net ALUB13: now also U310.12
- net ALUB5: now also U309.12
- net ALUB7: now also U309.8
- net ALUS0: now also U322.8
- net ALUS2: now also U322.6
- net AMAD1: now also U315.9 (S2), U316.9 (S2)
- net AMAD2: now also U315.10 (S1), U316.10 (S1)
- net AMAD3: now also U315.11 (S0), U316.11 (S0)
- net API10: now also U310.5
- net API12: now also U309.5
- net API5: now also U309.13
- net API7: now also U309.11
- net BMAD1: now also U312.14 (S0)
- net CADRA: now also U311.14 (S0), U314.14 (S0), U317.14 (S0)
- net CADRB: now also U311.2 (S1), U314.2 (S1), U317.2 (S1)
- net CLKONQ: now also U327.10
- net ENALUB: now also U309.10, U309.2, U309.4, U310.2, U310.4, U322.3
- net ENAPI: now also U322.11
- net ENPCOUT: now also U327.9
- net ER1: now also U325.13
- net ER15SELA: now also U326.11, U326.4
- net ER15SELB: now also U326.5
- net GND: now also U311.1 (Ea), U311.15 (Eb), U311.8 (GND), U312.8 (GND), U313.8 (GND), U314.1 (Ea), U314.15 (Eb), U314.8 (GND), U315.1 (I3), U315.8 (GND), U316.1 (I3), U316.8 (GND), U317.1 (Ea), U317.15 (Eb), U317.8 (GND), U319.12 (A3), U319.8 (GND), U323.8 (GND)
- net INHMSB: now also U312.1 (Ea), U312.15 (Eb)
- net IR11: now also U323.15 (A0)
- net IR12: now also U313.7 (~{E})
- net IR13: now also U313.9 (S2)
- net IR14: now also U313.10 (S1)
- net IR15: now also U313.11 (S0)
- net IR5: now also U316.13 (I6)
- net IR6: now also U315.13 (I6)
- net IR8A: now also U312.13 (I3b), U312.3 (I3a)
- net LDST: now also U310.10
- net M0LF: now also U327.13
- net M1LE: now also U326.1
- net M8LBC: now also U325.12
- net MAR6: now also U312.6 (I0a)
- net MAR7: now also U312.10 (I0b)
- net MEM5: now also U316.14 (I5)
- net MEM6: now also U315.14 (I5)
- net PNL10: now also R144.2
- net PNL11: now also R140.2
- net PNL12: now also R142.2
- net PNL13: now also R146.2
- net PNL14: now also R141.2
- net PNL15: now also R145.2
- net PNL5: now also U316.15 (I4)
- net PNL6: now also U315.15 (I4)
- net PNL8: now also R147.2
- net PNL9: now also R143.2
- net R23: now also U319.13 (A2)
- net R24: now also U319.14 (A1)
- net R25: now also U319.15 (A0)
- net R5: now also U312.2 (S1)
- net R50: now also U327.5
- net SRAR16: now also U326.3
- net ST5: now also U316.4 (I0)
- net ST6: now also U315.4 (I0)
- net UR0: now also U313.4 (I0)
- net UR1: now also U313.3 (I1)
- net UR2: now also U313.2 (I2)
- net UR3: now also U313.1 (I3)
- net UR4: now also U313.15 (I4)
- net UR5: now also U313.14 (I5)
- net VCC1: now also R140.1, R141.1, R142.1, R143.1, R144.1, R145.1, R146.1, R147.1, U310.11, U310.9, U311.16 (VCC), U312.16 (VCC), U313.16 (VCC), U314.16 (VCC), U315.16 (VCC), U316.16 (VCC), U317.16 (VCC), U318.12, U319.16 (VCC), U322.12, U323.16 (VCC)
- net ~{ALUEQA}: now also U322.10, U322.5
- net ~{AMAD0A}: now also U315.7 (~{E}), U316.7 (~{E})
- net ~{BRLD}: now also U324.9
- net ~{CY2}: now also U321.13
- net ~{DP5}: now also U316.3 (I1)
- net ~{DP6}: now also U315.3 (I1)
- net ~{ENALUB1}: now also U322.1
- net ~{ENDBR}: now also U324.12
- net ~{ENDMSD}: now also U327.6
- net ~{ENDPC}: now also U322.2
- net ~{ENMPYOV}: now also U318.4, U319.5 (4)
- net ~{ENSLR}: now also U323.6 (5)
- net ~{ENSMR}: now also U323.4 (3)
- net ~{ENSPC}: now also U323.9 (7)
- net ~{ENSSR}: now also U323.5 (4)
- net ~{ENSXR}: now also U323.3 (2)
- net ~{ER15SELB}: now also U326.10
- net ~{INHMUA2}: now also U327.1
- net ~{INHMUB2}: now also U327.2
- net ~{LRFENBR}: now also U324.13
- net ~{M4LF}: now also U323.12 (A3)
- net ~{MCL4}: now also U322.13
- net ~{R10}: now also U322.4
- net ~{R12}: now also U322.9
- net ~{SETBIT5}: now also U316.2 (I2)
- net ~{SETBIT6}: now also U315.2 (I2)
- net ~{SKIP}: now also U327.11
- net ~{ST2CLR}: now also U318.2
- net ~{STLD}: now also U318.6, U321.3
- net ~{UR0}: now also U325.2
- new net A0EQB0: U320.8
- new net AEQO: U320.12
- new net ALUEQUR0: U325.3, U326.12
- new net API13: U310.13
- new net B6: U312.7 (Za)
- new net B7: U312.9 (Zb)
- new net C10: U317.7 (Za)
- new net C11: U317.9 (Zb)
- new net C12: U314.7 (Za)
- new net C13: U314.9 (Zb)
- new net C8: U311.7 (Za)
- new net C9: U311.9 (Zb)
- new net ENARITH: U320.6
- new net ENASOV: U320.2
- new net ENBRLOAD: U324.8
- new net ENDVOV: U320.10
- new net ENLSOV: U320.4
- new net ENOVCK: U318.8
- new net ER0SELD: U325.11
- new net ER15IN: U326.8
- new net ER15INA: U326.13
- new net INHLSB: U327.3
- new net IR10: U323.14 (A1)
- new net IR9: U323.13 (A2)
- new net MDR6: U312.4 (I2a)
- new net MDR7: U312.12 (I2b)
- new net PCS5: U316.12 (I7)
- new net PCS6: U315.12 (I7)
- new net SKIP: U321.8, U327.12
- new net ST3D: U321.12
- new net STLD: U310.8
- new net UR6: U312.5 (I1a), U313.13 (I6)
- new net UR7: U312.11 (I1b), U313.12 (I7)
- new net ~{A0EQB0}: U320.9
- new net ~{AEQO}: U320.13
- new net ~{ALU0T}: U321.4
- new net ~{AMS5}: U316.6 (~{Z})
- new net ~{AMS6}: U315.6 (~{Z})
- new net ~{APIS2EN}: U318.11
- new net ~{AXB0}: U321.5
- new net ~{BIT1}: U313.6 (~{Z})
- new net ~{BITSK}: U321.11
- new net ~{CY1}: U321.2, U321.6
- new net ~{ENARITH}: U319.7 (6), U320.5
- new net ~{ENASOV}: U318.1, U319.2 (1), U320.1
- new net ~{ENDVOV}: U318.5, U319.6 (5), U320.11
- new net ~{ENLOGIC}: U319.9 (7)
- new net ~{ENLSOV}: U318.3, U319.4 (3), U320.3
- new net ~{ENSAR}: U323.1 (0)
- new net ~{ENSBR}: U323.7 (6), U324.10
- new net ~{ENSFR}: U323.2 (1)
- new net ~{ENSZ1}: U323.10 (8)
- new net ~{ENSZ2}: U323.11 (9)
- new net ~{ENTCOV}: U319.3 (2)
- new net ~{INDSK}: U321.10
- new net ~{MB12}: U327.4
- new net ~{PCOUTA}: U327.8
- new net ~{REGSK}: U321.9
- new net ~{STALU3}: U321.1
- no-connect marks 123 -> 141
