File: TI980A-Arithmetic-Unit/AU2.kicad_sch (KiCad schematic)
At the start: 181 parts, among them U15 74H40N, U16 74H40N, U17 74H40N, U18 74H11N, U19 74H04N, U20 74H40N, U231 7451N, U232 74H101, U233 74187, U234 74187, U235 74187, U236 74187, U237 74H04N, U238 74187, U239 74187, U240 74187, U241 74187, U242 74187, U243 7430N, U244 7430N, U245 74H11N, U246 74H00N, U247 74H74N, U248 74187, U249 74187, U250 74187, U251 74187, U252 74187, U253 7451N, U254 7437N, U255 74S65N, U256 74H00N, U257 74H74N, U258 74H74N, U259 74H74N, U260 7410N, U261 7420N, U262 74H21N, U263 74H11N, U264 7474N, U265 74H04N, U266 74153N, U267 74H20N, U268 7474N, U269 74181, U270 74153, U271 74153, U272 74H11N, U273 74174N, U274 74S10N, U275 7442N, U276 74H51N, U277 74H11N, U278 74H51N, U279 74153N, U280 74151N, U281 74151N, U282 74151N, U283 74151N, U284 74151N, U285 74153N, U286 74163N, U287 74153N, U288 74H51N, U289 74H51N, U290 74H00N, U291 74H00N, U292 74H11N, U293 74153N, U294 74163N, U295 74153N, U296 7442N, U297 74H00N, U298 74H21N, U299 74153N, U300 74H04N, U301 74H103N, U302 7410N, U303 74H51N, U304 7442N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

Commit message: Finished Column 7 on AU2
Parts:
- added C5: C_Polarized, symbol Device:C_Polarized
- added U328, U342: 74H11N, symbol 74xx:74LS11
- added U329: 74157N, symbol 74xx:74LS157
- added U330, U335, U341: 74H00N, symbol 74xx:7400
- added U331, U332, U338, U339: 74163N, symbol 74xx:74LS163
- added U333: 74181, symbol 74xx:74LS181
- added U334, U344: 74174N, symbol 74xx:74LS174
- added U336: 74H55N, symbol TI980A:74H55N
- added U337: 74S40N, symbol 74xx:74LS40
- added U340: 74H54W, symbol TI980A:74H54N
- added U343: 7408N, symbol 74xx:74LS08
Connections:
- net A0: now also U336.12
- net A0EQB0: now also U336.4
- net AEQB: now also U333.14 (A=B)
- net ALU0: now also U329.3 (I1a)
- net ALU0T: now also U336.2
- net ALU1: now also U329.6 (I1b)
- net ALU14: now also U328.3
- net ALU2: now also U329.13 (I1d)
- net ALU3: now also U329.10 (I1c)
- net ALU4: now also U333.13 (F3)
- net ALU5: now also U333.11 (F2)
- net ALU6: now also U333.10 (F1)
- net ALU7: now also U333.9 (F0)
- net ALUB14: now also U328.6
- net ALUM: now also U333.8 (M)
- net ALUS0: now also U333.6 (S0)
- net ALUS1: now also U333.5 (S1)
- net ALUS2: now also U333.4 (S2)
- net ALUS3: now also U333.3 (S3)
- net AMAD2: now also U337.8
- net AMAD3: now also U337.6
- net B4: now also U333.18 (B3)
- net B5: now also U333.20 (B2)
- net B6: now also U333.22 (B1)
- net B7: now also U333.1 (B0)
- net BYTEINC: now also U343.9
- net C0: now also U338.6 (D3)
- net C1: now also U338.5 (D2)
- net C10: now also U331.4 (D1)
- net C11: now also U331.3 (D0)
- net C12: now also U332.6 (D3)
- net C13: now also U332.5 (D2)
- net C14: now also U332.4 (D1)
- net C15: now also U332.3 (D0)
- net C2: now also U338.4 (D1)
- net C3: now also U338.3 (D0)
- net C4: now also U339.6 (D3)
- net C5: now also U339.5 (D2)
- net C6: now also U339.4 (D1)
- net C7: now also U339.3 (D0)
- net C8: now also U331.6 (D3)
- net C9: now also U331.5 (D2)
- net CADRA: now also U342.6
- net ENALUB: now also U328.4
- net ENAPI: now also U330.4, U340.6
- net ENARITH: now also U336.1, U336.10
- net ENIRLOAD: now also U330.12
- net ENLRLOAD: now also U341.4
- net ENMAINC: now also U331.7 (CEP), U332.7 (CEP)
- net ENPCINC: now also U338.7 (CEP)
- net ER15INA: now also U343.3
- net ER15SELB: now also U341.11, U343.1
- net GCLKA:1: now also U330.10, U330.13, U341.5
- net GND: now also U331.8 (GND), U332.8 (GND), U333.12 (GND), U334.8 (GND), U338.8 (GND), U339.8 (GND), U344.8 (GND)
- net IFLAGQ: now also U343.5
- net INAQ: now also U343.4
- net IOUT0: now also U329.4 (Za)
- net IOUT1: now also U329.7 (Zb)
- net IOUT2: now also U329.12 (Zd)
- net IOUT3: now also U329.9 (Zc)
- net IR12: now also U341.2
- net IR14: now also U335.9
- net IR15: now also U335.12
- net LDST: now also U330.3
- net M0LF: now also U340.2
- net MACR2: now also U331.15 (TC)
- net MADOIT: now also U340.10
- net MAR10: now also U331.13 (Q1)
- net MAR11: now also U331.14 (Q0)
- net MAR12: now also U332.11 (Q3)
- net MAR13: now also U332.12 (Q2)
- net MAR14: now also U332.13 (Q1)
- net MAR15: now also U332.14 (Q0)
- net MAR8: now also U331.11 (Q3)
- net MAR9: now also U331.12 (Q2)
- net MDR10: now also U344.12 (Q4)
- net MDR6: now also U344.2 (Q0)
- net MDR7: now also U344.5 (Q1)
- net MEM10: now also U344.13 (D4)
- net MEM11: now also U344.14 (D5)
- net MEM6: now also U344.3 (D0)
- net MEM7: now also U344.4 (D1)
- net MEM8: now also U344.6 (D2)
- net MEM9: now also U344.11 (D3)
- net PCS0: now also U334.2 (Q0)
- net PCS1: now also U334.5 (Q1)
- net PCS2: now also U334.7 (Q2)
- net PCS3: now also U334.10 (Q3)
- net PCS4: now also U334.12 (Q4)
- net PCS5: now also U334.15 (Q5)
- net PFAIL: now also U342.1
- net R35: now also U340.13
- net R47: now also U335.10, U335.13
- net SC4: now also U342.9
- net SKIP: now also U340.3
- net SR16: now also U343.10
- net ST9G: now also U328.8
- net STLDCLR: now also U330.9
- net VCC1: now also C5.1, U328.9, U329.16 (VCC), U331.1 (~{MR}), U331.16 (VCC), U332.1 (~{MR}), U332.10 (CET), U332.16 (VCC), U333.24 (VCC), U334.1 (~{Mr}), U334.16 (VCC), U336.13, U338.1 (~{MR}), U338.16 (VCC), U339.16 (VCC), U340.1, U340.4, U340.9, U342.10, U342.11, U344.1 (~{Mr}), U344.16 (VCC)
- net ~{A0EQB0}: now also U336.11
- net ~{AMS4}: now also U335.2
- net ~{AMS5}: now also U335.5
- net ~{API14}: now also U330.5
- net ~{ARDOIT}: now also U343.11
- net ~{BYTESHFT}: now also U342.5
- net ~{DIVIT}: now also U341.13
- net ~{ENARCLR}: now also U339.1 (~{MR})
- net ~{ENARLOAD}: now also U339.9 (~{PE})
- net ~{ENDST}: now also U330.2
- net ~{ENIOUT}: now also U329.15 (E)
- net ~{ENMAINC}: now also U340.8
- net ~{ENMALOAD}: now also U331.9 (~{PE}), U332.9 (~{PE})
- net ~{ENPCLOAD}: now also U338.9 (~{PE})
- net ~{ENSAR}: now also U343.13
- net ~{ER15SELA}: now also U343.2
- net ~{GCLKC:1}: now also U331.2 (CP), U332.2 (CP), U338.2 (CP)
- net ~{GCLKC:2}: now also U339.2 (CP)
- net ~{IFLAG}: now also U328.10, U342.2
- net ~{MB12}: now also U341.3
- net ~{MB}: now also U341.1
- net ~{MDCLK}: now also U344.9 (Cp)
- net ~{MPYIT}: now also U341.10, U342.4
- net ~{PCOUTA}: now also U329.1 (S)
- net ~{R17}: now also U342.3
- net ~{R27}: now also U330.1
- net ~{R32}: now also U341.9
- net ~{R33}: now also U341.12
- net ~{R3}: now also U337.13
- net ~{R4}: now also U337.5
- net ~{ST479CK}: now also U330.8
- new net A4: U333.19 (A3), U335.3
- new net A5: U333.21 (A2), U335.6
- new net A6: U333.23 (A1)
- new net A7: U333.2 (A0)
- new net API14: U328.5, U330.6
- new net APIMAINC: U340.5
- new net AR4: U339.11 (Q3)
- new net AR5: U339.12 (Q2)
- new net AR6: U339.13 (Q1)
- new net AR7: U339.14 (Q0)
- new net ARCR2: U339.10 (CET)
- new net CYGZ: U333.17 (Y)
- new net CYPZ: U333.15 (X)
- new net ENARINC: U339.7 (CEP)
- new net ENSRINC: U343.8
- new net ER0SELA: U341.8
- new net GND1: C5.2, U329.8 (GND)
- new net MACR1: U331.10 (CET), U332.15 (TC)
- new net MDR11: U344.15 (Q5)
- new net MDR8: U344.7 (Q2)
- new net MDR9: U344.10 (Q3)
- new net PC0: U329.2 (I0a), U334.3 (D0), U338.11 (Q3)
- new net PC1: U329.5 (I0b), U334.4 (D1), U338.12 (Q2)
- new net PC2: U329.14 (I0d), U334.6 (D2), U338.13 (Q1)
- new net PC3: U329.11 (I0c), U334.11 (D3), U338.14 (Q0)
- new net PC4: U334.13 (D4)
- new net PC5: U334.14 (D5)
- new net PCCR3: U338.10 (CET)
- new net SC4X: U342.8
- new net ST15J: U342.12
- new net ST15KA: U343.6
- new net ST9: U328.11
- new net ~{AEQB}: U336.3
- new net ~{ALS4}: U335.1
- new net ~{ALS5}: U335.4
- new net ~{AMAD2A}: U337.9
- new net ~{AMAD2B}: U335.8, U337.10
- new net ~{AMAD2C}: U337.12
- new net ~{AMAD3A}: U337.1
- new net ~{AMAD3B}: U335.11, U337.2
- new net ~{AMAD3C}: U337.4
- new net ~{CYY}: U333.7 (Cn)
- new net ~{IRCLK}: U330.11
- new net ~{LRCLK}: U341.6
- new net ~{MBLAST2}: U343.12
- new net ~{PCSCLK}: U334.9 (Cp)
- new net ~{PENSKQ}: U342.13
- no-connect marks 141 -> 150

Commit message: Finished Column 8 on AU2
Parts:
- added U345: 74H04N, symbol 74xx:74LS04
- added U346: 7408N, symbol 74xx:74LS08
- added U347: 74175N, symbol 74xx:74LS175
- added U348: 74153N, symbol 74xx:74LS153
- added U349: 74174N, symbol 74xx:74LS174
- added U350, U352: 74H21N, symbol 74xx:74LS21
- added U351: 74182N, symbol 74xx:74LS182
- added U353, U359: 74S00N, symbol 74xx:7400
- added U354: 74H55N, symbol TI980A:74H55N
- added U355, U357: 74H20N, symbol 74xx:74LS20
- added U356: 7400N, symbol 74xx:7400
- added U358: 74H00N, symbol 74xx:7400
- added U360: 74H10N, symbol 74xx:74LS10
Connections:
- net A0EQB0: now also U354.3
- net A4: now also U352.1
- net A5: now also U352.2
- net A6: now also U352.4, U353.3
- net A7: now also U352.5, U353.6
- net AEQB: now also U345.13
- net ALU0T: now also U354.2
- net ALU3: now also U356.13
- net APICYCRQ: now also U345.2
- net APIMAINC: now also U345.4
- net APIMALD: now also U345.6
- net B0: now also U354.11
- net BMAD1: now also U348.14 (S0), U353.11
- net C10: now also U349.13 (D4)
- net C11: now also U349.14 (D5)
- net C6: now also U349.3 (D0)
- net C7: now also U349.4 (D1)
- net C8: now also U349.6 (D2)
- net C9: now also U349.11 (D3)
- net CYGZ: now also U351.14 (G2)
- net CYPZ: now also U351.15 (P2)
- net ENAPI: now also U345.11
- net ENDMSC: now also U358.3
- net ENMASK: now also U360.11, U360.5
- net ENMRLOAD: now also U356.9
- net ER0SELA: now also U346.2
- net GCLKA:1: now also U356.10, U356.2, U356.5, U358.13, U358.5
- net GND: now also U347.8 (GND), U348.8 (GND), U349.8 (GND), U351.8 (GND)
- net INHMSB: now also U348.1 (Ea), U348.15 (Eb)
- net IR10: now also U347.10 (Q2)
- net IR11: now also U347.15 (Q3), U359.4
- net IR8: now also U347.2 (Q0), U348.3 (I3a)
- net IR9: now also U347.7 (Q1), U348.13 (I3b)
- net MALA: now also U359.10, U359.13, U359.2
- net MAR8: now also U348.6 (I0a)
- net MAR9: now also U348.10 (I0b)
- net MDR8: now also U348.4 (I2a)
- net MDR9: now also U348.12 (I2b)
- net MEM10: now also U347.12 (D2)
- net MEM11: now also U347.13 (D3)
- net MEM8: now also U347.4 (D0)
- net MEM9: now also U347.5 (D1)
- net R43: now also U356.1
- net R46: now also U359.5
- net R49: now also U356.4
- net R5: now also U348.2 (S1)
- net R50: now also U358.2
- net SC2: now also U359.9
- net SC3: now also U359.12
- net SC4X: now also U359.1
- net SOOA: now also U355.9
- net ST5J: now also U345.8
- net STLD: now also U356.12
- net SZEA: now also U355.1
- net TRP13Q: now also U360.1
- net TRP14Q: now also U360.10
- net UR6: now also U349.2 (Q0)
- net UR7: now also U349.5 (Q1)
- net VCC1: now also U347.1 (~{Mr}), U347.16 (VCC), U348.16 (VCC), U349.1 (~{Mr}), U349.16 (VCC), U351.16 (VCC), U354.12
- net ~{A0}: now also U354.10
- net ~{ADRV}: now also U345.9
- net ~{AEQB}: now also U345.12, U354.1
- net ~{AEQO}: now also U355.8
- net ~{AEQZ}: now also U355.6
- net ~{ALS4}: now also U352.9
- net ~{ALS5}: now also U352.10
- net ~{AMAD2C}: now also U359.11
- net ~{AMAD3A}: now also U359.6
- net ~{AMAD3C}: now also U359.3
- net ~{AMS6}: now also U353.2
- net ~{APICYCRQ}: now also U345.1
- net ~{APIMAINC}: now also U345.3
- net ~{APIMALD}: now also U345.5
- net ~{CYIN}: now also U351.13 (Cn)
- net ~{CYY}: now also U351.11 (Cn+y)
- net ~{CYZ}: now also U351.9 (Cn+z)
- net ~{ENDER}: now also U357.13
- net ~{ENSER}: now also U357.12
- net ~{IR10}: now also U347.11 (~{Q2})
- net ~{IR8}: now also U347.3 (~{Q0})
- net ~{IRCLK}: now also U347.9 (Cp)
- net ~{MBLAST2}: now also U357.10
- net ~{MDCLK}: now also U356.6
- net ~{R6}: now also U353.13
- net ~{STALU3}: now also U356.11
- new net A10: U350.4, U353.8
- new net A11: U350.5
- new net A8: U350.1
- new net A9: U350.2
- new net B8: U348.7 (Za)
- new net B9: U348.9 (Zb)
- new net CYGX: U351.3 (G0)
- new net CYGY: U351.1 (G1)
- new net CYPX: U351.4 (P0)
- new net CYPY: U351.2 (P1)
- new net ENAMSK: U360.13
- new net ENDVCK: U358.4
- new net ENERS1: U357.8
- new net ENLOGIC: U354.13, U354.4
- new net ENST12CK: U358.12
- new net ER0SELB: U346.3
- new net SOOB: U352.6, U355.10
- new net SOOC: U350.6, U355.12
- new net SOOD: U355.13
- new net ST0D: U357.6
- new net SZEB: U352.8, U355.2
- new net SZEC: U350.8, U355.4
- new net SZED: U355.5
- new net UR10: U349.12 (Q4)
- new net UR11: U349.15 (Q5)
- new net UR8: U348.5 (I1a), U349.7 (Q2)
- new net UR9: U348.11 (I1b), U349.10 (Q3)
- new net ~{AGTHN}: U357.4
- new net ~{ALS10}: U350.12, U353.9
- new net ~{ALS11}: U350.13
- new net ~{ALS6}: U352.12, U353.1
- new net ~{ALS7}: U352.13, U353.4
- new net ~{ALS8}: U350.9
- new net ~{ALS9}: U350.10
- new net ~{AMAD1C}: U359.8
- new net ~{AMS10}: U353.10
- new net ~{AMS7}: U353.5
- new net ~{APIS0D}: U357.5
- new net ~{CYX}: U351.12 (Cn+x)
- new net ~{DMACLR}: U360.12
- new net ~{ENAPI}: U345.10
- new net ~{EXPCLR}: U360.6
- new net ~{FORSD}: U353.12
- new net ~{IICLR}: U360.8
- new net ~{IR11}: U347.14 (~{Q3})
- new net ~{IR13}: U358.1
- new net ~{IR9}: U347.6 (~{Q1})
- new net ~{LDST0}: U357.2
- new net ~{LGTHN}: U354.8, U357.1
- new net ~{MRCLK}: U356.8
- new net ~{R28LRF}: U357.9
- new net ~{R31A}: U346.1
- new net ~{ST12CK}: U358.11
- new net ~{ST2CK}: U358.6
- new net ~{TRP13A}: U360.3, U360.9
- new net ~{TRP14A}: U360.2, U360.4
- new net ~{URCLK}: U349.9 (Cp), U356.3
- no-connect marks 150 -> 168

Commit message: Finished Column 9 on AU2
Parts:
- added C6: C_Polarized, symbol Device:C_Polarized
- added U361: 74157N, symbol 74xx:74LS157
- added U362, U363, U364, U367, U369, U373: 74151N, symbol 74xx:74LS151
- added U365, U375: 74S00N, symbol 74xx:7400
- added U366: 74181, symbol 74xx:74LS181
- added U368: 74163N, symbol 74xx:74LS163
- added U370, U374: 7408N, symbol 74xx:74LS08
- added U371: 7404N, symbol 74xx:74LS04
- added U372: 74H52N, symbol TI980A:74H52N
- added U376: 7451N, symbol TI980A:7451N
- added U377: 74H04N, symbol 74xx:74LS04
- added U378: 7432N, symbol 74xx:74LS32
Connections:
- net A10: now also U366.23 (A1)
- net A11: now also U365.6, U366.2 (A0)
- net A8: now also U365.3, U366.19 (A3)
- net A9: now also U365.11, U366.21 (A2)
- net AEQB: now also U366.14 (A=B)
- net ALU0: now also U375.12
- net ALU0T: now also U372.5
- net ALU10: now also U366.10 (F1)
- net ALU11: now also U366.9 (F0)
- net ALU14: now also U372.11
- net ALU15A: now also U372.13
- net ALU4: now also U361.3 (I1a), U370.1
- net ALU5: now also U361.6 (I1b)
- net ALU6: now also U361.13 (I1d)
- net ALU7: now also U361.10 (I1c)
- net ALU8: now also U366.13 (F3)
- net ALU9: now also U366.11 (F2), U370.9
- net ALUM: now also U366.8 (M), U371.4
- net ALUS0: now also U366.6 (S0)
- net ALUS1: now also U366.5 (S1)
- net ALUS2: now also U366.4 (S2)
- net ALUS3: now also U366.3 (S3)
- net AMAD1: now also U362.9 (S2), U363.9 (S2), U364.9 (S2), U367.9 (S2), U369.9 (S2)
- net AMAD2: now also U362.10 (S1), U363.10 (S1), U364.10 (S1), U367.10 (S1), U369.10 (S1)
- net AMAD3: now also U362.11 (S0), U363.11 (S0), U364.11 (S0), U367.11 (S0), U369.11 (S0)
- net AR1: now also U369.4 (I0)
- net AXB0: now also U371.9
- net B8: now also U366.18 (B3)
- net B9: now also U366.20 (B2)
- net C0: now also U368.6 (D3)
- net C1: now also U368.5 (D2)
- net C2: now also U368.4 (D1)
- net C3: now also U368.3 (D0)
- net CYGY: now also U366.17 (Y)
- net CYPY: now also U366.15 (X)
- net ENERS0: now also U378.5
- net ENERS1: now also U378.4
- net ENLOGIC: now also U371.2
- net ENNSC0: now also U377.3
- net ENNSC15: now also U377.5
- net ENSRINC: now also U368.7 (CEP)
- net ER0SELA: now also U371.13, U374.13
- net ER0SELB: now also U372.12
- net ER0SELD: now also U372.2
- net ER1: now also U369.3 (I1)
- net ERIN0: now also U372.8
- net ERLD: now also U378.6
- net EXPADR12: now also U370.4
- net GND: now also U362.8 (GND), U363.8 (GND), U364.8 (GND), U366.12 (GND), U367.8 (GND), U368.8 (GND), U369.8 (GND), U373.8 (GND)
- net GND1: now also C6.2, U361.8 (GND)
- net IFLAGQ: now also U374.10
- net INHMSA: now also U369.7 (~{E})
- net IOUT4: now also U361.4 (Za)
- net IOUT5: now also U361.7 (Zb)
- net IOUT6: now also U361.12 (Zd)
- net IOUT7: now also U361.9 (Zc)
- net IR10: now also U373.11 (S0), U375.1
- net IR10T: now also U377.10
- net IR11: now also U364.13 (I6), U376.1, U376.9
- net IR12T: now also U377.2
- net IR13: now also U375.9
- net IR3: now also U376.10
- net IR7: now also U367.13 (I6)
- net IR8: now also U363.13 (I6), U373.9 (S2), U376.13
- net IR9: now also U362.13 (I6), U373.10 (S1), U375.4
- net IR9T: now also U377.12
- net MEM11: now also U364.14 (I5)
- net MEM7: now also U367.14 (I5)
- net MEM8: now also U363.14 (I5)
- net MEM9: now also U362.14 (I5)
- net MRESETQA: now also U378.10
- net PC1: now also U369.12 (I7)
- net PC4: now also U361.2 (I0a)
- net PC5: now also U361.5 (I0b)
- net PNL11: now also U364.15 (I4)
- net PNL7: now also U367.15 (I4)
- net PNL8: now also U363.15 (I4)
- net PNL9: now also U362.15 (I4)
- net R31: now also U371.11, U374.12, U374.4
- net R46: now also U375.2, U375.5
- net R47: now also U375.10
- net ST11: now also U364.4 (I0)
- net ST15KA: now also U378.9
- net ST2: now also U373.1 (I3)
- net ST7: now also U367.4 (I0)
- net ST8: now also U363.4 (I0)
- net ST9: now also U362.4 (I0)
- net STLD: now also U370.10, U370.2
- net TRP14Q: now also U377.9
- net VCC1: now also C6.1, U361.16 (VCC), U362.16 (VCC), U363.16 (VCC), U364.16 (VCC), U366.24 (VCC), U367.16 (VCC), U368.1 (~{MR}), U368.16 (VCC), U369.16 (VCC), U373.16 (VCC), U375.13
- net ~{ALS0}: now also U371.5
- net ~{ALS11}: now also U365.4
- net ~{ALS8}: now also U365.1
- net ~{ALS9}: now also U365.12
- net ~{AMAD2A}: now also U375.3
- net ~{AMS1}: now also U369.6 (~{Z})
- net ~{AMS7}: now also U367.6 (~{Z})
- net ~{AXB0}: now also U371.8
- net ~{CYX}: now also U366.7 (Cn)
- net ~{DP11}: now also U364.3 (I1)
- net ~{DP7}: now also U367.3 (I1)
- net ~{DP8}: now also U363.3 (I1)
- net ~{DP9}: now also U362.3 (I1)
- net ~{ENARITH}: now also U370.12
- net ~{ENIOUT}: now also U361.15 (E)
- net ~{ENLOGIC}: now also U370.13, U371.1
- net ~{ENNSC0}: now also U377.4
- net ~{ENNSC15}: now also U377.6
- net ~{ENSRLOAD}: now also U368.9 (~{PE})
- net ~{GCLKC:1}: now also U368.2 (CP)
- net ~{INDSK}: now also U373.6 (~{Z})
- net ~{IR10}: now also U377.11
- net ~{IR9}: now also U377.13
- net ~{LRFENER}: now also U374.2
- net ~{PCOUTA}: now also U361.1 (S)
- net ~{R13}: now also U371.3
- net ~{R28LRF}: now also U374.3
- net ~{R28}: now also U374.1
- net ~{R31A}: now also U371.10, U372.4
- net ~{SETBIT7}: now also U367.2 (I2)
- net ~{TRP14A}: now also U377.8
- new net A13: U365.8
- new net ALS0: U371.6
- new net B10: U366.22 (B1)
- new net B11: U366.1 (B0)
- new net BR1: U369.13 (I6)
- new net ER0SELC: U372.10, U374.11
- new net ER0SELE: U372.1, U374.6
- new net EXPTRAP: U370.5
- new net LR1: U369.14 (I5)
- new net MR1: U369.1 (I3)
- new net PC6: U361.14 (I0d)
- new net PC7: U361.11 (I0c)
- new net PCS11: U364.12 (I7)
- new net PCS7: U367.12 (I7)
- new net PCS8: U363.12 (I7)
- new net PCS9: U362.12 (I7)
- new net PEMSKJ: U374.8
- new net SEQ: U373.3 (I1), U378.12, U378.2
- new net SGE: U373.15 (I4), U378.3
- new net SGT: U373.2 (I2), U378.1
- new net SLE: U373.13 (I6), U378.11
- new net SLT: U373.4 (I0), U378.13
- new net SR0: U368.11 (Q3)
- new net SR1: U368.12 (Q2), U369.15 (I4)
- new net SR2: U368.13 (Q1)
- new net SR3: U368.14 (Q0)
- new net SRCR3: U368.10 (CET)
- new net SRMAX: U368.15 (TC)
- new net ST15: U374.9
- new net ST15K: U378.8
- new net ST4D: U370.3
- new net ST9D: U370.8
- new net TRAP11: U364.1 (I3)
- new net TRAP12: U370.6
- new net TRAP7: U367.1 (I3)
- new net TRAP8: U363.1 (I3)
- new net TRAP9: U362.1 (I3)
- new net XR1: U369.2 (I2)
- new net ~{ALS13}: U365.9
- new net ~{ALU0A}: U375.11
- new net ~{AMAD0B}: U362.7 (~{E}), U363.7 (~{E}), U364.7 (~{E}), U367.7 (~{E})
- new net ~{AMAD1A}: U375.6
- new net ~{AMAD1B}: U375.8
- new net ~{AMS11}: U364.6 (~{Z}), U365.5
- new net ~{AMS13}: U365.10
- new net ~{AMS8}: U363.6 (~{Z}), U365.2
- new net ~{AMS9}: U362.6 (~{Z}), U365.13
- new net ~{ENINDSK}: U373.7 (~{E})
- new net ~{ENST01}: U370.11
- new net ~{ER0SELA}: U371.12, U372.3, U374.5
- new net ~{IR12}: U377.1
- new net ~{SEQ}: U373.14 (I5)
- new net ~{SETBIT11}: U364.2 (I2)
- new net ~{SETBIT8}: U363.2 (I2)
- new net ~{SETBIT9}: U362.2 (I2)
- new net ~{SKSELOG2}: U376.8
- new net ~{ST2}: U373.12 (I7)
- no-connect marks 168 -> 181
