File: TI980A-Arithmetic-Unit/AU2.kicad_sch (KiCad schematic)
At the start: 234 parts, among them U15 74H40N, U16 74H40N, U17 74H40N, U18 74H11N, U19 74H04N, U20 74H40N, U231 7451N, U232 74H101, U233 74187, U234 74187, U235 74187, U236 74187, U237 74H04N, U238 74187, U239 74187, U240 74187, U241 74187, U242 74187, U243 7430N, U244 7430N, U245 74H11N, U246 74H00N, U247 74H74N, U248 74187, U249 74187, U250 74187, U251 74187, U252 74187, U253 7451N, U254 7437N, U255 74S65N, U256 74H00N, U257 74H74N, U258 74H74N, U259 74H74N, U260 7410N, U261 7420N, U262 74H21N, U263 74H11N, U264 7474N, U265 74H04N, U266 74153N, U267 74H20N, U268 7474N, U269 74181, U270 74153, U271 74153, U272 74H11N, U273 74174N, U274 74S10N, U275 7442N, U276 74H51N, U277 74H11N, U278 74H51N, U279 74153N, U280 74151N, U281 74151N, U282 74151N, U283 74151N, U284 74151N, U285 74153N, U286 74163N, U287 74153N, U288 74H51N, U289 74H51N, U290 74H00N, U291 74H00N, U292 74H11N, U293 74153N, U294 74163N, U295 74153N, U296 7442N, U297 74H00N, U298 74H21N, U299 74153N, U300 74H04N, U301 74H103N, U302 7410N, U303 74H51N, U304 7442N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

Commit message: Finished Column 10 on AU2
Parts:
- added R148, R149, R150, R151, R152, R153, R154, R155: R, symbol Device:R
- added U379: 7442N, symbol 74xx:74LS42
- added U380, U393: 7408N, symbol 74xx:74LS08
- added U381, U385, U388, U390, U391, U392: 74151N, symbol 74xx:74LS151
- added U382, U387, U389: 74174N, symbol 74xx:74LS174
- added U383, U386: 74163N, symbol 74xx:74LS163
- added U384: 74H21N, symbol 74xx:74LS21
- added U394: 7404N, symbol 74xx:74LS04
- added U395: 74H11N, symbol 74xx:74LS11
- added U396: 74S40N, symbol 74xx:74LS40
- added U397: 74H20N, symbol 74xx:74LS20
- added U398: 74175N, symbol 74xx:74LS175
Connections:
- net A13: now also U384.2
- net ALS0: now also U391.1 (I3)
- net ALU0T: now also U396.8
- net ALU15: now also U395.5
- net ALU15A: now also U395.6
- net ALUEQZ: now also U395.8
- net ALUZ115: now also U395.11
- net AMAD1: now also U381.9 (S2), U385.9 (S2), U388.9 (S2), U390.9 (S2), U396.6
- net AMAD2: now also U381.10 (S1), U385.10 (S1), U388.10 (S1), U390.10 (S1)
- net AMAD3: now also U381.11 (S0), U385.11 (S0), U388.11 (S0), U390.11 (S0)
- net AR0: now also U390.4 (I0)
- net AR5: now also U388.4 (I0)
- net AR7: now also U385.4 (I0)
- net C0: now also U387.3 (D0), U389.3 (D0)
- net C1: now also U387.4 (D1), U389.4 (D1)
- net C2: now also U387.6 (D2), U389.6 (D2)
- net C3: now also U387.11 (D3), U389.11 (D3)
- net C4: now also U383.6 (D3), U386.6 (D3), U387.13 (D4), U389.13 (D4)
- net C5: now also U383.5 (D2), U386.5 (D2), U387.14 (D5), U389.14 (D5)
- net C6: now also U383.4 (D1), U386.4 (D1)
- net C7: now also U383.3 (D0), U386.3 (D0)
- net ENPCINC: now also U383.7 (CEP)
- net ENSRINC: now also U386.7 (CEP)
- net ENST12CK: now also U397.6
- net ER0: now also U390.3 (I1)
- net EXPADR10: now also R152.2, U380.12
- net EXPADR11: now also R150.2, U380.9
- net EXPADR12: now also R148.2
- net EXPADR8: now also U380.1
- net EXPADR9: now also U380.4
- net EXPTRAP: now also U380.10, U380.13, U380.2, U380.5, U393.6
- net GND: now also U379.8 (GND), U381.8 (GND), U382.8 (GND), U383.8 (GND), U385.8 (GND), U386.8 (GND), U387.8 (GND), U388.8 (GND), U389.8 (GND), U390.8 (GND), U391.8 (GND), U392.8 (GND), U398.8 (GND)
- net INHMSA: now also U385.7 (~{E}), U388.7 (~{E}), U390.7 (~{E})
- net IR0: now also U398.2 (Q0)
- net IR1: now also U398.7 (Q1)
- net IR10: now also U381.13 (I6), U391.11 (S0)
- net IR13: now also U379.13 (A2)
- net IR14: now also U379.14 (A1)
- net IR15: now also U379.15 (A0)
- net IR2: now also U398.10 (Q2)
- net IR3: now also U392.9 (S2), U398.15 (Q3)
- net IR5: now also U397.9
- net IR6: now also U393.13, U397.10
- net IR7: now also U397.12
- net IR8: now also U391.9 (S2)
- net IR9: now also U391.10 (S1)
- net LR1: now also U389.5 (Q1)
- net MEM0: now also U398.4 (D0)
- net MEM1: now also U398.5 (D1)
- net MEM10: now also U381.14 (I5)
- net MEM2: now also U398.12 (D2)
- net MEM3: now also U398.13 (D3)
- net MR1: now also U387.5 (Q1)
- net PC0: now also U390.12 (I7)
- net PC4: now also U383.11 (Q3)
- net PC5: now also U383.12 (Q2), U388.12 (I7)
- net PC6: now also U382.3 (D0), U383.13 (Q1)
- net PC7: now also U382.4 (D1), U383.14 (Q0), U385.12 (I7)
- net PCCR3: now also U383.15 (TC)
- net PCS11: now also U382.15 (Q5)
- net PCS6: now also U382.2 (Q0)
- net PCS7: now also U382.5 (Q1)
- net PCS8: now also U382.7 (Q2)
- net PCS9: now also U382.10 (Q3)
- net PNL10: now also U381.15 (I4)
- net R51: now also U397.13
- net R54: now also U394.11
- net SEQ: now also U394.13
- net SOOD: now also U384.6
- net SR0: now also U390.15 (I4)
- net SRCR3: now also U386.15 (TC)
- net ST10: now also U381.4 (I0)
- net ST3: now also U392.1 (I3)
- net ST6J: now also U393.3
- net SZED: now also U384.8
- net TRAP11: now also U380.8
- net TRAP8: now also U380.3
- net TRAP9: now also U380.6
- net VCC1: now also R148.1, R149.1, R150.1, R151.1, R152.1, R153.1, R154.1, R155.1, U379.16 (VCC), U381.16 (VCC), U382.1 (~{Mr}), U382.16 (VCC), U383.1 (~{MR}), U383.16 (VCC), U385.16 (VCC), U386.1 (~{MR}), U386.16 (VCC), U387.1 (~{Mr}), U387.16 (VCC), U388.16 (VCC), U389.1 (~{Mr}), U389.16 (VCC), U390.16 (VCC), U391.16 (VCC), U392.16 (VCC), U395.13, U395.2, U395.3, U395.4, U395.9, U396.10, U396.12, U396.13, U398.1 (~{Mr}), U398.16 (VCC)
- net ~{ADRV}: now also U393.1
- net ~{AEQO}: now also U391.14 (I5)
- net ~{AEQZ}: now also U391.15 (I4)
- net ~{ALS0}: now also U390.6 (~{Z}), U391.12 (I7)
- net ~{ALS13}: now also U384.10
- net ~{ALS5}: now also U388.6 (~{Z})
- net ~{ALS7}: now also U385.6 (~{Z})
- net ~{ALU0A}: now also U396.9
- net ~{ALU0}: now also U395.10
- net ~{AMAD0A}: now also U395.1
- net ~{AMAD0B}: now also U381.7 (~{E}), U395.12
- net ~{AMAD1A}: now also U396.1
- net ~{AMAD1B}: now also U396.2
- net ~{AMAD1C}: now also U396.4
- net ~{AMS10}: now also U381.6 (~{Z})
- net ~{BITSK}: now also U392.6 (~{Z})
- net ~{DMACLR}: now also U397.4
- net ~{DP10}: now also R149.2, U381.3 (I1)
- net ~{DP11}: now also R154.2
- net ~{DP7}: now also R155.2
- net ~{DP8}: now also R153.2
- net ~{DP9}: now also R151.2
- net ~{ENPCLOAD}: now also U383.9 (~{PE})
- net ~{ENSRLOAD}: now also U386.9 (~{PE})
- net ~{EXPCLR}: now also U397.2
- net ~{FORSD}: now also U397.8
- net ~{GCLKC:1}: now also U383.2 (CP), U386.2 (CP)
- net ~{IICLR}: now also U397.5
- net ~{IR11}: now also U393.10
- net ~{IR12}: now also U379.12 (A3)
- net ~{IRCLK}: now also U398.9 (Cp)
- net ~{LRCLK}: now also U389.9 (Cp)
- net ~{MRCLK}: now also U387.9 (Cp)
- net ~{PCSCLK}: now also U382.9 (Cp)
- net ~{R2}: now also U396.5
- net ~{REGSK}: now also U391.6 (~{Z})
- net ~{SEQ}: now also U394.12
- net ~{SETBIT11}: now also U379.4 (3)
- net ~{SETBIT8}: now also U379.1 (0)
- net ~{SETBIT9}: now also U379.2 (1)
- net ~{TRP13A}: now also U393.4
- net ~{TRP14A}: now also U393.5
- new net A12: U384.1
- new net A14: U384.4
- new net A15: U384.5, U391.2 (I2)
- new net AEQD: U391.3 (I1)
- new net AEQZ: U391.4 (I0)
- new net BITEQ0: U392.14 (I5)
- new net BITEQO: U394.1
- new net BR0: U390.13 (I6)
- new net BR5: U388.13 (I6)
- new net BR7: U385.13 (I6)
- new net ER5: U388.3 (I1)
- new net ER7: U385.3 (I1)
- new net ERZ115: U394.6
- new net INSTV: U393.2
- new net LR0: U389.2 (Q0), U390.14 (I5)
- new net LR2: U389.7 (Q2)
- new net LR3: U389.10 (Q3)
- new net LR4: U389.12 (Q4)
- new net LR5: U388.14 (I5), U389.15 (Q5)
- new net LR7: U385.14 (I5)
- new net MR0: U387.2 (Q0), U390.1 (I3)
- new net MR2: U387.7 (Q2)
- new net MR3: U387.10 (Q3)
- new net MR4: U387.12 (Q4)
- new net MR5: U387.15 (Q5), U388.1 (I3)
- new net MR7: U385.1 (I3)
- new net PC10: U382.13 (D4)
- new net PC11: U382.14 (D5)
- new net PC8: U382.6 (D2)
- new net PC9: U382.11 (D3)
- new net PCCR2: U383.10 (CET)
- new net PCS10: U381.12 (I7), U382.12 (Q4)
- new net SELSKA: U392.11 (S0)
- new net SELSKB: U392.10 (S1), U393.11
- new net SR4: U386.11 (Q3)
- new net SR5: U386.12 (Q2), U388.15 (I4)
- new net SR6: U386.13 (Q1)
- new net SR7: U385.15 (I4), U386.14 (Q0)
- new net SRCR2: U386.10 (CET)
- new net SSNEQ: U392.3 (I1), U394.3
- new net TOFB0: U394.9
- new net TRAP10: U380.11, U381.1 (I3)
- new net XR0: U390.2 (I2)
- new net XR5: U388.2 (I2)
- new net XR7: U385.2 (I2)
- new net ~{ALS12}: U384.9
- new net ~{ALS14}: U384.12
- new net ~{ALS15}: U384.13, U391.13 (I6)
- new net ~{BITEEQO}: U394.2
- new net ~{BITEQ0}: U392.15 (I4)
- new net ~{ENREGSK}: U391.7 (~{E})
- new net ~{ERZ115}: U394.5
- new net ~{IR0}: U398.3 (~{Q0})
- new net ~{IR1}: U398.6 (~{Q1})
- new net ~{IR2}: U398.11 (~{Q2})
- new net ~{IR3}: U393.12, U398.14 (~{Q3})
- new net ~{IR6O11}: U392.7 (~{E}), U393.8
- new net ~{IR6}: U393.9
- new net ~{R54A}: U394.10
- new net ~{SETBIT10}: U379.3 (2), U381.2 (I2)
- new net ~{SETBIT12}: U379.5 (4)
- new net ~{SETBIT13}: U379.6 (5)
- new net ~{SETBIT14}: U379.7 (6)
- new net ~{SETBIT15}: U379.9 (7)
- new net ~{SLTD}: U397.1
- new net ~{SSNEQ}: U392.4 (I0), U394.4
- new net ~{ST3}: U392.2 (I2)
- new net ~{TOFB0}: U394.8
- no-connect marks 181 -> 191
