File: TI980A-Arithmetic-Unit/AU2.kicad_sch (KiCad schematic)
At the start: 262 parts, among them U15 74H40N, U16 74H40N, U17 74H40N, U18 74H11N, U19 74H04N, U20 74H40N, U231 7451N, U232 74H101, U233 74187, U234 74187, U235 74187, U236 74187, U237 74H04N, U238 74187, U239 74187, U240 74187, U241 74187, U242 74187, U243 7430N, U244 7430N, U245 74H11N, U246 74H00N, U247 74H74N, U248 74187, U249 74187, U250 74187, U251 74187, U252 74187, U253 7451N, U254 7437N, U255 74S65N, U256 74H00N, U257 74H74N, U258 74H74N, U259 74H74N, U260 7410N, U261 7420N, U262 74H21N, U263 74H11N, U264 7474N, U265 74H04N, U266 74153N, U267 74H20N, U268 7474N, U269 74181, U270 74153, U271 74153, U272 74H11N, U273 74174N, U274 74S10N, U275 7442N, U276 74H51N, U277 74H11N, U278 74H51N, U279 74153N, U280 74151N, U281 74151N, U282 74151N, U283 74151N, U284 74151N, U285 74153N, U286 74163N, U287 74153N, U288 74H51N, U289 74H51N, U290 74H00N, U291 74H00N, U292 74H11N, U293 74153N, U294 74163N, U295 74153N, U296 7442N, U297 74H00N, U298 74H21N, U299 74153N, U300 74H04N, U301 74H103N, U302 7410N, U303 74H51N, U304 7442N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

Commit message: Finished Column 11 on AU2
Parts:
- added R156, R157, R158, R159, R160, R161, R162, R163, R164, R165, R166, R167, R168, R169, R170, R171: R, symbol Device:R
- added U399: 7451N, symbol TI980A:7451N
- added U400: 7432N, symbol 74xx:74LS32
- added U401, U402, U405, U407: 74151N, symbol 74xx:74LS151
- added U403: 74S00N, symbol 74xx:7400
- added U404: 74181, symbol 74xx:74LS181
- added U406: 74174N, symbol 74xx:74LS174
- added U408: 7400N, symbol 74xx:7400
- added U409: 74H55N, symbol TI980A:74H55N
- added U410: 74H30N, symbol 74xx:74LS30
- added U411: 74194N, symbol 74xx:74LS194
- added U412: 7486N, symbol 74xx:74LS86
- added U413: 7408N, symbol 74xx:74LS08
Connections:
- net A0: now also U409.2, U412.10, U412.13, U412.4
- net A1: now also U412.12
- net A12: now also U403.3, U404.19 (A3)
- net A13: now also U404.21 (A2)
- net A14: now also U403.11, U404.23 (A1)
- net A15: now also U403.8, U404.2 (A0), U408.4
- net AEQB: now also U404.14 (A=B)
- net ALU0T: now also U409.13
- net ALU12: now also U404.13 (F3), U411.3 (P0)
- net ALU13: now also U404.11 (F2), U411.4 (P1)
- net ALU14: now also U404.10 (F1), U411.5 (P2)
- net ALU15: now also U404.9 (F0), U411.6 (P3)
- net ALUM: now also U404.8 (M)
- net ALUS0: now also U404.6 (S0)
- net ALUS1: now also U404.5 (S1)
- net ALUS2: now also U404.4 (S2)
- net ALUS3: now also U404.3 (S3)
- net AMAD1: now also U401.9 (S2), U402.9 (S2), U405.9 (S2), U407.9 (S2)
- net AMAD2: now also U401.10 (S1), U402.10 (S1), U405.10 (S1), U407.10 (S1)
- net AMAD3: now also U401.11 (S0), U402.11 (S0), U405.11 (S0), U407.11 (S0)
- net AR16: now also U413.13
- net AR4: now also U405.4 (I0)
- net AXB0: now also U412.6
- net B0: now also U412.2, U412.9
- net BITEQO: now also U408.3
- net BR0: now also U406.2 (Q0)
- net BR1: now also U406.5 (Q1)
- net BR5: now also U406.15 (Q5)
- net BYTEINC: now also U400.13, U413.12
- net C0: now also U406.3 (D0)
- net C1: now also U406.4 (D1)
- net C2: now also U406.6 (D2)
- net C3: now also U406.11 (D3)
- net C4: now also U406.13 (D4)
- net C5: now also U406.14 (D5)
- net CYGX: now also U404.17 (Y)
- net CYPX: now also U404.15 (X)
- net ENARINC: now also U413.11
- net ENASOV: now also U409.10, U409.4
- net ENERS0: now also U411.9 (S0)
- net ENERS1: now also U411.10 (S1)
- net ENLSOV: now also U408.13
- net ER14: now also U411.13 (Q2)
- net ER15: now also U411.12 (Q3)
- net ER15IN: now also U411.7 (Dsl)
- net EXPADR13: now also R161.2
- net EXPADR9: now also R167.2
- net GND: now also U401.1 (I3), U401.8 (GND), U402.8 (GND), U404.12 (GND), U405.8 (GND), U406.8 (GND), U407.8 (GND), U411.8 (GND)
- net INHMSA: now also U405.7 (~{E}), U407.7 (~{E})
- net INVB0: now also U412.1
- net IR12: now also U399.13, U402.13 (I6)
- net IR13: now also U399.9
- net IR15: now also U401.13 (I6)
- net IR7: now also U408.10
- net LR3: now also U407.14 (I5)
- net LR4: now also U405.14 (I5)
- net MEM12: now also U402.14 (I5)
- net MEM15: now also U401.14 (I5)
- net MR3: now also U407.1 (I3)
- net MR4: now also U405.1 (I3)
- net PC3: now also U407.12 (I7)
- net PC4: now also U405.12 (I7)
- net PNL12: now also U402.15 (I4)
- net PNL15: now also U401.15 (I4)
- net R22: now also R170.2
- net R37: now also R160.2, U400.12
- net R51: now also R169.2
- net R54: now also U408.5
- net SEQ: now also U413.6
- net SGT: now also U413.8
- net SLT: now also U413.3
- net SR3: now also U407.15 (I4)
- net SR4: now also U405.15 (I4)
- net ST0: now also U413.9
- net ST1: now also U413.5
- net ST12: now also U402.4 (I0)
- net ST15: now also U401.4 (I0)
- net TOFB0: now also U409.3, U412.3, U412.5
- net TRAP12: now also U402.1 (I3)
- net VCC1: now also R156.1, R157.1, R158.1, R159.1, R160.1, R161.1, R162.1, R163.1, R164.1, R165.1, R166.1, R167.1, R168.1, R169.1, R170.1, R171.1, U401.16 (VCC), U402.16 (VCC), U404.24 (VCC), U405.16 (VCC), U406.1 (~{Mr}), U406.16 (VCC), U407.16 (VCC), U410.12, U410.2, U411.1 (Mr), U411.16 (VCC)
- net ~{A0EQB0}: now also U412.8
- net ~{A0}: now also U409.12
- net ~{AGTHN}: now also U336.8
- net ~{ALS12}: now also U403.1
- net ~{ALS14}: now also U403.12
- net ~{ALS15}: now also U403.9
- net ~{ALS3}: now also U407.6 (~{Z})
- net ~{ALS4}: now also U405.6 (~{Z})
- net ~{ALU0}: now also U409.1
- net ~{ALUEQ8K}: now also U410.4
- net ~{AMAD0B}: now also U401.7 (~{E}), U402.7 (~{E})
- net ~{APIS0D}: now also U400.3
- net ~{APIST0}: now also U400.1
- net ~{BIT1}: now also U408.1
- net ~{CYIN}: now also U404.7 (Cn)
- net ~{DP12}: now also R157.2, U402.3 (I1)
- net ~{DP13}: now also R156.2
- net ~{DP14}: now also R158.2
- net ~{DP15}: now also R159.2, U401.3 (I1)
- net ~{DP5}: now also R162.2
- net ~{DP6}: now also R163.2
- net ~{ENAPI}: now also U400.2
- net ~{ENINDSK}: now also U408.8
- net ~{GCLKC:1}: now also U411.11 (Cp)
- net ~{IR6O11}: now also U408.9
- net ~{R17}: now also R171.2
- net ~{R19}: now also R166.2
- net ~{R33}: now also R165.2
- net ~{R36}: now also R164.2
- net ~{R44}: now also R168.2
- net ~{SETBIT12}: now also U402.2 (I2)
- net ~{SETBIT15}: now also U401.2 (I2)
- net ~{SNS1}: now also U399.1
- net ~{SNS2}: now also U399.10
- net ~{TOFB0}: now also U409.11
- new net A0XA1A: U408.12, U412.11
- new net AR3: U407.4 (I0)
- new net B12: U404.18 (B3)
- new net B13: U404.20 (B2)
- new net B14: U404.22 (B1)
- new net B15: U404.1 (B0)
- new net BR2: U406.7 (Q2)
- new net BR3: U406.10 (Q3), U407.13 (I6)
- new net BR4: U405.13 (I6), U406.12 (Q4)
- new net ENXRINC: U400.11
- new net ER11: U411.2 (Dsr)
- new net ER12: U411.15 (Q0)
- new net ER13: U411.14 (Q1)
- new net ER3: U407.3 (I1)
- new net ER4: U405.3 (I1)
- new net PCS12: U402.12 (I7)
- new net PCS15: U401.12 (I7)
- new net ST2D: U410.8
- new net XR3: U407.2 (I2)
- new net XR4: U405.2 (I2)
- new net ~{AMS12}: U402.6 (~{Z}), U403.2
- new net ~{AMS14}: U403.13
- new net ~{AMS15}: U401.6 (~{Z}), U403.10
- new net ~{APIS2D}: U410.11
- new net ~{AR15ER1}: U408.6
- new net ~{ASOV}: U409.8, U410.1
- new net ~{BIT2}: U408.2
- new net ~{BRCLK}: U406.9 (Cp)
- new net ~{DIVOV}: U410.5
- new net ~{LSOV}: U408.11, U410.3
- new net ~{SSNEQ1}: U399.8
- new net ~{ST0}: U413.1, U413.4
- new net ~{ST1}: U413.10, U413.2
- new net ~{ST2LD}: U410.6
- no-connect marks 191 -> 212

Commit message: Finished Column 12 on AU2
Parts:
- added U414: 74174N, symbol 74xx:74LS174
- added U415: 7451N, symbol TI980A:7451N
- added U416, U420, U422, U423: 74151N, symbol 74xx:74LS151
- added U417, U428: 74175N, symbol 74xx:74LS175
- added U418, U419: 74153N, symbol 74xx:74LS153
- added U421, U429: 74163N, symbol 74xx:74LS163
- added U424: 74194N, symbol 74xx:74LS194
- added U425: 7410N, symbol 74xx:74LS10
- added U426: 7400N, symbol 74xx:7400
- added U427, U430: 74H103N, symbol TI980A:74H103N
- added U431: 7474N, symbol 74xx:74LS74
- added U432: 74H04N, symbol 74xx:74LS04
Connections:
- net AEQB: now also U426.4
- net AEQZ: now also U432.2
- net ALU1: now also U426.9
- net ALU4: now also U424.3 (P0)
- net ALU5: now also U424.4 (P1)
- net ALU6: now also U424.5 (P2)
- net ALU7: now also U424.6 (P3)
- net AMAD1: now also U416.9 (S2), U422.9 (S2), U423.9 (S2)
- net AMAD2: now also U416.10 (S1), U422.10 (S1), U423.10 (S1)
- net AMAD3: now also U416.11 (S0), U422.11 (S0), U423.11 (S0)
- net AR2: now also U423.4 (I0)
- net AR6: now also U422.4 (I0)
- net ARCR2: now also U429.15 (TC)
- net B12: now also U418.7 (Za)
- net B13: now also U418.9 (Zb)
- net B14: now also U419.7 (Za)
- net B15: now also U419.9 (Zb)
- net BMAD1: now also U418.14 (S0), U419.14 (S0)
- net BR2: now also U423.13 (I6)
- net C10: now also U429.4 (D1)
- net C11: now also U429.3 (D0)
- net C4: now also U421.6 (D3)
- net C5: now also U421.5 (D2)
- net C6: now also U421.4 (D1)
- net C7: now also U421.3 (D0)
- net C8: now also U429.6 (D3)
- net C9: now also U429.5 (D2)
- net CPUCR: now also U432.8
- net ENARINC: now also U429.7 (CEP)
- net ENERS0: now also U424.9 (S0)
- net ENERS1: now also U424.10 (S1)
- net ENXRINC: now also U421.7 (CEP)
- net ER3: now also U424.2 (Dsr)
- net ER4: now also U424.15 (Q0)
- net ER5: now also U424.14 (Q1)
- net ER7: now also U424.12 (Q3)
- net GCLKA:1: now also U425.5
- net GCLKB:1: now also U427.5 (CLK), U430.1 (CLK), U430.5 (CLK)
- net GND: now also U414.13 (D4), U414.14 (D5), U414.8 (GND), U416.4 (I0), U416.8 (GND), U417.8 (GND), U418.8 (GND), U419.8 (GND), U420.8 (GND), U421.8 (GND), U422.8 (GND), U423.8 (GND), U424.8 (GND), U428.8 (GND), U429.8 (GND)
- net INAQ: now also U425.3
- net INHMSA: now also U422.7 (~{E}), U423.7 (~{E})
- net INHMSB: now also U418.1 (Ea), U418.15 (Eb), U419.1 (Ea), U419.15 (Eb)
- net INSTV: now also U432.6
- net IR12: now also U417.2 (Q0), U418.3 (I3a)
- net IR13: now also U416.13 (I6), U417.7 (Q1), U418.13 (I3b), U420.9 (S2)
- net IR14: now also U415.13, U417.10 (Q2), U419.3 (I3a), U420.10 (S1)
- net IR14T: now also U432.10
- net IR15: now also U415.9, U417.15 (Q3), U419.13 (I3b), U420.11 (S0)
- net IR15T: now also U432.12
- net IR4: now also U428.2 (Q0)
- net IR5: now also U428.7 (Q1)
- net IR6: now also U425.2, U428.10 (Q2)
- net IR7: now also U428.15 (Q3)
- net LR2: now also U423.14 (I5)
- net MAR12: now also U418.6 (I0a)
- net MAR13: now also U418.10 (I0b)
- net MAR14: now also U419.6 (I0a)
- net MAR15: now also U419.10 (I0b)
- net MEM12: now also U414.3 (D0), U417.4 (D0)
- net MEM13: now also U414.4 (D1), U416.14 (I5), U417.5 (D1)
- net MEM14: now also U414.6 (D2), U417.12 (D2)
- net MEM15: now also U414.11 (D3), U417.13 (D3)
- net MEM4: now also U428.4 (D0)
- net MEM5: now also U428.5 (D1)
- net MEM6: now also U428.12 (D2)
- net MEM7: now also U428.13 (D3)
- net MPERR: now also U427.7 (J)
- net MR2: now also U423.1 (I3)
- net MRESETQA: now also U430.3 (K)
- net PC2: now also U423.12 (I7)
- net PC6: now also U422.12 (I7)
- net PNL13: now also U416.15 (I4)
- net R5: now also U418.2 (S1), U419.2 (S1)
- net SR2: now also U423.15 (I4)
- net SR6: now also U422.15 (I4)
- net SSNEQ: now also U426.3
- net ST11: now also U431.9 (Q)
- net ST14: now also U427.9 (Q)
- net ST15: now also U430.9 (Q)
- net ST15J: now also U430.7 (J)
- net ST15K: now also U430.10 (K)
- net ST2: now also U431.5 (Q)
- net ST2D: now also U431.2 (D)
- net STLD: now also U426.10
- net TRP13Q: now also U432.3
- net UR10: now also U420.2 (I2)
- net UR11: now also U420.1 (I3)
- net UR8: now also U420.4 (I0)
- net UR9: now also U420.3 (I1)
- net VCC1: now also U414.1 (~{Mr}), U414.16 (VCC), U416.16 (VCC), U417.1 (~{Mr}), U417.16 (VCC), U418.16 (VCC), U419.16 (VCC), U420.16 (VCC), U421.1 (~{MR}), U421.16 (VCC), U422.16 (VCC), U423.16 (VCC), U424.1 (Mr), U424.16 (VCC), U427.6 (~{R}), U428.1 (~{Mr}), U428.16 (VCC), U429.16 (VCC), U430.2 (~{R}), U430.6 (~{R}), U431.1 (~{R}), U431.10 (~{S}), U431.13 (~{R}), U431.4 (~{S})
- net XR4: now also U421.11 (Q3)
- net XR5: now also U421.12 (Q2)
- net XR7: now also U421.14 (Q0)
- net ~{ADRV}: now also U425.4
- net ~{AEQZ}: now also U432.1
- net ~{ALS2}: now also U423.6 (~{Z})
- net ~{ALS6}: now also U422.6 (~{Z})
- net ~{AMAD0B}: now also U416.7 (~{E})
- net ~{AMS13}: now also U416.6 (~{Z})
- net ~{BIT2}: now also U420.6 (~{Z})
- net ~{CPUCR}: now also U432.9
- net ~{DP13}: now also U416.3 (I1)
- net ~{ENAPI}: now also U426.5
- net ~{ENARCLR}: now also U429.1 (~{MR})
- net ~{ENARLOAD}: now also U429.9 (~{PE})
- net ~{ENREGSK}: now also U426.11
- net ~{ENXRLOAD}: now also U421.9 (~{PE})
- net ~{GCLKC:1}: now also U421.2 (CP), U424.11 (Cp)
- net ~{GCLKC:2}: now also U429.2 (CP)
- net ~{INSTV}: now also U432.5
- net ~{IR12}: now also U417.3 (~{Q0}), U420.7 (~{E})
- net ~{IR13}: now also U417.6 (~{Q1})
- net ~{IR3}: now also U425.1
- net ~{IR6O11}: now also U426.12
- net ~{IR6}: now also U428.11 (~{Q2})
- net ~{IR8}: now also U425.13
- net ~{IRCLK}: now also U417.9 (Cp), U428.9 (Cp)
- net ~{MDCLK}: now also U414.9 (Cp)
- net ~{PCSCLK}: now also U425.6
- net ~{SETBIT13}: now also U416.2 (I2)
- net ~{SNS3}: now also U415.1
- net ~{SNS4}: now also U415.10
- net ~{SSNEQ1}: now also U426.1
- net ~{ST15}: now also U430.8 (~{Q})
- net ~{ST2CK}: now also U431.3 (C)
- net ~{ST2}: now also U431.6 (~{Q})
- net ~{TRP13A}: now also U432.4
- new net AR10: U429.13 (Q1)
- new net AR11: U429.14 (Q0)
- new net AR8: U429.11 (Q3)
- new net AR9: U429.12 (Q2)
- new net ARCR1: U429.10 (CET)
- new net BR6: U422.13 (I6)
- new net ER2: U423.3 (I1)
- new net ER6: U422.3 (I1), U424.13 (Q2)
- new net ER8: U424.7 (Dsl)
- new net LR6: U422.14 (I5)
- new net MDR12: U414.2 (Q0), U418.4 (I2a)
- new net MDR13: U414.5 (Q1), U418.12 (I2b)
- new net MDR14: U414.7 (Q2), U419.4 (I2a)
- new net MDR15: U414.10 (Q3), U419.12 (I2b)
- new net MR6: U422.1 (I3)
- new net PCS13: U416.12 (I7)
- new net PFMSKJ: U430.14 (J)
- new net PFMSKQ: U430.12 (Q)
- new net ST11D: U431.12 (D)
- new net ST1D: U425.8
- new net ST814LD: U427.10 (K)
- new net TRAP13: U416.1 (I3)
- new net UR12: U418.5 (I1a), U420.15 (I4)
- new net UR13: U418.11 (I1b), U420.14 (I5)
- new net UR14: U419.5 (I1a), U420.13 (I6)
- new net UR15: U419.11 (I1b), U420.12 (I7)
- new net XR2: U423.2 (I2)
- new net XR6: U421.13 (Q1), U422.2 (I2)
- new net XRCR2: U421.10 (CET)
- new net XRCR3: U421.15 (TC)
- new net ~{AEQBX}: U425.10, U426.6
- new net ~{APIS1D}: U425.11
- new net ~{IR14}: U417.11 (~{Q2}), U432.11
- new net ~{IR15}: U417.14 (~{Q3}), U432.13
- new net ~{IR4}: U428.3 (~{Q0})
- new net ~{IR5}: U428.6 (~{Q1})
- new net ~{IR7}: U426.13, U428.14 (~{Q3})
- new net ~{LDST1}: U425.9, U426.8
- new net ~{PFMSKQ}: U430.13 (~{Q})
- new net ~{SKSELOG1}: U425.12
- new net ~{SSNEQ2}: U415.8, U426.2
- new net ~{ST11CK}: U431.11 (C)
- new net ~{ST11}: U431.8 (~{Q})
- new net ~{ST14}: U427.8 (~{Q})
- no-connect marks 212 -> 229

Commit message: Finished Column 13 on AU2
Parts:
- added R172, R173, R174, R175, R176, R177, R178, R179: R, symbol Device:R
- added U433: 7432N, symbol 74xx:74LS32
- added U434: 74H00N, symbol 74xx:7400
- added U435: 74S65N, symbol TI980A:74S65N
- added U436, U440: 74151N, symbol 74xx:74LS151
- added U437, U449, U450: 7474N, symbol 74xx:74LS74
- added U438, U439, U441, U442: 74174N, symbol 74xx:74LS174
- added U443: 74194N, symbol 74xx:74LS194
- added U444: 7408N, symbol 74xx:74LS08
- added U445: 7402N, symbol 74xx:7402
- added U446, U448: 74153N, symbol 74xx:74LS153
- added U447, U451: 7400N, symbol 74xx:7400
Connections:
- net ALU0T: now also U447.12
- net ALU10: now also U443.5 (P2)
- net ALU11: now also U443.6 (P3), U444.12
- net ALU12: now also U444.9
- net ALU2: now also U446.13 (I3b), U447.1
- net ALU3: now also U446.3 (I3a)
- net ALU5: now also U435.2
- net ALU6: now also U435.9
- net ALU7: now also U435.1, U444.1
- net ALU8: now also U435.4, U443.3 (P0), U444.4
- net ALU9: now also U443.4 (P1)
- net ALUZ115: now also U435.8
- net AMAD1: now also U436.9 (S2), U440.9 (S2)
- net AMAD2: now also U436.10 (S1), U440.10 (S1)
- net AMAD3: now also U436.11 (S0), U440.11 (S0)
- net AR11: now also U440.4 (I0)
- net B10: now also U448.7 (Za)
- net B11: now also U448.9 (Zb)
- net BMAD1: now also U448.14 (S0)
- net BR6: now also U441.2 (Q0)
- net BR7: now also U441.5 (Q1)
- net C10: now also U439.13 (D4), U441.13 (D4), U442.13 (D4)
- net C11: now also U439.14 (D5), U441.14 (D5), U442.14 (D5)
- net C12: now also U438.3 (D0)
- net C13: now also U438.4 (D1)
- net C14: now also U438.6 (D2)
- net C15: now also U438.11 (D3)
- net C6: now also U439.3 (D0), U441.3 (D0), U442.3 (D0)
- net C7: now also U439.4 (D1), U441.4 (D1), U442.4 (D1)
- net C8: now also U439.6 (D2), U441.6 (D2), U442.6 (D2)
- net C9: now also U439.11 (D3), U441.11 (D3), U442.11 (D3)
- net ENBRLOAD: now also U447.9
- net ENERS0: now also U443.9 (S0), U446.14 (S0)
- net ENERS1: now also U443.10 (S1), U446.2 (S1)
- net ER0: now also U451.9
- net ER1: now also U446.11 (I1b)
- net ER11: now also U440.3 (I1), U443.12 (Q3), U445.11
- net ER12: now also U443.7 (Dsl), U445.12
- net ER15SELA: now also U451.3
- net ER2: now also U446.5 (I1a)
- net ER3: now also U445.8, U446.12 (I2b)
- net ER4: now also U445.9, U446.4 (I2a)
- net ER5: now also U445.2
- net ER6: now also U445.3
- net ER7: now also U443.2 (Dsr), U445.5
- net ER8: now also U443.15 (Q0), U445.6
- net ERLD: now also U434.9
- net EXPADR13: now also U434.1
- net EXPADR14: now also R173.2, U434.4
- net EXPADR8: now also R177.2
- net EXPTRAP: now also U434.2, U434.5
- net GCLKA:1: now also U434.10, U447.10
- net GND: now also U436.8 (GND), U438.13 (D4), U438.14 (D5), U438.8 (GND), U439.8 (GND), U440.8 (GND), U441.8 (GND), U442.8 (GND), U443.8 (GND), U446.1 (Ea), U446.15 (Eb), U446.8 (GND), U448.8 (GND)
- net INHMSA: now also U440.7 (~{E})
- net INHMSB: now also U448.1 (Ea), U448.15 (Eb)
- net IR10: now also U448.3 (I3a)
- net IR11: now also U448.13 (I3b)
- net IR14: now also U436.13 (I6)
- net LR6: now also U442.2 (Q0)
- net LR7: now also U442.5 (Q1)
- net MAR10: now also U448.6 (I0a)
- net MAR11: now also U448.10 (I0b)
- net MDR10: now also U448.4 (I2a)
- net MDR11: now also U448.12 (I2b)
- net MEM14: now also U436.14 (I5)
- net MR6: now also U439.2 (Q0)
- net MR7: now also U439.5 (Q1)
- net PC11: now also U440.12 (I7)
- net PNL14: now also U436.15 (I4)
- net R39: now also R176.2
- net R5: now also U448.2 (S1)
- net SELSKA: now also U451.6
- net ST0: now also U449.5 (Q)
- net ST0D: now also U449.2 (D)
- net ST11D: now also U444.11
- net ST12: now also U450.5 (Q)
- net ST14: now also U436.4 (I0)
- net ST56A: now also U451.11
- net ST7: now also U450.9 (Q)
- net ST8: now also U449.9 (Q)
- net ST9: now also U437.9 (Q)
- net ST9D: now also U437.12 (D)
- net STLD: now also U444.10, U444.13, U444.2, U444.5, U447.13, U447.2
- net TRAP13: now also U434.11
- net UR10: now also U448.5 (I1a)
- net UR11: now also U448.11 (I1b)
- net UR12: now also U438.2 (Q0)
- net UR13: now also U438.5 (Q1)
- net UR14: now also U438.7 (Q2)
- net UR15: now also U438.10 (Q3)
- net VCC1: now also R172.1, R173.1, R174.1, R175.1, R176.1, R177.1, R178.1, R179.1, U435.10, U435.11, U435.12, U435.13, U435.3, U435.5, U435.6, U436.16 (VCC), U437.10 (~{S}), U437.13 (~{R}), U438.1 (~{Mr}), U438.16 (VCC), U439.1 (~{Mr}), U439.16 (VCC), U440.16 (VCC), U441.1 (~{Mr}), U441.16 (VCC), U442.1 (~{Mr}), U442.16 (VCC), U443.1 (Mr), U443.16 (VCC), U446.16 (VCC), U448.16 (VCC), U449.1 (~{R}), U449.10 (~{S}), U449.13 (~{R}), U449.4 (~{S}), U450.1 (~{R}), U450.10 (~{S}), U450.13 (~{R}), U450.4 (~{S})
- net ~{ALS11}: now also U440.6 (~{Z})
- net ~{AMAD0B}: now also U436.7 (~{E})
- net ~{AMS14}: now also U436.6 (~{Z})
- net ~{APIS01CK}: now also U433.9
- net ~{APIS1D}: now also U433.6
- net ~{APIS2CK}: now also U433.1
- net ~{APIS2D}: now also U433.11
- net ~{APIS2EN}: now also U433.3
- net ~{APIST1}: now also U433.4
- net ~{APIST2}: now also U433.12
- net ~{AR15ER1}: now also U447.4
- net ~{BRCLK}: now also U441.9 (Cp), U447.8
- net ~{DP14}: now also U436.3 (I1)
- net ~{ENAPI}: now also U433.10, U433.13, U433.2, U433.5
- net ~{GCLKC:1}: now also U443.11 (Cp)
- net ~{LDST0}: now also U447.11
- net ~{LRCLK}: now also U442.9 (Cp)
- net ~{MRCLK}: now also U439.9 (Cp)
- net ~{R34}: now also R179.2, U451.1
- net ~{R54A}: now also U451.10
- net ~{SCER}: now also U451.2
- net ~{SETBIT14}: now also U436.2 (I2)
- net ~{SNS1}: now also R175.2
- net ~{SNS2}: now also R178.2
- net ~{SNS3}: now also R174.2
- net ~{SNS4}: now also R172.2
- net ~{ST0}: now also U449.6 (~{Q})
- net ~{ST12CK}: now also U450.3 (C)
- net ~{ST2LD}: now also U447.3
- net ~{ST479CK}: now also U437.11 (C), U450.11 (C)
- net ~{ST5}: now also U451.12
- net ~{ST6}: now also U451.13
- net ~{TRP13A}: now also U434.13
- net ~{URCLK}: now also U438.9 (Cp)
- new net BR10: U441.12 (Q4)
- new net BR11: U440.13 (I6), U441.15 (Q5)
- new net BR8: U441.7 (Q2)
- new net BR9: U441.10 (Q3)
- new net ER10: U443.13 (Q2)
- new net ER9: U443.14 (Q1)
- new net ERIN1A: U447.6
- new net ERIN2: U446.9 (Zb)
- new net ERIN3: U446.7 (Za)
- new net LR10: U442.12 (Q4)
- new net LR11: U440.14 (I5), U442.15 (Q5)
- new net LR8: U442.7 (Q2)
- new net LR9: U442.10 (Q3)
- new net MR10: U439.12 (Q4)
- new net MR11: U439.15 (Q5), U440.1 (I3)
- new net MR8: U439.7 (Q2)
- new net MR9: U439.10 (Q3)
- new net PCS14: U436.12 (I7)
- new net SR11: U440.15 (I4)
- new net ST12D: U444.8, U450.2 (D)
- new net ST7D: U444.3, U450.12 (D)
- new net ST8D: U444.6, U449.12 (D)
- new net TRAP14: U436.1 (I3)
- new net XR11: U440.2 (I2)
- new net ~{APIS01EN}: U433.8
- new net ~{ER0ER1}: U447.5, U451.8
- new net ~{ER123CK}: U434.8
- new net ~{ERB}: U445.10
- new net ~{ERC}: U445.1
- new net ~{ERD}: U445.4
- new net ~{ERE}: U445.13
- new net ~{SKSELO01}: U451.4
- new net ~{SKSFLOG2}: U451.5
- new net ~{ST01CK}: U449.3 (C)
- new net ~{ST12}: U450.6 (~{Q})
- new net ~{ST7}: U450.8 (~{Q})
- new net ~{ST8CK}: U449.11 (C)
- new net ~{ST8}: U449.8 (~{Q})
- new net ~{ST9}: U437.8 (~{Q})
- new net ~{TRAP13A}: U434.12, U434.3
- new net ~{TRAP14A}: U434.6
- no-connect marks 229 -> 241
