File: TI980A-Arithmetic-Unit/AU2.kicad_sch (KiCad schematic)
At the start: 339 parts, among them U15 74H40N, U16 74H40N, U17 74H40N, U18 74H11N, U19 74H04N, U20 74H40N, U231 7451N, U232 74H101, U233 74187, U234 74187, U235 74187, U236 74187, U237 74H04N, U238 74187, U239 74187, U240 74187, U241 74187, U242 74187, U243 7430N, U244 7430N, U245 74H11N, U246 74H00N, U247 74H74N, U248 74187, U249 74187, U250 74187, U251 74187, U252 74187, U253 7451N, U254 7437N, U255 74S65N, U256 74H00N, U257 74H74N, U258 74H74N, U259 74H74N, U260 7410N, U261 7420N, U262 74H21N, U263 74H11N, U264 7474N, U265 74H04N, U266 74153N, U267 74H20N, U268 7474N, U269 74181, U270 74153, U271 74153, U272 74H11N, U273 74174N, U274 74S10N, U275 7442N, U276 74H51N, U277 74H11N, U278 74H51N, U279 74153N, U280 74151N, U281 74151N, U282 74151N, U283 74151N, U284 74151N, U285 74153N, U286 74163N, U287 74153N, U288 74H51N, U289 74H51N, U290 74H00N, U291 74H00N, U292 74H11N, U293 74153N, U294 74163N, U295 74153N, U296 7442N, U297 74H00N, U298 74H21N, U299 74153N, U300 74H04N, U301 74H103N, U302 7410N, U303 74H51N, U304 7442N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

Commit message: Finished Column 14 on AU2
Parts:
- added U452, U453: 74157N, symbol 74xx:74LS157
- added U454: 74S65N, symbol TI980A:74S65N
- added U455, U468: 74174N, symbol 74xx:74LS174
- added U456, U457, U461, U462, U469, U471, U472: 74163N, symbol 74xx:74LS163
- added U458, U459, U460: 74151N, symbol 74xx:74LS151
- added U463: 7402N, symbol 74xx:7402
- added U464: 7430N, symbol 74xx:74LS30
- added U465: 74H10N, symbol 74xx:74LS10
- added U466: 74153N, symbol 74xx:74LS153
- added U467: 74H00N, symbol 74xx:7400
- added U470: 7474N, symbol 74xx:74LS74
Connections:
- net ALU1: now also U466.3 (I3a)
- net ALU10: now also U453.10 (I1c), U454.9, U470.12 (D)
- net ALU11: now also U453.13 (I1d), U454.1
- net ALU12: now also U452.3 (I1a), U454.4
- net ALU13: now also U452.6 (I1b)
- net ALU14: now also U452.10 (I1c)
- net ALU15: now also U452.13 (I1d)
- net ALU8: now also U453.3 (I1a)
- net ALU9: now also U453.6 (I1b), U454.2
- net ALUZ115: now also U454.8
- net AMAD1: now also U458.9 (S2), U459.9 (S2), U460.9 (S2)
- net AMAD2: now also U458.10 (S1), U459.10 (S1), U460.10 (S1)
- net AMAD3: now also U458.11 (S0), U459.11 (S0), U460.11 (S0)
- net AR0: now also U472.11 (Q3)
- net AR1: now also U472.12 (Q2)
- net AR10: now also U460.4 (I0)
- net AR14: now also U471.13 (Q1)
- net AR15: now also U471.14 (Q0)
- net AR2: now also U472.13 (Q1)
- net AR3: now also U472.14 (Q0)
- net AR8: now also U458.4 (I0)
- net AR9: now also U459.4 (I0)
- net ARCR1: now also U471.15 (TC)
- net BR10: now also U460.13 (I6)
- net BR8: now also U458.13 (I6)
- net BR9: now also U459.13 (I6)
- net C0: now also U468.3 (D0), U469.6 (D3), U472.6 (D3)
- net C1: now also U468.4 (D1), U469.5 (D2), U472.5 (D2)
- net C10: now also U456.4 (D1), U457.4 (D1), U461.4 (D1)
- net C11: now also U456.3 (D0), U457.3 (D0), U461.3 (D0)
- net C12: now also U462.6 (D3), U471.6 (D3)
- net C13: now also U462.5 (D2), U471.5 (D2)
- net C14: now also U462.4 (D1), U471.4 (D1)
- net C15: now also U462.3 (D0), U471.3 (D0)
- net C2: now also U468.6 (D2), U469.4 (D1), U472.4 (D1)
- net C3: now also U468.11 (D3), U469.3 (D0), U472.3 (D0)
- net C4: now also U468.13 (D4)
- net C5: now also U468.14 (D5)
- net C8: now also U456.6 (D3), U457.6 (D3), U461.6 (D3)
- net C9: now also U456.5 (D2), U457.5 (D2), U461.5 (D2)
- net ENARINC: now also U471.7 (CEP), U472.7 (CEP)
- net ENERS0: now also U466.14 (S0)
- net ENERS1: now also U466.2 (S1)
- net ENPCINC: now also U456.7 (CEP)
- net ENSRINC: now also U461.7 (CEP), U462.7 (CEP)
- net ENXRINC: now also U457.7 (CEP), U469.7 (CEP)
- net ER1: now also U463.11
- net ER10: now also U460.3 (I1), U463.3
- net ER13: now also U463.8
- net ER14: now also U463.9
- net ER15: now also U463.5
- net ER2: now also U463.12, U466.4 (I2a)
- net ER8: now also U458.3 (I1)
- net ER9: now also U459.3 (I1), U463.2
- net GCLKA:1: now also U467.10, U467.5
- net GND: now also U455.13 (D4), U455.14 (D5), U455.8 (GND), U456.8 (GND), U457.8 (GND), U458.8 (GND), U459.8 (GND), U460.8 (GND), U461.8 (GND), U462.8 (GND), U463.6, U466.1 (Ea), U466.8 (GND), U468.8 (GND), U469.8 (GND), U471.8 (GND), U472.8 (GND)
- net GND1: now also U452.8 (GND), U453.8 (GND)
- net INHMSA: now also U458.7 (~{E}), U459.7 (~{E}), U460.7 (~{E})
- net IOUT10: now also U453.9 (Zc)
- net IOUT11: now also U453.12 (Zd)
- net IOUT12: now also U452.4 (Za)
- net IOUT13: now also U452.7 (Zb)
- net IOUT14: now also U452.9 (Zc)
- net IOUT15: now also U452.12 (Zd)
- net IOUT8: now also U453.4 (Za)
- net IOUT9: now also U453.7 (Zb)
- net LR10: now also U460.14 (I5)
- net LR8: now also U458.14 (I5)
- net LR9: now also U459.14 (I5)
- net MR10: now also U460.1 (I3)
- net MR8: now also U458.1 (I3)
- net MR9: now also U459.1 (I3)
- net PC10: now also U453.11 (I0c), U456.13 (Q1), U460.12 (I7)
- net PC11: now also U453.14 (I0d), U456.14 (Q0)
- net PC8: now also U453.2 (I0a), U456.11 (Q3), U458.12 (I7)
- net PC9: now also U453.5 (I0b), U456.12 (Q2), U459.12 (I7)
- net PCCR2: now also U456.15 (TC)
- net PCS12: now also U455.2 (Q0)
- net PCS13: now also U455.5 (Q1)
- net PCS14: now also U455.7 (Q2)
- net PCS15: now also U455.10 (Q3)
- net SR11: now also U461.14 (Q0)
- net SRCR2: now also U461.15 (TC)
- net ST1: now also U470.5 (Q)
- net ST10: now also U470.9 (Q)
- net ST1D: now also U470.2 (D)
- net ST814LD: now also U467.11
- net STLD: now also U467.4
- net TRAP14: now also U467.3
- net UR0: now also U468.2 (Q0)
- net UR1: now also U468.5 (Q1)
- net UR2: now also U468.7 (Q2)
- net UR3: now also U468.10 (Q3)
- net UR4: now also U468.12 (Q4)
- net UR5: now also U468.15 (Q5)
- net VCC1: now also U452.16 (VCC), U453.16 (VCC), U454.10, U454.11, U454.12, U454.13, U454.3, U454.5, U454.6, U455.1 (~{Mr}), U455.16 (VCC), U456.1 (~{MR}), U456.16 (VCC), U457.1 (~{MR}), U457.16 (VCC), U458.16 (VCC), U459.16 (VCC), U460.16 (VCC), U461.1 (~{MR}), U461.16 (VCC), U462.1 (~{MR}), U462.10 (CET), U462.16 (VCC), U466.16 (VCC), U468.1 (~{Mr}), U468.16 (VCC), U469.1 (~{MR}), U469.16 (VCC), U470.1 (~{R}), U470.10 (~{S}), U470.13 (~{R}), U470.4 (~{S}), U471.1 (~{MR}), U471.10 (CET), U471.16 (VCC), U472.1 (~{MR}), U472.16 (VCC)
- net XR0: now also U469.11 (Q3)
- net XR1: now also U469.12 (Q2)
- net XR11: now also U457.14 (Q0)
- net XR2: now also U469.13 (Q1)
- net XR3: now also U469.14 (Q0)
- net XRCR2: now also U457.15 (TC)
- net XRCR3: now also U469.10 (CET)
- net XRMAX: now also U469.15 (TC)
- net ~{ALS10}: now also U460.6 (~{Z})
- net ~{ALS8}: now also U458.6 (~{Z})
- net ~{ALS9}: now also U459.6 (~{Z})
- net ~{APIS01EN}: now also U465.5
- net ~{ENARLOAD}: now also U471.9 (~{PE}), U472.9 (~{PE})
- net ~{ENIOUT}: now also U452.15 (E), U453.15 (E)
- net ~{ENPCLOAD}: now also U456.9 (~{PE})
- net ~{ENSRLOAD}: now also U461.9 (~{PE}), U462.9 (~{PE})
- net ~{ENST01}: now also U465.3
- net ~{ENXRLOAD}: now also U457.9 (~{PE}), U469.9 (~{PE})
- net ~{ERB}: now also U464.2
- net ~{ERC}: now also U464.3
- net ~{ERD}: now also U464.4
- net ~{ERE}: now also U463.1, U464.5
- net ~{ERZ115}: now also U464.8
- net ~{GCLKC:1}: now also U456.2 (CP), U457.2 (CP), U461.2 (CP), U462.2 (CP), U469.2 (CP)
- net ~{GCLKC:2}: now also U471.2 (CP), U472.2 (CP)
- net ~{IICLR}: now also U467.13
- net ~{PCOUTA}: now also U452.1 (S), U453.1 (S)
- net ~{PCSCLK}: now also U455.9 (Cp)
- net ~{ST01CK}: now also U470.3 (C)
- net ~{ST11CK}: now also U467.6, U470.11 (C)
- net ~{ST1}: now also U470.6 (~{Q})
- net ~{STLD}: now also U465.4, U467.12
- net ~{TRAP14A}: now also U467.1
- net ~{TRP14A}: now also U467.2
- net ~{URCLK}: now also U468.9 (Cp)
- new net AR12: U471.11 (Q3)
- new net AR13: U471.12 (Q2)
- new net ARCR3: U472.10 (CET)
- new net ARMAX: U472.15 (TC)
- new net ENCMPCK: U465.6, U467.9
- new net ENINIA: U466.5 (I1a)
- new net ERIN1: U466.7 (Za)
- new net PC12: U452.2 (I0a), U455.3 (D0)
- new net PC13: U452.5 (I0b), U455.4 (D1)
- new net PC14: U452.11 (I0c), U455.6 (D2)
- new net PC15: U452.14 (I0d), U455.11 (D3)
- new net PCCR1: U456.10 (CET)
- new net SR10: U460.15 (I4), U461.13 (Q1)
- new net SR12: U462.11 (Q3)
- new net SR13: U462.12 (Q2)
- new net SR14: U462.13 (Q1)
- new net SR15: U462.14 (Q0)
- new net SR8: U458.15 (I4), U461.11 (Q3)
- new net SR9: U459.15 (I4), U461.12 (Q2)
- new net SRCR1: U461.10 (CET), U462.15 (TC)
- new net XR10: U457.13 (Q1), U460.2 (I2)
- new net XR8: U457.11 (Q3), U458.2 (I2)
- new net XR9: U457.12 (Q2), U459.2 (I2)
- new net XRCR1: U457.10 (CET)
- new net ~{ERA}: U463.13, U464.1
- new net ~{ERF}: U464.6
- new net ~{ERG}: U463.10, U464.11
- new net ~{ERH}: U463.4, U464.12
- new net ~{ST10}: U470.8 (~{Q})
- new net ~{STO1CK}: U467.8
- no-connect marks 241 -> 261
