File: TI980A-Arithmetic-Unit/AU2.kicad_sch (KiCad schematic)
At the start: 375 parts, among them U15 74H40N, U16 74H40N, U17 74H40N, U18 74H11N, U19 74H04N, U20 74H40N, U231 7451N, U232 74H101, U233 74187, U234 74187, U235 74187, U236 74187, U237 74H04N, U238 74187, U239 74187, U240 74187, U241 74187, U242 74187, U243 7430N, U244 7430N, U245 74H11N, U246 74H00N, U247 74H74N, U248 74187, U249 74187, U250 74187, U251 74187, U252 74187, U253 7451N, U254 7437N, U255 74S65N, U256 74H00N, U257 74H74N, U258 74H74N, U259 74H74N, U260 7410N, U261 7420N, U262 74H21N, U263 74H11N, U264 7474N, U265 74H04N, U266 74153N, U267 74H20N, U268 7474N, U269 74181, U270 74153, U271 74153, U272 74H11N, U273 74174N, U274 74S10N, U275 7442N, U276 74H51N, U277 74H11N, U278 74H51N, U279 74153N, U280 74151N, U281 74151N, U282 74151N, U283 74151N, U284 74151N, U285 74153N, U286 74163N, U287 74153N, U288 74H51N, U289 74H51N, U290 74H00N, U291 74H00N, U292 74H11N, U293 74153N, U294 74163N, U295 74153N, U296 7442N, U297 74H00N, U298 74H21N, U299 74153N, U300 74H04N, U301 74H103N, U302 7410N, U303 74H51N, U304 7442N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

Commit message: All Register Except Status Register Done
Connections:
- net ENINIA is gone; now on net ERIN1A: U466.5 (I1a)
Other:
- note added: "A Register(AR) and Control"
- note added: "B Register and Control"
- note added: "E Register"
- note added: "Instruction Register (IR) and Control"
- note added: "L Register and Control"
- note added: "M Register and Control"
- note added: "MA Increment Control (For AU Only)"
- note added: "MA Increment Control (For Memory Controller Only)"
- note added: "MA Load Control"
- note added: "Memory Address Register (MAR) and Control"
- note added: "Memory Control MA Load Control"
- note added: "Memory Data Register (MDR) and Control"
- note added: "Program Counter (PC)"
- note added: "Program Counter Content Save Register (PCS)"
- note added: "S Register Bit 16 (For Byte Addressing)"
- note added: "S Register and Control"
- note added: "Shift & Load Controls"
- note added: "Utility Register (UR) and Control"
- note added: "X Register and Control"
- moved on the sheet: U487A

Commit message: Finished AU2 Logic Blocks Identification
Connections:
- net ENDVCK is gone; now on net ENOVCK: U358.4
- net PEMSKJ is gone; now on net PFMSKJ: U374.8
- net ST40 is gone; now on net ST4D: U268.12 (D)
- net ~{ENMRLOV} is gone; now on net ~{ENRMLOV}: U264.6 (~{Q})
- net ~{ENSFR} is gone; now on net ~{ENSER}: U323.2 (1)
- net ~{PENSKQ} is gone; now on net ~{PFMSKQ}: U342.13
- net ~{STO1CK} is gone; now on net ~{ST01CK}: U467.8
- net R20: now also R129.2; no longer R131.2
- net ~{ERE}: no longer U445.13
- net ~{ERF}: now also U445.13
- net ~{R12}: now also R126.2; no longer R120.2
- net ~{R21}: now also R131.2; no longer R129.2
- net ~{R9}: now also R120.2; no longer R126.2
Other:
- note added: "A0=B0"
- note added: "ALU Mode Select Input"
- note added: "ALU Outputs are Zeros"
- note added: "ALU1-ALU15 are Zeros"
- note added: "Buffered ROM Address"
- note added: "Control Logic ROMs"
- note added: "Control ROMs Pullups"
- note added: "Data Bus A = data Bus B"
- note added: "E Register Bits 1-15 are Zeros"
- note added: "Enable Normal Overflow Flag"
- note added: "Input Data Bus Pullups"
- note added: "Invert B0 Control"
- note added: "Output to Backplane"
- note added: "PIF Enable Signal"
- note added: "Panel Switches Pullups"
- note added: "ROM Address Registers"
- note added: "ST0 Arithmetic Greater Than Input Term"
- note added: "ST0 Load Term"
- note added: "ST0 Logical Greater Than Output Term"
- note added: "ST2 Add-Subtract Overflow Input Term"
- note added: "ST3 Carry Term 1"
- note added: "ST3 Carry Term 2"
- note added: "ST3 Load Input Term"
- note added: "Sense Register Pullups"
- note added: "Status Bit 0-ST0 (Greater Than Condition Bit)"
- note added: "Status Bit 1-ST1 (Equal to Condition Bit)"
- note added: "Status Bit 10-ST10 (Indexing Bit)"
- note added: "Status Bit 11-ST11 (Memory Parity Error Mask Bit)"
- note added: "Status Bit 12-ST12 (DMAC Interrupt Mask Bit)"
- note added: "Status Bit 14-ST14 (Memory Parity Error Indicator)"
- note added: "Status Bit 15-ST15 (Power Failure Indicator)"
- note added: "Status Bit 2-ST2 (Overflow Condition Bit)"
- note added: "Status Bit 3-ST3 (Carry Indicator)"
- note added: "Status Bit 4-ST4 (PIF Mask Bit)"
- note added: "Status Bit 5-ST5 (PIF Address Violation Indicator)"
- note added: "Status Bit 6-ST6 (PIF Instruction Violation Indicator)"
- note added: "Status Bit 7-ST7 (I/O Interrupt Mask Bit)"
- note added: "Status Bit 8-ST8 (Extended Interrupt Feature Control)"
- note added: "Status Bit 9-ST9 (Lower Limit Memory Bias Enable)"
- note added: "Status Bit Control Decoder"
- note added: "Subtract Immediate Flag"
- moved on the sheet: U487A

Commit message: AU Schematic COMPLETE!!!
Connections:
- net A10: now also U353.8
Other:
- note added: "Bus A (Least Significant)"
- note added: "Bus A (Most Significant)"
- note added: "Status Register and Control"
- title: (none) -> Arithetic Unit #2 
- moved on the sheet: AX08-CTP1, AX08-CTP2, U487A, U487B
