File: IO_Modules/IO_Interface_Card/IO_Interface_Card.kicad_pcb (KiCad board)
At the start: 2 copper layers, 105 parts

Commit message: Implemented Footprint for Card Edge connectors
Parts:
- added P1: Conn_02x40_Odd_Even, TI980-Backplane:Backplane-Connector, F.Cu at (155.9, 169.8)
- added P2: Conn_02x36_Top_Bottom, TI980-Backplane:Type-2-Top-Edge-Connector, F.Cu at (155.9, -27.1)
- moved E12 195.1 mm to (222.3, 52.3)
- moved E11 195.0 mm to (222.4, 49.1)
- moved C11 38.3 mm to (227.6, 1.75)
- moved R8 36.7 mm to (228.7, 17.6)
- moved C8 36.4 mm to (204.0, 1.26)
- moved R6 36.1 mm to (223.3, 17.3)
- moved R24 35.6 mm to (219.1, 17.3)
- moved R5 35.6 mm to (215.6, 17.2)
- moved C10 34.1 mm to (215.6, 24.1)
- moved Z20 33.8 mm to (223.5, 44.3)
- moved R4 31.7 mm to (179.4, 16.8)
- moved R1 31.7 mm to (176.2, 16.9)
- moved R7 31.7 mm to (182.5, 16.7)
- moved R18 30.7 mm to (167.3, 16.7)
- moved R17 30.7 mm to (163.3, 16.7)
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Other:
- board outline added: 177.8 x 180.8 mm
- board text added: "( )"
- board text added: "9607590"
- board text added: "ASSY NO. 960757-0001"
- board text added: "I/"
- board text added: "INTERFACE"
- board text added: "LOGIC"
- board text added: "NO."
- board text added: "O"
- board text added: "SERIAL"
