File: IO_Modules/IO_Interface_Card/IO_Interface_Card.kicad_sch (KiCad schematic)
At the start: 95 parts, among them P1 Conn_02x40_Odd_Even, P2 Conn_02x36_Top_Bottom

Commit message: Implemented Footprint for Card Edge connectors
Parts:
- P1: footprint (none) -> TI980-Backplane:Backplane-Connector
- P2: footprint (none) -> TI980-Backplane:Type-2-Top-Edge-Connector; symbol Connector_Generic:Conn_02x36_Top_Bottom -> Connector_Generic:Conn_02x36_Odd_Even
Connections:
- net A: now also P2.2 (Pin_2); no longer P2.37 (Pin_37)
- net B: now also P2.4 (Pin_4); no longer P2.38 (Pin_38)
- net C: now also P2.6 (Pin_6); no longer P2.39 (Pin_39)
- net D: now also P2.8 (Pin_8); no longer P2.40 (Pin_40)
- net E: now also P2.10 (Pin_10); no longer P2.41 (Pin_41)
- net F: now also P2.12 (Pin_12); no longer P2.42 (Pin_42)
- net GND: now also P2.15 (Pin_15), P2.21 (Pin_21), P2.35 (Pin_35), P2.37 (Pin_37), P2.39 (Pin_39), P2.43 (Pin_43), P2.45 (Pin_45), P2.49 (Pin_49), P2.53 (Pin_53), P2.57 (Pin_57), P2.61 (Pin_61), P2.65 (Pin_65), P2.67 (Pin_67), P2.71 (Pin_71); no longer P2.10 (Pin_10), P2.16 (Pin_16), P2.18 (Pin_18), P2.2 (Pin_2), P2.20 (Pin_20), P2.22 (Pin_22), P2.23 (Pin_23), P2.27 (Pin_27), P2.29 (Pin_29), P2.34 (Pin_34), P2.36 (Pin_36), P2.4 (Pin_4), P2.6 (Pin_6), P2.8 (Pin_8)
- net H: now also P2.14 (Pin_14); no longer P2.43 (Pin_43)
- net J: now also P2.16 (Pin_16); no longer P2.44 (Pin_44)
- net K: now also P2.18 (Pin_18); no longer P2.45 (Pin_45)
- net L: now also P2.20 (Pin_20); no longer P2.46 (Pin_46)
- net M: now also P2.22 (Pin_22); no longer P2.47 (Pin_47)
- net N: now also P2.24 (Pin_24); no longer P2.48 (Pin_48)
- net P: now also P2.26 (Pin_26); no longer P2.49 (Pin_49)
- net P2-15: now also P2.29 (Pin_29); no longer P2.15 (Pin_15)
- net R: now also P2.28 (Pin_28); no longer P2.50 (Pin_50)
- net S: now also P2.30 (Pin_30); no longer P2.51 (Pin_51)
- net SYSCLK: now also P2.60 (Pin_60); no longer P2.66 (Pin_66)
- net T: now also P2.32 (Pin_32); no longer P2.52 (Pin_52)
- net U: now also P2.34 (Pin_34); no longer P2.53 (Pin_53)
- net V: now also P2.36 (Pin_36); no longer P2.54 (Pin_54)
- net W: now also P2.38 (Pin_38); no longer P2.55 (Pin_55)
- net X: now also P2.40 (Pin_40); no longer P2.56 (Pin_56)
- net Y: now also P2.42 (Pin_42); no longer P2.57 (Pin_57)
- net Z: now also P2.44 (Pin_44); no longer P2.58 (Pin_58)
- net ~{A}: now also P2.46 (Pin_46); no longer P2.59 (Pin_59)
- net ~{B}: now also P2.48 (Pin_48); no longer P2.60 (Pin_60)
- net ~{C}: now also P2.50 (Pin_50); no longer P2.61 (Pin_61)
- net ~{DP10A}: now also P2.41 (Pin_41); no longer P2.21 (Pin_21)
- net ~{DP12A}: now also P2.68 (Pin_68); no longer P2.70 (Pin_70)
- net ~{DP13A}: now also P2.66 (Pin_66); no longer P2.69 (Pin_69)
- net ~{DP14A}: now also P2.63 (Pin_63); no longer P2.32 (Pin_32)
- net ~{DP15A}: now also P2.64 (Pin_64); no longer P2.68 (Pin_68)
- net ~{DP2A}: now also P2.27 (Pin_27); no longer P2.14 (Pin_14)
- net ~{DP5A}: now also P2.23 (Pin_23); no longer P2.12 (Pin_12)
- net ~{D}: now also P2.52 (Pin_52); no longer P2.62 (Pin_62)
- net ~{E}: now also P2.54 (Pin_54); no longer P2.63 (Pin_63)
- net ~{F}: now also P2.56 (Pin_56); no longer P2.64 (Pin_64)
- net ~{H}: now also P2.58 (Pin_58); no longer P2.65 (Pin_65)
- net ~{IOUT0}: now also P2.55 (Pin_55); no longer P2.28 (Pin_28)
- net ~{IOUT12}: now also P2.47 (Pin_47); no longer P2.24 (Pin_24)
- net ~{IOUT15}: now also P2.51 (Pin_51); no longer P2.26 (Pin_26)
- net ~{IOUT4}: now also P2.70 (Pin_70); no longer P2.71 (Pin_71)
- net ~{IOUT5}: now also P2.69 (Pin_69); no longer P2.35 (Pin_35)
- net ~{IOUT6}: now also P2.59 (Pin_59); no longer P2.30 (Pin_30)
- net ~{IOUT7}: now also P2.62 (Pin_62); no longer P2.67 (Pin_67)
