File: IO_Modules/IO_Expander_2/IO_Expander_2.kicad_sch (KiCad schematic)
At the start: 57 parts, among them P1 Card Edge

Commit message: Added IO Card Images and Fixed Error on AU1
Parts:
- C1, C7: footprint (none) -> Capacitor_THT:CP_Axial_L11.0mm_D6.0mm_P18.00mm_Horizontal
- C2, C3, C4, C5, C6: footprint (none) -> Capacitor_THT:C_Disc_D7.5mm_W2.5mm_P5.00mm
- E1, E10, E11, E12, E13, E14, E15, E16, E17, E18, E2, E9: footprint (none) -> Connector_PinHeader_2.54mm:PinHeader_1x01_P2.54mm_Vertical
- P1: footprint (none) -> TI980-Backplane:Backplane-Connector
- R1, R10, R11, R12, R13, R14, R15, R16, R17, R2, R3, R4, R5, R6, R7, R8, R9: footprint (none) -> Resistor_THT:R_Axial_DIN0207_L6.3mm_D2.5mm_P10.16mm_Horizontal
- Z1, Z10, Z11, Z12, Z13, Z14, Z15, Z16, Z17, Z18, Z19, Z2, Z20, Z3, Z4, Z5, Z6, Z7, Z8, Z9: footprint (none) -> Package_DIP:DIP-14_W7.62mm_Socket_LongPads
Connections:
- net GND: now also C2.1, C3.1, C4.1, C5.1, C6.1; no longer C2.2, C3.2, C4.2, C5.2, C6.2
- net VCC: now also C2.2, C3.2, C4.2, C5.2, C6.2; no longer C2.1, C3.1, C4.1, C5.1, C6.1
Other:
- moved on the sheet: C2, C3, C4, C5, C6
